File: antennas.kicad_sch (KiCad schematic)
At the start: 20 parts, among them U5 Antenna_1002427, U8 Antenna_1002427

Commit message: WIP
Parts:
- removed C40: 1.8pF, Capacitor_SMD:C_0402_1005Metric, symbol Device:C_Small
- removed C41: 5.6pF, Capacitor_SMD:C_0402_1005Metric, symbol Device:C_Small
- removed C42: DNP, Capacitor_SMD:C_0402_1005Metric, symbol Device:C_Small
- removed R40, R41, R42, R43: 0ohm, Resistor_SMD:R_0402_1005Metric, symbol Device:R
- removed RF4: KH-IPEX-4-K501-29, cacophony-footprints:IPEX4-SMD_4P-L1.8-W1.7-LS2.0-L_KH-IPEX4-2020, symbol cacophony-symbols:KH-IPEX-4-K501-29
- removed U8: Antenna_1002427, cacophony-footprints:ANTENNA_1002427_ISM, symbol cacophony-symbols:Antenna_1002427
Other:
- note removed: "ISM Layout"
