File: thermal-camera-v2.kicad_pcb (KiCad board)
At the start: 2 copper layers, 100 x 100 mm, 71 parts, among them J1 Raspberry_Pi_2_3, J2 Conn_01x02, J3 Conn_01x10, Q1 Q_PMOS_GSD, Q2 Q_PMOS_GSD, U1 STM32F030C8Tx, U10 ME6216A28XG, U12 3N25000G33YC, U13 TD6810, U14 TD6810, U15 MMC5633NJL, U16 Ai-Thinker-Ra-01, U2 SHT30-DIS, U3 ATtiny85-20P, U4 LMR16030S, U5 XC6206PxxxMR, U7 PCF8563T, U8 XC6206PxxxMR, U9 MAX98357, Y1 Crystal

Commit message: WIP
Parts:
- removed D5: D_Shockley, Diode_SMD:D_SMA
- removed LS1: Speaker, Connector_JST:JST_XA_S02B-XASK-1_1x02_P2.50mm_Horizontal
- removed Q2: Q_PMOS_GSD, Package_TO_SOT_SMD:SOT-23
- removed R`1: 3.3R, Resistor_SMD:R_0805_2012Metric
- added AE1: Antenna, cacophony-footprints:ANT-8_9-PW-LPN, F.Cu at (177.1, 77.5)
- added C101: 220uF, Capacitor_SMD:CP_Elec_8x10, B.Cu at (84.9, 81.6)
- added C102: 22uF, Capacitor_SMD:C_0805_2012Metric, B.Cu at (105.5, 87.1)
- added C103: 22uF, Capacitor_SMD:C_0805_2012Metric, B.Cu at (103.4, 87.1)
- added C104: 1nF, Capacitor_SMD:C_0402_1005Metric, B.Cu at (101.8, 87.2)
- added C105: 1nF, Capacitor_SMD:C_0402_1005Metric, B.Cu at (91.3, 87.8)
- added C106: 47pF, Capacitor_SMD:C_0402_1005Metric, B.Cu at (92.8, 87.3)
- added C107: 10nF, Capacitor_SMD:C_0402_1005Metric, B.Cu at (101.8, 90.1)
- added C108: 100nF, Capacitor_SMD:C_0402_1005Metric, B.Cu at (92.8, 86.2)
- added C109: 1nF, Capacitor_SMD:C_0402_1005Metric, B.Cu at (101.8, 82.1)
- added C110: 22uF, Capacitor_SMD:C_0603_1608Metric, B.Cu at (103.1, 82.1)
- added C111: 22uF, Capacitor_SMD:C_0603_1608Metric, B.Cu at (104.7, 82.1)
- added C201: 220uF, Capacitor_SMD:CP_Elec_8x10, B.Cu at (84.9, 68.3)
- added C202: 22uF, Capacitor_SMD:C_0805_2012Metric, B.Cu at (104.8, 64.0)
- added C203: 22uF, Capacitor_SMD:C_0805_2012Metric, B.Cu at (107.0, 64.0)
- added C204: 1nF, Capacitor_SMD:C_0402_1005Metric, B.Cu at (108.5, 63.5)
- added C205: 1nF, Capacitor_SMD:C_0402_1005Metric, B.Cu at (119.0, 62.9)
- added C206: 47pF, Capacitor_SMD:C_0402_1005Metric, B.Cu at (117.5, 63.4)
- added C207: 10nF, Capacitor_SMD:C_0402_1005Metric, B.Cu at (108.5, 60.5)
- added C208: 100nF, Capacitor_SMD:C_0402_1005Metric, B.Cu at (117.5, 64.5)
- added C209: 1nF, Capacitor_SMD:C_0402_1005Metric, B.Cu at (108.5, 68.5)
- added C26: 22uF, Capacitor_SMD:C_0603_1608Metric, F.Cu at (162.0, 126.7)
- added C27: 220nF, Capacitor_SMD:C_0402_1005Metric, F.Cu at (153.4, 136.6)
- added C28: 22uF, Capacitor_SMD:C_0603_1608Metric, B.Cu at (105.5, 68.7)
- added C29: 22uF, Capacitor_SMD:C_0603_1608Metric, B.Cu at (104.0, 68.7)
- added C30: 22uF, Capacitor_SMD:C_0603_1608Metric, B.Cu at (102.3, 68.7)
- added C31: 22uF, Capacitor_SMD:C_0603_1608Metric, B.Cu at (107.9, 82.1)
- added C32: 22uF, Capacitor_SMD:C_0603_1608Metric, B.Cu at (107.2, 68.7)
- added C33: 22uF, Capacitor_SMD:C_0603_1608Metric, B.Cu at (106.3, 82.1)
- added C34: 10uF, Capacitor_SMD:C_0603_1608Metric, F.Cu at (155.3, 71.0)
- added C35: 22uF, Capacitor_SMD:C_0805_2012Metric, B.Cu at (102.8, 64.0)
- added C36: 22uF, Capacitor_SMD:C_0805_2012Metric, B.Cu at (107.6, 87.1)
- added C37: 220nF, Capacitor_SMD:C_0402_1005Metric, B.Cu at (120.2, 102.2)
- added C38: 220nF, Capacitor_SMD:C_0402_1005Metric, B.Cu at (152.9, 93.4)
- added C39: DNP, Capacitor_SMD:C_0402_1005Metric, F.Cu at (161.9, 62.9)
- added C40: 1.8pF, Capacitor_SMD:C_0402_1005Metric, F.Cu at (174.2, 137.1)
- added C41: 5.6pF, Capacitor_SMD:C_0402_1005Metric, F.Cu at (172.4, 136.3)
- added C42: DNP, Capacitor_SMD:C_0402_1005Metric, F.Cu at (170.4, 136.8)
- added Card1: SIM-Nano, cacophony-footprints:SIM-Nano, F.Cu at (150.9, 144.9)
- added D101: D_Shockley, Diode_SMD:D_SMA, B.Cu at (97.7, 83.7)
- added D201: D_Shockley, Diode_SMD:D_SMA, B.Cu at (112.5, 67.0)
- added D6: SMF05CT1G, cacophony-footprints:SOT-363_L2.0-W1.3-P0.65-LS2.1-TL, F.Cu at (150.8, 135.9)
- added H1: MountingHole, MountingHole:MountingHole_3.5mm, F.Cu at (161.1, 143.7)
- added H2: MountingHole, MountingHole:MountingHole_3.5mm, F.Cu at (85.0, 143.7)
- added H3: MountingHole, MountingHole:MountingHole_3.5mm, F.Cu at (166.8, 66.8)
- added H4: MountingHole, MountingHole:MountingHole_3.5mm, F.Cu at (91.0, 60.7)
- added J4: Conn_01x05, cacophony-footprints:JST_XA_B05B-XASK-1-A_1x05_P2.50mm_Vertical, B.Cu at (84.7, 111.5)
- added J5: Conn_01x03, Connector_PinHeader_2.54mm:PinHeader_1x03_P2.54mm_Vertical, F.Cu at (163.8, 149.4)
- added J6: Screw_Terminal_01x01, cacophony-footprints:SMD_M2_nut, F.Cu at (149.5, 86.0)
- added J7: Conn_01x02, Connector_PinHeader_1.00mm:PinHeader_1x02_P1.00mm_Vertical, F.Cu at (147.2, 82.2)
- added J8: Conn_01x02, Connector_PinHeader_1.00mm:PinHeader_1x02_P1.00mm_Vertical, B.Cu at (136.0, 105.9)
- added L101: 6.8uF, cacophony-footprints:IND-SMD_L8.0-W8.0_1217AS, B.Cu at (96.0, 77.0)
- added L201: 6.8uF, cacophony-footprints:IND-SMD_L8.0-W8.0_1217AS, B.Cu at (114.2, 73.7)
- added R101: 33k, Resistor_SMD:R_0402_1005Metric, B.Cu at (92.8, 88.3)
- added R102: 22k, Resistor_SMD:R_0402_1005Metric, B.Cu at (91.1, 89.9)
- added R103: 10k, Resistor_SMD:R_0402_1005Metric, B.Cu at (92.2, 89.9)
- added R104: 100k, Resistor_SMD:R_0402_1005Metric, B.Cu at (93.3, 89.9)
- added R16: 100k, Resistor_SMD:R_0402_1005Metric, F.Cu at (162.7, 130.1)
- added R17: 22ohm, Resistor_SMD:R_0402_1005Metric, F.Cu at (148.9, 134.6)
- added R18: 22ohm, Resistor_SMD:R_0402_1005Metric, F.Cu at (147.9, 134.6)
- added R19: 22ohm, Resistor_SMD:R_0402_1005Metric, F.Cu at (146.9, 134.6)
- added R20: 100k, Resistor_SMD:R_0402_1005Metric, B.Cu at (120.2, 101.1)
- added R201: 33k, Resistor_SMD:R_0402_1005Metric, B.Cu at (117.5, 62.4)
- added R202: 150k, Resistor_SMD:R_0402_1005Metric, B.Cu at (119.2, 60.8)
- added R203: 100k, Resistor_SMD:R_0402_1005Metric, B.Cu at (118.0, 60.8)
- added R204: 22k, Resistor_SMD:R_0402_1005Metric, B.Cu at (117.0, 60.8)
- added R21: 100k, Resistor_SMD:R_0402_1005Metric, B.Cu at (123.0, 85.9)
- added R22: 22ohm, Resistor_SMD:R_0402_1005Metric, F.Cu at (132.5, 71.1)
- added R23: 22ohm, Resistor_SMD:R_0402_1005Metric, B.Cu at (135.8, 85.4)
- added R24: 22ohm, Resistor_SMD:R_0402_1005Metric, B.Cu at (135.8, 84.3)
- added R25: 22ohm, Resistor_SMD:R_0402_1005Metric, B.Cu at (136.2, 115.8)
- added R26: 22ohm, Resistor_SMD:R_0402_1005Metric, B.Cu at (147.5, 120.9)
- added R27: 22ohm, Resistor_SMD:R_0402_1005Metric, B.Cu at (125.1, 123.3)
- added R28: 10k, Resistor_SMD:R_0402_1005Metric, B.Cu at (154.8, 83.3)
- added R29: 22ohm, Resistor_SMD:R_0402_1005Metric, B.Cu at (124.7, 90.4)
- added R30: 22ohm, Resistor_SMD:R_0402_1005Metric, B.Cu at (135.5, 101.8)
- added R31: 22ohm, Resistor_SMD:R_0402_1005Metric, B.Cu at (135.6, 95.6)
- added R32: 22ohm, Resistor_SMD:R_0402_1005Metric, B.Cu at (135.5, 100.8)
- added R33: 22ohm, Resistor_SMD:R_0402_1005Metric, B.Cu at (127.8, 90.9)
- added R34: 10k, Resistor_SMD:R_0402_1005Metric, B.Cu at (127.8, 89.8)
- added R35: 0ohm, Resistor_SMD:R_0402_1005Metric, F.Cu at (161.4, 61.0)
- added R36: DNP, Resistor_SMD:R_0402_1005Metric, F.Cu at (138.1, 53.3)
- added R37: DNP, Resistor_SMD:R_0402_1005Metric, F.Cu at (140.6, 53.3)
- added R38: DNP, Resistor_SMD:R_0402_1005Metric, F.Cu at (143.1, 53.3)
- added R39: DNP, Resistor_SMD:R_0402_1005Metric, F.Cu at (145.6, 53.3)
- added R40: 0ohm, Resistor_SMD:R_0402_1005Metric, F.Cu at (176.4, 118.4)
- added R41: 0ohm, Resistor_SMD:R_0402_1005Metric, F.Cu at (176.4, 120.8)
- added R42: 0ohm, Resistor_SMD:R_0402_1005Metric, F.Cu at (176.9, 94.3)
- added R43: 0ohm, Resistor_SMD:R_0402_1005Metric, F.Cu at (174.5, 94.3)
- added RF1: KH-IPEX-4-K501-29, cacophony-footprints:IPEX4-SMD_4P-L1.8-W1.7-LS2.0-L_KH-IPEX4-2020, F.Cu at (155.1, 77.1)
- added RF2: KH-IPEX-4-K501-29, cacophony-footprints:IPEX4-SMD_4P-L1.8-W1.7-LS2.0-L_KH-IPEX4-2020, F.Cu at (177.0, 85.3)
- added RF3: KH-IPEX-4-K501-29, cacophony-footprints:IPEX4-SMD_4P-L1.8-W1.7-LS2.0-L_KH-IPEX4-2020, F.Cu at (161.4, 65.3)
- added RF4: KH-IPEX-4-K501-29, cacophony-footprints:IPEX4-SMD_4P-L1.8-W1.7-LS2.0-L_KH-IPEX4-2020, F.Cu at (168.0, 136.3)
- added TP1: TestPoint, TestPoint:TestPoint_Pad_1.0x1.0mm, B.Cu at (121.5, 94.8)
- added TP10: TestPoint, Connector_PinHeader_1.00mm:PinHeader_1x01_P1.00mm_Vertical, B.Cu at (147.8, 93.0)
- added TP12: TestPoint, TestPoint:TestPoint_Pad_1.0x1.0mm, F.Cu at (110.6, 100.2)
- added TP2: TestPoint, TestPoint:TestPoint_Pad_1.0x1.0mm, B.Cu at (121.5, 92.7)
- added TP3: TestPoint, TestPoint:TestPoint_Pad_1.0x1.0mm, B.Cu at (121.5, 96.9)
- added TP4: TestPoint, TestPoint:TestPoint_Pad_1.0x1.0mm, B.Cu at (121.5, 99.0)
- added TP5: TestPoint, Connector_PinHeader_1.00mm:PinHeader_1x01_P1.00mm_Vertical, F.Cu at (128.2, 93.3)
- added TP6: TestPoint, Connector_PinHeader_1.00mm:PinHeader_1x01_P1.00mm_Vertical, F.Cu at (127.5, 77.9)
- added TP7: TestPoint, Connector_PinHeader_1.00mm:PinHeader_1x01_P1.00mm_Vertical, F.Cu at (127.5, 80.1)
- added TP8: TestPoint, Connector_PinHeader_1.00mm:PinHeader_1x01_P1.00mm_Vertical, F.Cu at (127.5, 75.7)
- added TP9: TestPoint, Connector_PinHeader_1.00mm:PinHeader_1x01_P1.00mm_Vertical, B.Cu at (136.1, 92.0)
- added U101: TPS54331, Package_SO:SO-8_3.9x4.9mm_P1.27mm, B.Cu at (97.6, 88.3)
- added U11: Flir_LEPTON, cacophony-footprints:MOLEX_105028-1001, F.Cu at (107.0, 107.2)
- added U201: TPS54331, Package_SO:SO-8_3.9x4.9mm_P1.27mm, B.Cu at (112.7, 62.4)
- added U6: SPH0645LM4H, SPH0645LM4H-B:MIC_SPH0645LM4H-B, B.Cu at (125.0, 127.2)
- BT1, Q1, R3, U2, U7, U9, Y1: moved to B.Cu
- BZ1: footprint Buzzer_Beeper:MagneticBuzzer_PUI_AT-0927-TT-6-R -> cacophony-footprints:MagneticBuzzer_PUI_AT-0927-TT-6-R
- C1: value 220uF -> 220nF; footprint Capacitor_SMD:CP_Elec_8x10 -> Capacitor_SMD:C_0402_1005Metric
- C10, C19, C9: value 4.7uF -> 10uF; footprint Capacitor_SMD:C_0402_1005Metric -> Capacitor_SMD:C_0603_1608Metric
- C11, C12, C13, C8: value 100nF -> 220nF; moved to B.Cu
- C14: value 100nF -> 220nF
- C2: value 1uF -> 220nF
- C21: value 4.7uF -> 220nF; moved to B.Cu
- C22, C25: footprint Capacitor_SMD:C_0805_2012Metric -> Capacitor_SMD:C_0603_1608Metric
- C23, C24: value 4.7uF -> 22uF; footprint Capacitor_SMD:C_0402_1005Metric -> Capacitor_SMD:C_0603_1608Metric
- C3: value 10nF -> 220nF; moved to B.Cu
- C4: value 100nF -> 10uF
- C5: value 1uF -> 10uF; footprint Capacitor_SMD:C_0402_1005Metric -> Capacitor_SMD:C_0603_1608Metric; moved to B.Cu
- C6: value 1uF -> 3.0pF
- C7: footprint Capacitor_SMD:C_0805_2012Metric -> Capacitor_SMD:C_0603_1608Metric; moved to B.Cu
- D1: footprint Diode_SMD:D_SMA -> cacophony-footprints:LL-34_L3.5-W1.5-RD; moved to B.Cu
- D2: value WS2812B -> LED_RGB; footprint LED_SMD:LED_WS2812B_PLCC4_5.0x5.0mm_P3.2mm -> cacophony-footprints:LED_RGB
- D3, D4: value D_Shockley -> D; footprint Diode_SMD:D_SOD-323 -> Diode_SMD:D_SMA; moved to B.Cu
- J1: footprint Connector_PinSocket_2.54mm:PinSocket_2x20_P2.54mm_Vertical -> cacophony-footprints:RPi_SMD; moved to B.Cu
- J2: value Conn_01x02 -> Screw_Terminal_M2_L10; footprint Connector_JST:JST_XA_S02B-XASK-1_1x02_P2.50mm_Horizontal -> cacophony-footprints:SMD_M2_nut; moved to B.Cu
- J3: value Conn_01x10 -> Screw_Terminal_M2_L10; footprint Connector_PinSocket_2.54mm:PinSocket_1x10_P2.54mm_Vertical -> cacophony-footprints:SMD_M2_nut; moved to B.Cu
- R1: value 100K -> 100k; moved to B.Cu
- R10: value 10K -> 100k
- R11: value 330K -> 10k; moved to B.Cu
- R12: value 68K -> 100k; moved to B.Cu
- R13, R14, R15: value 100K -> 100k
- R2: value 47K -> 180R; footprint Resistor_SMD:R_0402_1005Metric -> Resistor_SMD:R_0603_1608Metric
- R4: value 100k -> 180R
- R5: value 6.8k -> 180R
- R6: value 560k -> 390k; footprint Resistor_SMD:R_0603_1608Metric -> Resistor_SMD:R_0402_1005Metric
- R7: value 68k -> 1M; moved to B.Cu
- R8: value 560k -> 22ohm; footprint Resistor_SMD:R_0603_1608Metric -> Resistor_SMD:R_0402_1005Metric; moved to B.Cu
- R9: footprint Resistor_SMD:R_0603_1608Metric -> Resistor_SMD:R_0402_1005Metric; moved to B.Cu
- U1: value STM32F030C8Tx -> ATtiny1616-M; footprint Package_QFP:LQFP-48_7x7mm_P0.5mm -> Package_DFN_QFN:VQFN-20-1EP_3x3mm_P0.4mm_EP1.7x1.7mm; moved to B.Cu
- U16: footprint RF_Module:Ai-Thinker-Ra-01-LoRa -> cacophony-footprints:Ai-Thinker-Ra-01-LoRa
- U3: value ATtiny85-20P -> SIM7600G-H-M.2; footprint Package_DIP:DIP-8_W7.62mm -> cacophony-footprints:M.2
- U4: value LMR16030S -> ME6211; footprint Package_SO:TI_SO-PowerPAD-8 -> Package_TO_SOT_SMD:SOT-23-5
- U5: value XC6206PxxxMR -> Antenna_1002427; footprint Package_TO_SOT_SMD:SOT-23 -> cacophony-footprints:ANTENNA_1002427_GPS
- U8: value XC6206PxxxMR -> Antenna_1002427; footprint Package_TO_SOT_SMD:SOT-23 -> cacophony-footprints:ANTENNA_1002427_ISM
- moved J3 144.9 mm to (92.9, 125.8), turned to 180 degrees
- moved C6 123.4 mm to (161.8, 59.3), turned to 0 degrees
- moved C1 111.2 mm to (152.9, 73.6)
- moved U5 111.1 mm to (135.4, 54.6)
- moved C22 111.0 mm to (133.7, 126.6), turned to -90 degrees
- moved R13 110.7 mm to (105.0, 119.2), turned to 180 degrees
- moved C2 110.1 mm to (172.0, 88.9)
- moved L2 109.8 mm to (110.3, 117.4)
- moved L3 107.9 mm to (96.2, 110.1), turned to -90 degrees
- moved C21 107.3 mm to (122.8, 125.6), turned to 90 degrees
- moved U14 107.2 mm to (96.8, 105.7), turned to 90 degrees
- moved C18 107.1 mm to (93.5, 106.7), turned to 90 degrees
- moved C17 106.9 mm to (107.0, 119.2), turned to 180 degrees
- moved C19 106.8 mm to (109.4, 114.3), turned to 180 degrees
- moved C4 106.6 mm to (157.6, 73.4), turned to 0 degrees
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Connections:
- net Net-(C18-Pad2) renamed /Lepton/FB_1V2
- net Net-(L2-Pad1) renamed /Lepton/SW_3V0
- net Net-(L3-Pad1) renamed /Lepton/SW_1V2
- BT1 pad 1: Net-(BT1-Pad1) -> RTC_BT_SENSE
- C1 pad 1: Net-(C1-Pad1) -> GND
- C1 pad 2: GND -> +3V3_Lin
- C17 pad 2: Net-(C17-Pad2) -> /Lepton/FB_3V0
- C2 pad 1: Net-(C1-Pad1) -> GND
- C2 pad 2: GND -> +3V3
- C21 pad 1: +3V0 -> GND
- C21 pad 2: GND -> +3V3_Lin
- C22 pad 1: VCC -> +3V3
- C23 pad 1: +3V0 -> +3V3
- C24 pad 1: +3V0 -> +3V3
- C25 pad 1: VCC -> +3V3
- C3 pad 1: Net-(C3-Pad1) -> GND
- C3 pad 2: GND -> +3V3
- C4 pad 1: Net-(C4-Pad1) -> +5V
- C4 pad 2: Net-(C4-Pad2) -> GND
- D1 pad 1: VCC -> +12V
- D2 pad 1: +3V3 -> Net-(D2-Pad1)
- D2 pad 2: unconnected-(D2-Pad2) -> Net-(D2-Pad2)
- D2 pad 3: GND -> Net-(D2-Pad3)
- D2 pad 4: LED -> GND
- D4 pad 2: Net-(BT1-Pad1) -> RTC_BT_SENSE
- J1 pad 10: unconnected-(J1-Pad10) -> Net-(J1-Pad10)
- J1 pad 11: unconnected-(J1-Pad11) -> Net-(J1-Pad11)
- J1 pad 12: unconnected-(J1-Pad12) -> Net-(J1-Pad12)
- J1 pad 13: unconnected-(J1-Pad13) -> Net-(J1-Pad13)
- J1 pad 15: unconnected-(J1-Pad15) -> Net-(J1-Pad15)
- J1 pad 16: unconnected-(J1-Pad16) -> ~{LORA_RESET}
- J1 pad 18: unconnected-(J1-Pad18) -> Net-(J1-Pad18)
- J1 pad 19: unconnected-(J1-Pad19) -> Net-(J1-Pad19)
- J1 pad 2: unconnected-(J1-Pad2) -> +5V
- J1 pad 21: unconnected-(J1-Pad21) -> MISO_0
- J1 pad 22: unconnected-(J1-Pad22) -> BUZZER
- J1 pad 23: unconnected-(J1-Pad23) -> Net-(J1-Pad23)
- J1 pad 24: unconnected-(J1-Pad24) -> Net-(J1-Pad24)
- J1 pad 26: unconnected-(J1-Pad26) -> LEPTON_POWER_EN
- J1 pad 27: unconnected-(J1-Pad27) -> Net-(J1-Pad27)
- J1 pad 28: unconnected-(J1-Pad28) -> Net-(J1-Pad28)
- J1 pad 29: unconnected-(J1-Pad29) -> LEPTON_VSYNC
- J1 pad 3: unconnected-(J1-Pad3) -> SDA
- J1 pad 31: unconnected-(J1-Pad31) -> LEPTON_CLK_EN
- J1 pad 32: unconnected-(J1-Pad32) -> LEPTON_PWR_DWN_L
- J1 pad 33: unconnected-(J1-Pad33) -> LEPTON_RESET_L
- J1 pad 35: unconnected-(J1-Pad35) -> Net-(J1-Pad35)
- J1 pad 36: unconnected-(J1-Pad36) -> 4G_POWER_ON
- J1 pad 37: unconnected-(J1-Pad37) -> ~{W_DISABLE1}
- J1 pad 38: unconnected-(J1-Pad38) -> I2S_DIN/MOSI1
- J1 pad 4: unconnected-(J1-Pad4) -> +5V
- J1 pad 40: unconnected-(J1-Pad40) -> Net-(J1-Pad40)
- J1 pad 5: unconnected-(J1-Pad5) -> SCL
- J1 pad 7: unconnected-(J1-Pad7) -> SPEAKER_SD_MODE
- J1 pad 8: unconnected-(J1-Pad8) -> Net-(J1-Pad8)
- J2 pad 1: GND -> unconnected-(J2-Pad1)
- J3 pad 1: /CS -> unconnected-(J3-Pad1)
- Q1 pad 2: VCC -> +12V
- Q1 pad 3: Net-(J2-Pad2) -> VIN
- R10 pad 1: Net-(R10-Pad1) -> LEPTON_CLK_EN
- R11 pad 1: +3V0 -> +3V3
- R11 pad 2: Net-(R11-Pad2) -> SDA
- R12 pad 1: Net-(C17-Pad2) -> +3V0
- R12 pad 2: Net-(R11-Pad2) -> LEPTON_PWR_DWN_L
- R13 pad 1: Net-(C17-Pad2) -> /Lepton/FB_3V0
- R2 pad 1: Net-(R2-Pad1) -> LED_R
- R2 pad 2: GND -> Net-(D2-Pad1)
- R4 pad 1: Net-(R4-Pad1) -> LED_G
- R4 pad 2: GND -> Net-(D2-Pad2)
- R5 pad 1: Net-(R4-Pad1) -> LED_B
- R5 pad 2: Net-(R5-Pad2) -> Net-(D2-Pad3)
- R6 pad 1: Net-(R5-Pad2) -> +3V0
- R6 pad 2: Net-(C6-Pad1) -> /Lepton/FB_3V0
- R7 pad 1: +5V -> SPEAKER_SD_MODE
- R8 pad 1: Net-(R7-Pad2) -> MISO_0
- U1 pad 1: unconnected-(U1-Pad1) -> Net-(R29-Pad1)
- U1 pad 10: unconnected-(U1-Pad10) -> BATT_SENSE
- U1 pad 11: unconnected-(U1-Pad11) -> Net-(TP7-Pad1)
- U1 pad 12: unconnected-(U1-Pad12) -> Net-(TP6-Pad1)
- U1 pad 13: unconnected-(U1-Pad13) -> SDA
- U1 pad 14: unconnected-(U1-Pad14) -> SCL
- U1 pad 15: unconnected-(U1-Pad15) -> ~{RTC_INT}
- U1 pad 16: unconnected-(U1-Pad16) -> RTC_BT_SENSE
- U1 pad 17: unconnected-(U1-Pad17) -> RTC_BT_LOAD
- U1 pad 18: unconnected-(U1-Pad18) -> Net-(TP5-Pad1)
- U1 pad 19: unconnected-(U1-Pad19) -> ATtiny_RESET
- U1 pad 2: unconnected-(U1-Pad2) -> SCLK_0
- U1 pad 20: unconnected-(U1-Pad20) -> MOSI_0
- U1 pad 21: unconnected-(U1-Pad21) -> GND
- U1 pad 3: unconnected-(U1-Pad3) -> GND
- U1 pad 4: unconnected-(U1-Pad4) -> +3V3
- U1 pad 5: unconnected-(U1-Pad5) -> 5V_EN
- U1 pad 6: unconnected-(U1-Pad6) -> LED_R
- U1 pad 7: unconnected-(U1-Pad7) -> LED_G
- U1 pad 8: unconnected-(U1-Pad8) -> LED_B
- U1 pad 9: unconnected-(U1-Pad9) -> Net-(TP8-Pad1)
- U12 pad 1: Net-(R10-Pad1) -> LEPTON_CLK_EN
- U12 pad 3: /MASTER_CLK -> /Lepton/MASTER_CLK
- U13 pad 1: /Enable -> LEPTON_POWER_EN
- U13 pad 5: Net-(C17-Pad2) -> /Lepton/FB_3V0
- U14 pad 1: /Enable -> LEPTON_POWER_EN
- U16 pad 1: unconnected-(U16-Pad1) -> Net-(RF1-Pad1)
- U16 pad 12: unconnected-(U16-Pad12) -> I2S_DOUT/SCLK1
- U16 pad 13: unconnected-(U16-Pad13) -> Net-(R22-Pad2)
- U16 pad 14: unconnected-(U16-Pad14) -> I2S_DIN/MOSI1
- U16 pad 15: unconnected-(U16-Pad15) -> LORA_CS
- U16 pad 16: Net-(U16-Pad16) -> GND
- U16 pad 2: Net-(U16-Pad16) -> GND
- U16 pad 3: unconnected-(U16-Pad3) -> +3V3_Lin
- U16 pad 4: unconnected-(U16-Pad4) -> ~{LORA_RESET}
- U16 pad 9: Net-(U16-Pad16) -> GND
- U3 pad 2: unconnected-(U3-Pad2) -> +3V3
- U3 pad 3: unconnected-(U3-Pad3) -> GND
- U3 pad 4: GND -> +3V3
- U3 pad 5: unconnected-(U3-Pad5) -> GND
- U3 pad 6: unconnected-(U3-Pad6) -> 4G_POWER_ON
- U3 pad 7: unconnected-(U3-Pad7) -> 4G_USB_D+
- U3 pad 8: +3V3 -> ~{W_DISABLE1}
- U4 pad 1: Net-(C4-Pad1) -> +5V
- U4 pad 2: Net-(C1-Pad1) -> GND
- U4 pad 3: Net-(C1-Pad1) -> +5V
- U4 pad 4: Net-(R2-Pad1) -> unconnected-(U4-Pad4)
- U4 pad 5: Net-(R4-Pad1) -> +3V3_Lin
- U5 pad 1: GND -> Net-(C6-Pad1)
- U5 pad 2: Net-(U5-Pad2) -> GND
- U5 pad 3: +5V -> Net-(R36-Pad1)
- U8 pad 1: GND -> Net-(C40-Pad1)
- U8 pad 2: +3V3 -> GND
- U8 pad 3: Net-(C6-Pad1) -> Net-(R40-Pad1)
- U9 pad 1: I2S_DOUT -> I2S_DOUT/SCLK1
- U9 pad 10: Net-(LS1-Pad1) -> SPEAKER_-
- U9 pad 14: I2S_LRCLK -> I2S_LRCLK/MISO1
- U9 pad 4: Net-(R8-Pad2) -> Net-(R7-Pad2)
- U9 pad 9: Net-(LS1-Pad2) -> SPEAKER_+
Routing:
- net GND: track 0.00 -> 148.6 mm, vias 0 -> 140
- net SDA: track 0.00 -> 116.9 mm, vias 0 -> 2
- net SCL: track 0.00 -> 115.8 mm, vias 0 -> 4
- net +3V3_Lin: track 0.00 -> 102.8 mm, vias 0 -> 1
- net I2S_DOUT/SCLK1: track 0.00 -> 83.8 mm, vias 0 -> 2
- net I2S_LRCLK/MISO1: track 0.00 -> 83.2 mm, vias 0 -> 4
- net I2S_BCLK: track 0.00 -> 78.3 mm, vias 0 -> 5
- net SPEAKER_+: track 0.00 -> 76.9 mm
- net SPEAKER_-: track 0.00 -> 75.1 mm
- net I2S_DIN/MOSI1: track 0.00 -> 73.8 mm, vias 0 -> 3
- net LEPTON_POWER_EN: track 0.00 -> 66.4 mm, vias 0 -> 2
- net BATT_SENSE: track 0.00 -> 66.3 mm, vias 0 -> 2
- net LEPTON_VSYNC: track 0.00 -> 55.4 mm, vias 0 -> 3
- net MOSI_0: track 0.00 -> 55.0 mm, vias 0 -> 3
- net LEPTON_PWR_DWN_L: track 0.00 -> 55.0 mm, vias 0 -> 3
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- added copper zone on B.Cu, net (none)
- added copper zone on F.Cu, net (none)
- added copper zone on B.Cu, net +12V
- added copper zone on F.Cu, net +1V2
- added copper zone on F.Cu, net +3V0
- added copper zone on B.Cu, net +3V3
- added copper zone on In2.Cu, net +3V3
- added copper zone on B.Cu, net +5V
- added copper zone on F.Cu, net +5V
- added copper zone on In2.Cu, net +5V
- added copper zone on F.Cu, net /Lepton/SW_1V2
- added copper zone on F.Cu, net /Lepton/SW_3V0
- added copper zone on B.Cu, net /Power/SW_3V3
- added copper zone on B.Cu, net /Power/SW_5V
- added copper zone on B.Cu, net GND
- added copper zone on F.Cu, net GND
- added copper zone on In1.Cu, net GND
- added copper zone on B.Cu, net VIN
Other:
- outline, holes or cut-outs redrawn
- copper layers 2 -> 4
- board text added: "JLCJLCJLCJLC"

Commit message: WIP
Parts:
- moved R22 0.30 mm to (132.8, 71.1)
Routing:
- net +3V3: track 41.5 -> 250.6 mm, vias 35 -> 25
- net +5V: track 27.1 -> 173.0 mm, vias 34 -> 19
- net I2S_LRCLK/MISO1: track 83.2 -> 83.8 mm, vias 4 -> 3
- net SDA: track 116.9 -> 116.4 mm
- net SPEAKER_SD_MODE: track 33.3 -> 33.8 mm
- net I2S_DOUT/SCLK1: track 83.8 -> 84.2 mm, vias 2 -> 4
- net GND: vias 140 -> 139
- added copper zone on F.Cu, net +3V3
- added copper zone on In2.Cu, net GND
- removed copper zone on In2.Cu, net +3V3
- removed copper zone on In2.Cu, net +5V

Commit message: WIP
Parts:
- removed AE1: Antenna, cacophony-footprints:ANT-8_9-PW-LPN
- removed C101, C201: 220uF, Capacitor_SMD:CP_Elec_8x10
- removed C102, C103, C202, C203, C35, C36: 22uF, Capacitor_SMD:C_0805_2012Metric
- removed C104, C105, C109, C204, C205, C209: 1nF, Capacitor_SMD:C_0402_1005Metric
- removed C106, C206: 47pF, Capacitor_SMD:C_0402_1005Metric
- removed C107, C207: 10nF, Capacitor_SMD:C_0402_1005Metric
- removed C108, C208: 100nF, Capacitor_SMD:C_0402_1005Metric
- removed C110, C111, C30, C31, C32, C33: 22uF, Capacitor_SMD:C_0603_1608Metric
- removed C34: 10uF, Capacitor_SMD:C_0603_1608Metric
- removed C39, C42: DNP, Capacitor_SMD:C_0402_1005Metric
- removed C40: 1.8pF, Capacitor_SMD:C_0402_1005Metric
- removed C41: 5.6pF, Capacitor_SMD:C_0402_1005Metric
- removed D101, D201: D_Shockley, Diode_SMD:D_SMA
- removed H1: MountingHole, MountingHole:MountingHole_3.5mm
- removed J7, J8: Conn_01x02, Connector_PinHeader_1.00mm:PinHeader_1x02_P1.00mm_Vertical
- removed L101, L201: 6.8uF, cacophony-footprints:IND-SMD_L8.0-W8.0_1217AS
- removed Q1: Q_PMOS_GSD, Package_TO_SOT_SMD:SOT-23
- removed R101, R201: 33k, Resistor_SMD:R_0402_1005Metric
- removed R102, R204: 22k, Resistor_SMD:R_0402_1005Metric
- removed R103: 10k, Resistor_SMD:R_0402_1005Metric
- removed R104, R203: 100k, Resistor_SMD:R_0402_1005Metric
- removed R202: 150k, Resistor_SMD:R_0402_1005Metric
- removed R29: 22ohm, Resistor_SMD:R_0402_1005Metric
- removed R40, R41, R42, R43: 0ohm, Resistor_SMD:R_0402_1005Metric
- removed RF2, RF4: KH-IPEX-4-K501-29, cacophony-footprints:IPEX4-SMD_4P-L1.8-W1.7-LS2.0-L_KH-IPEX4-2020
- removed U101, U201: TPS54331, Package_SO:SO-8_3.9x4.9mm_P1.27mm
- removed U11: Flir_LEPTON, cacophony-footprints:MOLEX_105028-1001
- added D5: D, Diode_SMD:D_SOD-523, F.Cu at (162.8, 137.1)
- added TP11: TestPoint, cacophony-library:TP, F.Cu at (175.8, 100.8)
- added TP13: TestPoint, cacophony-library:TP, F.Cu at (182.0, 98.3)
- added TP14: TestPoint, cacophony-library:TP, F.Cu at (167.9, 98.2)
- added TP15: TestPoint, cacophony-library:TP, F.Cu at (163.0, 98.2)
- added TP16: TestPoint, cacophony-library:TP, F.Cu at (165.4, 98.2)
- BT1, C37, C38, C5, C7, C8, R11, R20, R23, R24, R25, R26, R28, R30, R31, R32, R7, R8, R9, U2, U7, Y1: moved to F.Cu
- BZ1: footprint cacophony-footprints:MagneticBuzzer_PUI_AT-0927-TT-6-R -> cacophony-footprints:BUZ-TH_BD9.0-P5.00-D0.6-FD; moved to B.Cu
- C22, C23, C24, C25, C26, C27, Card1, D6, R17, R18, R19, U3: moved to B.Cu
- C28: value 22uF -> 3.0pF; footprint Capacitor_SMD:C_0603_1608Metric -> Capacitor_SMD:C_0402_1005Metric; moved to F.Cu
- C29: value 22uF -> DNP; footprint Capacitor_SMD:C_0603_1608Metric -> Capacitor_SMD:C_0402_1005Metric; moved to F.Cu
- C6: value 3.0pF -> 10uF; footprint Capacitor_SMD:C_0402_1005Metric -> Capacitor_SMD:C_0603_1608Metric
- D1: value D_Zener -> D; footprint cacophony-footprints:LL-34_L3.5-W1.5-RD -> Diode_SMD:D_SOD-523; moved to F.Cu
- D2: footprint cacophony-footprints:LED_RGB -> cacophony-library:LED-SMD_6PIN-L1.60-W1.50-BL-RD
- D3, D4: footprint Diode_SMD:D_SMA -> Diode_SMD:D_SOD-523; moved to F.Cu
- H2, H3, H4: footprint MountingHole:MountingHole_3.5mm -> cacophony-library:Mouning_Hole_M3
- J1: footprint cacophony-footprints:RPi_SMD -> cacophony-footprints:RPi_2_W_SMD
- J2, J3: footprint cacophony-footprints:SMD_M2_nut -> cacophony-library:SMD_NUT_D5.6-HD3.6-L10.0
- J4: value Conn_01x05 -> Conn_02x04_Odd_Even; footprint cacophony-footprints:JST_XA_B05B-XASK-1-A_1x05_P2.50mm_Vertical -> cacophony-library:power-pcb; moved to F.Cu
- J6: footprint cacophony-footprints:SMD_M2_nut -> cacophony-library:SMD_BD4.4-L4.4-D2.8; moved to B.Cu
- L2, L3: footprint Inductor_SMD:L_Taiyo-Yuden_NR-40xx -> cacophony-library:IND-SMD_L4.0-W4.0_SWPA4018S
- R1: value 100k -> 1k; moved to F.Cu
- R2, R4, R5: footprint Resistor_SMD:R_0603_1608Metric -> Resistor_SMD:R_0402_1005Metric; moved to B.Cu
- R3: footprint Resistor_SMD:R_0603_1608Metric -> Resistor_SMD:R_0402_1005Metric; moved to F.Cu
- TP1, TP2, TP3, TP4: footprint TestPoint:TestPoint_Pad_1.0x1.0mm -> cacophony-library:TP; moved to F.Cu
- TP10, TP9: footprint Connector_PinHeader_1.00mm:PinHeader_1x01_P1.00mm_Vertical -> cacophony-library:TP; moved to F.Cu
- TP12: footprint TestPoint:TestPoint_Pad_1.0x1.0mm -> cacophony-library:TP
- TP5, TP6, TP7, TP8: footprint Connector_PinHeader_1.00mm:PinHeader_1x01_P1.00mm_Vertical -> cacophony-library:TP
- U12: footprint Oscillator:Oscillator_SMD_Abracon_ASE-4Pin_3.2x2.5mm -> cacophony-library:OSC-SMD_4P-L3.2-W2.5-BL
- U16: footprint cacophony-footprints:Ai-Thinker-Ra-01-LoRa -> cacophony-library:WIRELM-SMD_RA-01H
- U5: value Antenna_1002427 -> Flir_LEPTON; footprint cacophony-footprints:ANTENNA_1002427_GPS -> cacophony-footprints:MOLEX_105028-1001
- U8: footprint cacophony-footprints:ANTENNA_1002427_ISM -> cacophony-footprints:ANTENNA_1002427_GPS
- U9: footprint Package_DFN_QFN:TQFN-16-1EP_3x3mm_P0.5mm_EP1.23x1.23mm -> Package_DFN_QFN:TQFN-16-1EP_3x3mm_P0.5mm_EP1.6x1.6mm; moved to F.Cu
- moved U8 90.8 mm to (109.4, 54.5), turned to 0 degrees
- moved C6 87.4 mm to (109.9, 129.6)
- moved D1 87.3 mm to (162.8, 135.1)
- moved H2 84.4 mm to (104.0, 61.5)
- moved U15 76.4 mm to (102.3, 53.3)
- moved C2 76.4 mm to (104.4, 53.3)
- moved R1 76.3 mm to (155.7, 76.8), turned to 0 degrees
- moved J3 75.8 mm to (141.9, 68.0), turned to -90 degrees
- moved J5 75.5 mm to (102.7, 105.1), turned to 0 degrees
- moved TP12 74.0 mm to (184.4, 106.1)
- moved U4 73.8 mm to (110.5, 127.1), turned to 180 degrees
- moved C4 69.7 mm to (113.4, 127.3), turned to 90 degrees
- moved U9 66.5 mm to (133.1, 127.3), turned to -90 degrees
- moved R9 65.2 mm to (134.8, 124.4), turned to 0 degrees
- moved C8 64.1 mm to (130.4, 127.8), turned to -90 degrees
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Connections:
- C28 pad 1: +5V -> Net-(C28-Pad1)
- C29 pad 1: +5V -> Net-(C29-Pad1)
- C6 pad 1: Net-(C6-Pad1) -> +3V3_Lin
- D1 pad 1: +12V -> Net-(D1-Pad1)
- D1 pad 2: Net-(D1-Pad2) -> PI_BUZZER
- J1 pad 10: Net-(J1-Pad10) -> ATtiny_RESET
- J4 pad 1: GND -> /Speaker+
- J4 pad 2: VIN -> GND
- J4 pad 3: SPEAKER_- -> /Speaker-
- J4 pad 4: SPEAKER_+ -> +5V
- J4 pad 5: BATT_SENSE -> 5V_EN
- R1 pad 1: Net-(D1-Pad2) -> ATtiny_RESET
- R1 pad 2: GND -> Net-(J1-Pad8)
- R2 pad 1: LED_R -> LED_G
- R3 pad 1: BUZZER -> Net-(D1-Pad1)
- R33 pad 1: ATtiny_RESET -> unconnected-(R33-Pad1)
- R35 pad 1: Net-(C6-Pad1) -> Net-(C28-Pad1)
- R35 pad 2: Net-(C39-Pad1) -> Net-(C29-Pad1)
- R4 pad 1: LED_G -> LED_R
- RF3 pad 1: Net-(C39-Pad1) -> Net-(C29-Pad1)
- U1 pad 19: ATtiny_RESET -> ATtiny_RESET_UPDI
- U1 pad 2: SCLK_0 -> Net-(TP16-Pad1)
- U1 pad 20: MOSI_0 -> Net-(TP14-Pad1)
- U1 pad 6: LED_R -> LED_G
- U1 pad 7: LED_G -> LED_R
- U5 pad 1: Net-(C6-Pad1) -> GND
- U5 pad 2: GND -> LEPTON_VSYNC
- U5 pad 3: Net-(R36-Pad1) -> unconnected-(U5-Pad3)
- U5 pad 4: Net-(R36-Pad2) -> unconnected-(U5-Pad4)
- U5 pad 5: Net-(R37-Pad2) -> unconnected-(U5-Pad5)
- U5 pad 6: Net-(R38-Pad2) -> GND
- U5 pad 7: Net-(R39-Pad2) -> +1V2
- U8 pad 1: Net-(C40-Pad1) -> Net-(C28-Pad1)
- U8 pad 3: Net-(R40-Pad1) -> Net-(R36-Pad1)
- U8 pad 4: Net-(R40-Pad2) -> Net-(R36-Pad2)
- U8 pad 5: Net-(R41-Pad2) -> Net-(R37-Pad2)
- U8 pad 6: Net-(R42-Pad2) -> Net-(R38-Pad2)
- U8 pad 7: Net-(R43-Pad2) -> Net-(R39-Pad2)
Routing:
- net +3V3: track 250.6 -> 2.02 mm, vias 25 -> 0
- net +5V: track 173.0 -> 0.00 mm, vias 19 -> 0
- net GND: track 148.6 -> 2.02 mm, vias 139 -> 0
- net SDA: track 116.4 -> 0.00 mm, vias 2 -> 0
- net SCL: track 115.8 -> 0.00 mm, vias 4 -> 0
- net +3V3_Lin: track 102.8 -> 0.00 mm, vias 1 -> 0
- net I2S_DOUT/SCLK1: track 84.2 -> 0.00 mm, vias 4 -> 0
- net I2S_LRCLK/MISO1: track 83.8 -> 0.00 mm, vias 3 -> 0
- net I2S_BCLK: track 78.3 -> 0.00 mm, vias 5 -> 0
- net SPEAKER_+: track 76.9 -> 0.00 mm
- net SPEAKER_-: track 75.1 -> 0.00 mm
- net I2S_DIN/MOSI1: track 73.8 -> 0.00 mm, vias 3 -> 0
- net LEPTON_POWER_EN: track 66.4 -> 0.00 mm, vias 2 -> 0
- net BATT_SENSE: track 66.3 -> 0.00 mm, vias 2 -> 0
- net LEPTON_VSYNC: track 55.4 -> 0.00 mm, vias 3 -> 0
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- removed copper zone on B.Cu, net (none)
- removed copper zone on F.Cu, net (none)
- removed copper zone on B.Cu, net +12V
- removed copper zone on B.Cu, net +3V3
- removed copper zone on F.Cu, net +3V3
- removed copper zone on B.Cu, net +5V
- removed copper zone on B.Cu, net /Power/SW_3V3
- removed copper zone on B.Cu, net /Power/SW_5V
- removed copper zone on B.Cu, net GND
- removed copper zone on B.Cu, net VIN
Other:
- board size 100 x 100 mm -> 46.3 x 84.7 mm
- board text removed: "JLCJLCJLCJLC"

Commit message: WIP 2
Parts:
- removed R33: 22ohm, Resistor_SMD:R_0402_1005Metric
- removed TP16: TestPoint, cacophony-library:TP
- C3, R12, R2, R21, R34, R4, R5, U1: moved to F.Cu
- R16, R25, R8, RF1, TP11, TP2, TP3, TP4: moved to B.Cu
- TP10, TP13, TP5, TP6, TP7, TP8, TP9: footprint cacophony-library:TP -> cacophony-library:TP_PAD; moved to B.Cu
- TP15: footprint cacophony-library:TP -> cacophony-library:TP_PAD
- moved D3 67.5 mm to (144.4, 126.6)
- moved D4 67.1 mm to (144.4, 128.1), turned to 180 degrees
- moved R16 66.2 mm to (112.7, 101.0), turned to -90 degrees
- moved C5 65.8 mm to (144.4, 129.7), turned to 0 degrees
- moved C38 65.1 mm to (146.1, 125.4), turned to 0 degrees
- moved U2 63.9 mm to (144.9, 123.3)
- moved TP5 62.6 mm to (133.3, 130.1), turned to 180 degrees
- moved U7 62.0 mm to (140.2, 126.7), turned to -90 degrees
- moved TP2 59.4 mm to (118.2, 79.0), turned to 180 degrees
- moved TP9 58.2 mm to (137.5, 130.1), turned to 180 degrees
- moved TP6 57.5 mm to (134.7, 130.1), turned to 180 degrees
- moved TP8 57.1 mm to (138.9, 130.1), turned to 180 degrees
- moved Y1 55.8 mm to (140.8, 121.8), turned to 180 degrees
- moved TP3 55.8 mm to (120.7, 79.0), turned to 180 degrees
- moved R22 55.3 mm to (119.5, 102.9)
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Connections:
- Card1 pad C2: Net-(Card1-PadC2) -> Net-(R19-Pad2)
- Card1 pad C7: Net-(Card1-PadC7) -> Net-(R17-Pad2)
- D6 pad 4: Net-(Card1-PadC7) -> Net-(R19-Pad2)
- D6 pad 6: Net-(Card1-PadC2) -> Net-(R17-Pad2)
- J1 pad 10: ATtiny_RESET -> ATtiny_RESET_UPDI
- J1 pad 13: Net-(J1-Pad13) -> LEPTON_CLK_EN
- J1 pad 15: Net-(J1-Pad15) -> LEPTON_PWR_DWN_L
- J1 pad 16: ~{LORA_RESET} -> LEPTON_RESET_L
- J1 pad 18: Net-(J1-Pad18) -> LEPTON_VSYNC
- J1 pad 22: BUZZER -> LEPTON_POWER_EN
- J1 pad 26: LEPTON_POWER_EN -> unconnected-(J1-Pad26)
- J1 pad 29: LEPTON_VSYNC -> unconnected-(J1-Pad29)
- J1 pad 31: LEPTON_CLK_EN -> unconnected-(J1-Pad31)
- J1 pad 32: LEPTON_PWR_DWN_L -> ~{W_DISABLE1}
- J1 pad 33: LEPTON_RESET_L -> ~{LORA_RESET}
- J1 pad 37: ~{W_DISABLE1} -> PI_BUZZER
- J4 pad 1: /Speaker+ -> BATT_SENSE
- J4 pad 3: /Speaker- -> 5V_EN
- J4 pad 4: +5V -> +3V3
- J4 pad 5: 5V_EN -> SPEAKER_-
- J4 pad 6: +3V3 -> +5V
- J4 pad 7: /Batt_sense -> SPEAKER_+
- R1 pad 1: ATtiny_RESET -> ATtiny_RESET_UPDI
- R17 pad 1: Net-(R17-Pad1) -> Net-(U3-Pad34)
- R17 pad 2: Net-(Card1-PadC2) -> Net-(R17-Pad2)
- R19 pad 1: Net-(R19-Pad1) -> Net-(U3-Pad30)
- R19 pad 2: Net-(Card1-PadC7) -> Net-(R19-Pad2)
- R2 pad 1: LED_G -> LED_B
- R2 pad 2: Net-(D2-Pad1) -> Net-(D2-Pad3)
- R5 pad 1: LED_B -> LED_G
- R5 pad 2: Net-(D2-Pad3) -> Net-(D2-Pad1)
- TP10 pad 1: Net-(J1-Pad18) -> Net-(U1-Pad9)
- TP12 pad 1: /Lepton/MASTER_CLK -> Net-(J1-Pad28)
- TP13 pad 1: Net-(J1-Pad28) -> Net-(U2-Pad6)
- TP14 pad 1: Net-(TP14-Pad1) -> /Lepton/MASTER_CLK
- TP15 pad 1: Net-(TP15-Pad1) -> Net-(U2-Pad3)
- TP5 pad 1: Net-(TP5-Pad1) -> Net-(U1-Pad7)
- TP6 pad 1: Net-(TP6-Pad1) -> Net-(U1-Pad8)
- TP7 pad 1: Net-(TP7-Pad1) -> Net-(U1-Pad12)
- TP8 pad 1: Net-(TP8-Pad1) -> Net-(U1-Pad11)
- TP9 pad 1: Net-(J1-Pad15) -> Net-(U1-Pad10)
- U1 pad 1: Net-(TP15-Pad1) -> LED_G
- U1 pad 10: BATT_SENSE -> Net-(U1-Pad10)
- U1 pad 11: Net-(TP7-Pad1) -> Net-(U1-Pad11)
- U1 pad 12: Net-(TP6-Pad1) -> Net-(U1-Pad12)
- U1 pad 18: Net-(TP5-Pad1) -> LED_B
- U1 pad 2: Net-(TP16-Pad1) -> ATTiny_BUZZER
- U1 pad 20: Net-(TP14-Pad1) -> LED_R
- U1 pad 6: LED_G -> BATT_SENSE
- U1 pad 7: LED_R -> Net-(U1-Pad7)
- U1 pad 8: LED_B -> Net-(U1-Pad8)
- U1 pad 9: Net-(TP8-Pad1) -> Net-(U1-Pad9)
- U2 pad 3: unconnected-(U2-Pad3) -> Net-(U2-Pad3)
- U2 pad 6: unconnected-(U2-Pad6) -> Net-(U2-Pad6)
- U3 pad 30: Net-(R17-Pad1) -> Net-(U3-Pad30)
- U3 pad 34: Net-(R19-Pad1) -> Net-(U3-Pad34)
Routing:
- net SDA: track 0.00 -> 124.9 mm, vias 0 -> 5
- net SCL: track 0.00 -> 121.0 mm, vias 0 -> 9
- net GND: track 2.02 -> 105.5 mm, vias 0 -> 86
- net +3V3: track 2.02 -> 97.6 mm, vias 0 -> 25
- net Net-(D2-Pad3): track 0.00 -> 74.9 mm
- net I2S_BCLK: track 0.00 -> 74.5 mm, vias 0 -> 2
- net Net-(D2-Pad2): track 0.00 -> 74.3 mm
- net Net-(D2-Pad1): track 0.00 -> 73.8 mm
- net SPEAKER_SD_MODE: track 0.00 -> 69.7 mm, vias 0 -> 3
- net I2S_DIN/MOSI1: track 0.00 -> 68.5 mm, vias 0 -> 2
- net I2S_LRCLK/MISO1: track 0.00 -> 61.1 mm, vias 0 -> 3
- net ATtiny_RESET_UPDI: track 0.00 -> 59.9 mm, vias 0 -> 3
- net I2S_DOUT/SCLK1: track 0.00 -> 51.1 mm, vias 0 -> 3
- net LEPTON_POWER_EN: track 0.00 -> 49.7 mm, vias 0 -> 4
- net +3V3_Lin: track 0.00 -> 46.0 mm, vias 0 -> 1
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- added copper zone on B.Cu, net +3V3
- added copper zone on F.Cu, net +3V3
- added copper zone on B.Cu, net +5V
- added copper zone on B.Cu, net GND

Commit message: WIP
Changed lines of the file:
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@@
     (pad "32" smd rect (at -3.15 -4.31) (size 0.5 0.84) (layers "F.Cu" "F.Paste" "F.Mask")
       (net 133 "unconnected-(U5-Pad32)") (pinfunction "MIPI_DATA_P") (pintype "output+no_connect"))
+    (model "/home/cam/Downloads/105028-1001.stp"
+      (offset (xyz 0 0 2.1))
+      (scale (xyz 1 1 1))
+      (rotate (xyz -90 0 0))
+    )
   )
   (footprint "cacophony-library:TP" (layer "F.Cu")
@@
       (options (clearance outline) (anchor circle))
       (primitives
-    (gr_arc (start 1.238687 2.158493) (mid 0.331674 1.24433) (end 0 0) (width 1.2))
+    (gr_arc (start 1.238687 2.158493) (mid 0.332763 1.246221) (end 0.000008 0.004362) (width 1.2))
       ))
     (pad "1" smd custom (at 0 -2.5 180) (size 0.1 0.1) (layers "B.Cu" "B.Paste" "B.Mask")
@@
       (options (clearance outline) (anchor circle))
       (primitives
-    (gr_arc (start 1.234921 2.156287) (mid 0.330589 1.242437) (end 0 0) (width 1.2))
+    (gr_arc (start 1.234921 2.156287) (mid 0.332763 1.246219) (end 0.00002 0.008724) (width 1.2))
       ))
     (pad "1" smd custom (at 0 2.5) (size 0.1 0.1) (layers "B.Cu" "B.Paste" "B.Mask")
@@
       (options (clearance outline) (anchor circle))
       (primitives
-    (gr_arc (start 1.238686 2.158492) (mid 0.331673 1.24433) (end 0 0) (width 1.2))
+    (gr_arc (start 1.238686 2.158492) (mid 0.332761 1.246224) (end 0.000004 0.004369) (width 1.2))
       ))
     (pad "1" smd circle (at 0 0 270) (size 6.2 6.2) (layers "B.Cu" "B.Mask")
@@
       (options (clearance outline) (anchor circle))
       (primitives
-    (gr_arc (start 1.234922 2.156288) (mid 0.330589 1.242438) (end 0 0) (width 1.2))
+    (gr_arc (start 1.234922 2.156288) (mid 0.33059 1.242441) (end 0 0.000007) (width 1.2))
       ))
     (pad "1" thru_hole circle (at 0 0 270) (size 3.8 3.8) (drill 3.6) (layers *.Cu *.Mask)
@@
       (rotate (xyz 0 0 0))
     )
-    (model "${CAC_KICAD_LIBRARY}/cacophony-library.3dshapes/RaspberryPi3B.step"
+    (model "${CAC_KICAD_LIBRARY}/cacophony-library.3dshapes/RaspberryPi3B.step" hide
       (offset (xyz 0 0 26))
       (scale (xyz 1 1 1))
@@
       (options (clearance outline) (anchor circle))
       (primitives
-    (gr_arc (start 1.238686 2.158492) (mid 0.331673 1.24433) (end 0 0) (width 1.2))
+    (gr_arc (start 1.238686 2.158492) (mid 0.332761 1.246224) (end 0.000004 0.004369) (width 1.2))
       ))
     (pad "1" smd custom (at -2.5 0 270) (size 0.1 0.1) (layers "B.Cu" "B.Paste" "B.Mask")
@@
       (options (clearance outline) (anchor circle))
       (primitives
-    (gr_arc (start 1.238687 2.158493) (mid 0.331674 1.24433) (end 0 0) (width 1.2))
+    (gr_arc (start 1.238687 2.158493) (mid 0.332763 1.246221) (end 0.000008 0.004362) (width 1.2))
       ))
     (pad "1" smd custom (at 0 -2.5 180) (size 0.1 0.1) (layers "B.Cu" "B.Paste" "B.Mask")
@@
       (options (clearance outline) (anchor circle))
       (primitives
-    (gr_arc (start 1.234921 2.156287) (mid 0.330589 1.242437) (end 0 0) (width 1.2))
+    (gr_arc (start 1.234921 2.156287) (mid 0.332763 1.246219) (end 0.00002 0.008724) (width 1.2))
       ))
     (pad "1" thru_hole circle (at 0 0 270) (size 3.8 3.8) (drill 3.6) (layers *.Cu *.Mask)
@@
       (options (clearance outline) (anchor circle))
       (primitives
-    (gr_arc (start 1.234922 2.156288) (mid 0.330589 1.242438) (end 0 0) (width 1.2))
+    (gr_arc (start 1.234922 2.156288) (mid 0.33059 1.242441) (end 0 0.000007) (width 1.2))
       ))
     (model "${CAC_KICAD_LIBRARY}/cacophony-library.3dshapes/SMD_BD4.4-L4.4-D2.8.wrl"
@@
   (gr_arc (start 130.8 135.4) (mid 130.507107 136.107107) (end 129.8 136.4) (layer "Edge.Cuts") (width 0.1))
   (gr_arc (start 147.1 130.4) (mid 146.807107 131.107107) (end 146.1 131.4) (layer "Edge.Cuts") (width 0.1))
+  (dimension (type aligned) (layer "User.2")
+    (pts (xy 144 61.5) (xy 104 61.5))
+    (height 22.95)
+    (gr_text "40.0000 mm" (at 124 37.4) (layer "User.2")
+      (effects (font (size 1 1) (thickness 0.15)))
+    )
+    (format (units 3) (units_format 1) (precision 4))
+    (style (thickness 0.15) (arrow_length 1.27) (text_position_mode 0) (extension_height 0.58642) (extension_offset 0.5) keep_text_aligned)
+  )
+  (dimension (type aligned) (layer "User.2")
+    (pts (xy 104 61.5) (xy 104 107))
+    (height 21.299999)
+    (gr_text "45.5000 mm" (at 81.550001 84.25 90) (layer "User.2")
+      (effects (font (size 1 1) (thickness 0.15)))
+    )
+    (format (units 3) (units_format 1) (precision 4))
+    (style (thickness 0.15) (arrow_length 1.27) (text_position_mode 0) (extension_height 0.58642) (extension_offset 0.5) keep_text_aligned)
+  )
   (dimension (type orthogonal) (layer "User.2")
     (pts (xy 100.8 52.7) (xy 147.1 52.7))
