File: SIM7600G_M.2.kicad_sch (KiCad schematic)
At the start: 15 parts, among them J5 Conn_01x03, J6 Screw_Terminal_01x01, U3 SIM7600G-H-M.2

Commit message: WIP
Parts:
- added C28: 3.0pF, Capacitor_SMD:C_0402_1005Metric, symbol Device:C_Small
- added C29: DNP, Capacitor_SMD:C_0402_1005Metric, symbol Device:C_Small
- added R35: 0ohm, Resistor_SMD:R_0402_1005Metric, symbol Device:R
- added R36, R37, R38, R39: DNP, Resistor_SMD:R_0402_1005Metric, symbol Device:R
- added RF3: KH-IPEX-4-K501-29, cacophony-footprints:IPEX4-SMD_4P-L1.8-W1.7-LS2.0-L_KH-IPEX4-2020, symbol cacophony-symbols:KH-IPEX-4-K501-29
- added U8: Antenna_1002427, cacophony-footprints:ANTENNA_1002427_GPS, symbol cacophony-symbols:Antenna_1002427
- J6: footprint cacophony-footprints:SMD_M2_nut -> cacophony-library:SMD_BD4.4-L4.4-D2.8; LCSC C2928176 -> C2928178
Connections:
- net GND: now also C28.2, C29.2, RF3.2 (GND), RF3.3 (GND), RF3.4 (GND), U8.2 (Gnd)
- new net: C28.1, R35.1, U8.1 (Feed)
- new net: C29.1, R35.2, RF3.1 (SIG)
- new net: R37.2, R38.1, U8.5 (R3)
- new net: R38.2, R39.1, U8.6 (R4)
- new net: R39.2, U8.7 (R5)
- new net: R36.1, U8.3 (R1)
- new net: R36.2, R37.1, U8.4 (R2)
Other:
- note added: "GPS Antenna"

Commit message: WIP 2
Connections:
- net at U3.30 (USIM_RST): now also R19.1; no longer R17.1
- net at U3.34 (USIM_DATA): now also R17.1; no longer R19.1
- net at D6.4, R19.2: now also Card1.C2 (RST); no longer Card1.C7 (I/O)
- net at D6.6, R17.2: now also Card1.C7 (I/O); no longer Card1.C2 (RST)
Other:
- moved on the sheet: R17, R19
Changed lines of the file:
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@@
   (junction (at 209.55 88.9) (diameter 0) (color 0 0 0 0)
   )
-  (junction (at 177.8 86.36) (diameter 0) (color 0 0 0 0)
-  )
   (junction (at 180.34 88.9) (diameter 0) (color 0 0 0 0)
   )
   (junction (at 83.82 168.91) (diameter 0) (color 0 0 0 0)
   )
-  (junction (at 182.88 91.44) (diameter 0) (color 0 0 0 0)
+  (junction (at 177.8 91.44) (diameter 0) (color 0 0 0 0)
   )
   (junction (at 243.84 38.1) (diameter 0) (color 0 0 0 0)
@@
   )
   (junction (at 83.82 156.21) (diameter 0) (color 0 0 0 0)
+  )
+  (junction (at 182.88 86.36) (diameter 0) (color 0 0 0 0)
   )
   (junction (at 83.82 166.37) (diameter 0) (color 0 0 0 0)
@@
     (stroke (width 0) (type default) (color 0 0 0 0))
   )
-  (wire (pts (xy 182.88 91.44) (xy 187.96 91.44))
+  (wire (pts (xy 162.56 91.44) (xy 177.8 91.44))
     (stroke (width 0) (type default) (color 0 0 0 0))
   )
@@
     (stroke (width 0) (type default) (color 0 0 0 0))
   )
+  (wire (pts (xy 182.88 86.36) (xy 187.96 86.36))
+    (stroke (width 0) (type default) (color 0 0 0 0))
+  )
   (wire (pts (xy 209.55 95.25) (xy 209.55 91.44))
     (stroke (width 0) (type default) (color 0 0 0 0))
@@
     (stroke (width 0) (type default) (color 0 0 0 0))
   )
+  (wire (pts (xy 182.88 86.36) (xy 182.88 93.98))
+    (stroke (width 0) (type default) (color 0 0 0 0))
+  )
   (wire (pts (xy 254 35.56) (xy 254 38.1))
     (stroke (width 0) (type default) (color 0 0 0 0))
@@
     (stroke (width 0) (type default) (color 0 0 0 0))
   )
-  (wire (pts (xy 182.88 91.44) (xy 182.88 93.98))
-    (stroke (width 0) (type default) (color 0 0 0 0))
-  )
   (wire (pts (xy 83.82 69.85) (xy 85.09 69.85))
     (stroke (width 0) (type default) (color 0 0 0 0))
@@
     (stroke (width 0) (type default) (color 0 0 0 0))
   )
+  (wire (pts (xy 177.8 91.44) (xy 177.8 93.98))
+    (stroke (width 0) (type default) (color 0 0 0 0))
+  )
   (wire (pts (xy 175.26 83.82) (xy 175.26 93.98))
     (stroke (width 0) (type default) (color 0 0 0 0))
@@
     (stroke (width 0) (type default) (color 0 0 0 0))
   )
-  (wire (pts (xy 177.8 86.36) (xy 177.8 93.98))
-    (stroke (width 0) (type default) (color 0 0 0 0))
-  )
   (wire (pts (xy 185.42 78.74) (xy 186.69 78.74))
     (stroke (width 0) (type default) (color 0 0 0 0))
@@
     (stroke (width 0) (type default) (color 0 0 0 0))
   )
+  (wire (pts (xy 177.8 91.44) (xy 187.96 91.44))
+    (stroke (width 0) (type default) (color 0 0 0 0))
+  )
   (wire (pts (xy 243.84 38.1) (xy 245.11 38.1))
     (stroke (width 0) (type default) (color 0 0 0 0))
@@
     (stroke (width 0) (type default) (color 0 0 0 0))
   )
-  (wire (pts (xy 162.56 91.44) (xy 182.88 91.44))
-    (stroke (width 0) (type default) (color 0 0 0 0))
-  )
   (wire (pts (xy 264.16 60.96) (xy 264.16 59.69))
     (stroke (width 0) (type default) (color 0 0 0 0))
   )
-  (wire (pts (xy 162.56 86.36) (xy 177.8 86.36))
+  (wire (pts (xy 162.56 86.36) (xy 182.88 86.36))
     (stroke (width 0) (type default) (color 0 0 0 0))
   )
@@
   )
   (wire (pts (xy 252.73 38.1) (xy 254 38.1))
-    (stroke (width 0) (type default) (color 0 0 0 0))
-  )
-  (wire (pts (xy 177.8 86.36) (xy 187.96 86.36))
     (stroke (width 0) (type default) (color 0 0 0 0))
   )
@@
     (pin "2")
   )
-  (symbol (lib_id "Device:R") (at 158.75 91.44 90) (unit 1)
+  (symbol (lib_id "Device:R") (at 158.75 86.36 90) (unit 1)
     (in_bom yes) (on_board yes)
-    (property "Reference" "R19" (id 0) (at 154.94 90.17 90))
-    (property "Value" "22ohm" (id 1) (at 165.1 90.17 90))
-    (property "Footprint" "Resistor_SMD:R_0402_1005Metric" (id 2) (at 158.75 93.218 90)
-      (effects (font (size 1.27 1.27)) hide)
-    )
-    (property "Datasheet" "~" (id 3) (at 158.75 91.44 0)
-      (effects (font (size 1.27 1.27)) hide)
-    )
-    (property "LCSC" "C25092" (id 4) (at 158.75 91.44 0)
+    (property "Reference" "R19" (id 0) (at 154.94 85.09 90))
+    (property "Value" "22ohm" (id 1) (at 165.1 85.09 90))
+    (property "Footprint" "Resistor_SMD:R_0402_1005Metric" (id 2) (at 158.75 88.138 90)
+      (effects (font (size 1.27 1.27)) hide)
+    )
+    (property "Datasheet" "~" (id 3) (at 158.75 86.36 0)
+      (effects (font (size 1.27 1.27)) hide)
+    )
+    (property "LCSC" "C25092" (id 4) (at 158.75 86.36 0)
       (effects (font (size 1.27 1.27)) hide)
     )
@@
     (pin "2")
   )
-  (symbol (lib_id "Device:R") (at 158.75 86.36 90) (unit 1)
+  (symbol (lib_id "Device:R") (at 158.75 91.44 90) (unit 1)
     (in_bom yes) (on_board yes)
-    (property "Reference" "R17" (id 0) (at 154.94 85.09 90))
-    (property "Value" "22ohm" (id 1) (at 165.1 85.09 90))
-    (property "Footprint" "Resistor_SMD:R_0402_1005Metric" (id 2) (at 158.75 88.138 90)
-      (effects (font (size 1.27 1.27)) hide)
-    )
-    (property "Datasheet" "~" (id 3) (at 158.75 86.36 0)
-      (effects (font (size 1.27 1.27)) hide)
-    )
-    (property "LCSC" "C25092" (id 4) (at 158.75 86.36 0)
-      (effects (font (size 1.27 1.27)) hide)
-    )
+    (property "Reference" "R17" (id 0) (at 154.94 90.17 90))
+    (property "Value" "22ohm" (id 1) (at 165.1 90.17 90))
+    (property "Footprint" "Resistor_SMD:R_0402_1005Metric" (id 2) (at 158.75 93.218 90)
+      (effects (font (size 1.27 1.27)) hide)
+    )
+    (property "Datasheet" "~" (id 3) (at 158.75 91.44 0)
+      (effects (font (size 1.27 1.27)) hide)
+    )
+    (property "LCSC" "C25092" (id 4) (at 158.75 91.44 0)
+      (effects (font (size 1.27 1.27)) hide)
+    )
