File: lepton.kicad_sch (KiCad schematic)
At the start: 33 parts, among them U10 ME6216A28XG, U11 Flir_LEPTON, U12 3N25000G33YC, U13 TD6810, U14 TD6810

Commit message: WIP
Parts:
- L2, L3: footprint Inductor_SMD:L_Taiyo-Yuden_NR-40xx -> cacophony-library:IND-SMD_L4.0-W4.0_SWPA4018S
- TP1, TP12, TP2, TP3, TP4: footprint TestPoint:TestPoint_Pad_1.0x1.0mm -> cacophony-library:TP
- U12: footprint Oscillator:Oscillator_SMD_Abracon_ASE-4Pin_3.2x2.5mm -> cacophony-library:OSC-SMD_4P-L3.2-W2.5-BL
- renumbered U11 to U5
Changed lines of the file:
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@@
     (property "Reference" "L3" (id 0) (at 243.84 66.04 0))
     (property "Value" "4.7uH" (id 1) (at 243.84 68.58 0))
-    (property "Footprint" "Inductor_SMD:L_Taiyo-Yuden_NR-40xx" (id 2) (at 243.84 72.39 0)
+    (property "Footprint" "cacophony-library:IND-SMD_L4.0-W4.0_SWPA4018S" (id 2) (at 243.84 72.39 0)
       (effects (font (size 1.27 1.27)) hide)
     )
@@
       (effects (font (size 1.27 1.27)) (justify left))
     )
-    (property "Footprint" "TestPoint:TestPoint_Pad_1.0x1.0mm" (id 2) (at 127 107.95 0)
+    (property "Footprint" "cacophony-library:TP" (id 2) (at 127 107.95 0)
       (effects (font (size 1.27 1.27)) hide)
     )
@@
       (effects (font (size 1.27 1.27)) (justify left))
     )
-    (property "Footprint" "TestPoint:TestPoint_Pad_1.0x1.0mm" (id 2) (at 259.08 144.78 0)
+    (property "Footprint" "cacophony-library:TP" (id 2) (at 259.08 144.78 0)
       (effects (font (size 1.27 1.27)) hide)
     )
@@
     (property "Reference" "L2" (id 0) (at 243.84 34.29 0))
     (property "Value" "4.7uH" (id 1) (at 243.84 36.83 0))
-    (property "Footprint" "Inductor_SMD:L_Taiyo-Yuden_NR-40xx" (id 2) (at 243.84 40.64 0)
+    (property "Footprint" "cacophony-library:IND-SMD_L4.0-W4.0_SWPA4018S" (id 2) (at 243.84 40.64 0)
       (effects (font (size 1.27 1.27)) hide)
     )
@@
       (effects (font (size 1.27 1.27)) (justify left))
     )
-    (property "Footprint" "TestPoint:TestPoint_Pad_1.0x1.0mm" (id 2) (at 259.08 147.32 0)
+    (property "Footprint" "cacophony-library:TP" (id 2) (at 259.08 147.32 0)
       (effects (font (size 1.27 1.27)) hide)
     )
@@
     (property "Reference" "U12" (id 0) (at 121.92 92.71 0))
     (property "Value" "3N25000G33YC" (id 1) (at 121.92 95.25 0))
-    (property "Footprint" "Oscillator:Oscillator_SMD_Abracon_ASE-4Pin_3.2x2.5mm" (id 2) (at 121.92 96.52 0)
+    (property "Footprint" "cacophony-library:OSC-SMD_4P-L3.2-W2.5-BL" (id 2) (at 121.92 96.52 0)
       (effects (font (size 1.27 1.27)) hide)
     )
@@
       (effects (font (size 1.27 1.27)) (justify left))
     )
-    (property "Footprint" "TestPoint:TestPoint_Pad_1.0x1.0mm" (id 2) (at 259.08 142.24 0)
+    (property "Footprint" "cacophony-library:TP" (id 2) (at 259.08 142.24 0)
       (effects (font (size 1.27 1.27)) hide)
     )
@@
   (symbol (lib_id "Sensor_Optical:Flir_LEPTON") (at 102.87 156.21 0) (unit 1)
     (in_bom yes) (on_board yes) (fields_autoplaced)
-    (property "Reference" "U11" (id 0) (at 107.4294 132.715 0)
-      (effects (font (size 1.27 1.27)) (justify left))
-    )
-    (property "Value" "Flir_LEPTON" (id 1) (at 107.4294 135.255 0)
+    (property "Reference" "U5" (id 0) (at 107.4294 133.35 0)
+      (effects (font (size 1.27 1.27)) (justify left))
+    )
+    (property "Value" "Flir_LEPTON" (id 1) (at 107.4294 135.89 0)
       (effects (font (size 1.27 1.27)) (justify left))
     )
@@
       (effects (font (size 1.27 1.27)) (justify left))
     )
-    (property "Footprint" "TestPoint:TestPoint_Pad_1.0x1.0mm" (id 2) (at 259.08 149.86 0)
-      (effects (font (size 1.27 1.27)) hide)
-    )
+    (property "Footprint" "cacophony-library:TP" (id 2) (at 259.08 149.86 0)
+      (effects (font (size 1.27 1.27)) hide)
+    )

Commit message: WIP 2
Parts:
- removed TP12: TestPoint, cacophony-library:TP, symbol Connector:TestPoint
- added TP14: TestPoint, cacophony-library:TP, symbol Connector:TestPoint
Connections:
- net MASTER_CLK: now also TP14.1
Changed lines of the file:
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@@
     (pin "2")
-  )
-  (symbol (lib_id "Connector:TestPoint") (at 132.08 107.95 180) (unit 1)
-    (in_bom yes) (on_board yes)
-    (property "Reference" "TP12" (id 0) (at 132.08 123.19 90)
-      (effects (font (size 1.27 1.27)) (justify left))
-    )
-    (property "Value" "TestPoint" (id 1) (at 132.08 113.03 90)
-      (effects (font (size 1.27 1.27)) (justify left))
-    )
-    (property "Footprint" "cacophony-library:TP" (id 2) (at 127 107.95 0)
-      (effects (font (size 1.27 1.27)) hide)
-    )
-    (property "Datasheet" "~" (id 3) (at 127 107.95 0)
-      (effects (font (size 1.27 1.27)) hide)
-    )
-    (pin "1")
   )
   (symbol (lib_id "Device:R") (at 251.46 77.47 180) (unit 1)
@@
     (pin "2")
   )
+  (symbol (lib_id "Connector:TestPoint") (at 132.08 107.95 270) (unit 1)
+    (in_bom no) (on_board yes)
+    (property "Reference" "TP14" (id 0) (at 137.16 107.95 90)
+      (effects (font (size 1.27 1.27)) (justify left))
+    )
+    (property "Value" "TestPoint" (id 1) (at 137.16 107.95 90)
+      (effects (font (size 1.27 1.27)) (justify left) hide)
+    )
+    (property "Footprint" "cacophony-library:TP" (id 2) (at 132.08 113.03 0)
+      (effects (font (size 1.27 1.27)) hide)
+    )
+    (property "Datasheet" "~" (id 3) (at 132.08 113.03 0)
+      (effects (font (size 1.27 1.27)) hide)
+    )
+    (pin "1")
+  )
   (symbol (lib_id "Device:R") (at 196.85 135.89 0) (unit 1)
