File: thermal-camera-v2.kicad_sch (KiCad schematic)
At the start: 83 parts, among them J1 Raspberry_Pi_2_3, J10 Screw_Terminal_01x01, J2 Conn_01x02, J3 Conn_01x10, J4 Screw_Terminal_01x01, J5 Screw_Terminal_01x01, J6 Bus_PCI_Express_Mini, J7 Screw_Terminal_01x01, J8 Screw_Terminal_01x01, J9 SIM_Card_Shielded, Q1 Q_PMOS_GSD, Q2 Q_PMOS_GSD, U1 STM32F030C8Tx, U10 ME6216A28XG, U11 Flir_LEPTON, U12 3N25000G33YC, U13 TD6810, U14 TD6810, U15 MMC5633NJL, U16 Ai-Thinker-Ra-01, U2 SHT30-DIS, U3 ATtiny85-20P, U4 LMR16030S, U5 XC6206PxxxMR, U6 SPH0645LM4H, U7 PCF8563T, U8 XC6206PxxxMR, U9 MAX98357, Y1 Crystal

Commit message: WIP
Parts:
- removed AE?: Antenna, symbol Device:Antenna
- removed C10, C19, C23, C24, C9: 4.7uF, Capacitor_SMD:C_0402_1005Metric, symbol Device:C_Small
- removed C11, C12, C13, C14: 100nF, Capacitor_SMD:C_0402_1005Metric, symbol Device:C_Small
- removed C15, C16, C20: 10uF, Capacitor_SMD:C_0603_1608Metric, symbol Device:C_Small
- removed C17, C18: 22pF, Capacitor_SMD:C_0402_1005Metric, symbol Device:C_Small
- removed C22, C25: 22uF, Capacitor_SMD:C_0805_2012Metric, symbol Device:C_Small
- removed C4: 100nF, Capacitor_SMD:C_0603_1608Metric, symbol Device:C_Small
- removed C6: 1uF, Capacitor_SMD:C_0402_1005Metric, symbol Device:C_Small
- removed D1: D_Zener, Diode_SMD:D_SMA, symbol Device:D_Zener
- removed D2: WS2812B, LED_SMD:LED_WS2812B_PLCC4_5.0x5.0mm_P3.2mm, symbol LED:WS2812B
- removed D3, D4: D_Shockley, Diode_SMD:D_SOD-323, symbol Device:D_Shockley
- removed D5: D_Shockley, Diode_SMD:D_SMA, symbol Device:D_Shockley
- removed J10, J4, J5, J7, J8, J?: Screw_Terminal_01x01, symbol Connector:Screw_Terminal_01x01
- removed J2: Conn_01x02, Connector_JST:JST_XA_S02B-XASK-1_1x02_P2.50mm_Horizontal, symbol Connector_Generic:Conn_01x02
- removed J3: Conn_01x10, Connector_PinSocket_2.54mm:PinSocket_1x10_P2.54mm_Vertical, symbol Connector_Generic:Conn_01x10
- removed J6: Bus_PCI_Express_Mini, BUS_PCI_Express_Mini_Full, symbol Connector:Bus_PCI_Express_Mini
- removed J9: SIM_Card_Shielded, JAE_SIM_Card_SF72S006, symbol Connector:SIM_Card_Shielded
- removed L1: 15uH, battery-dc-dc-converter:SWRH1207B, symbol pspice:INDUCTOR
- removed L2, L3: 4.7uH, Inductor_SMD:L_Taiyo-Yuden_NR-40xx, symbol cacophony-symbols:Power Inductor
- removed LS1: Speaker, Connector_JST:JST_XA_S02B-XASK-1_1x02_P2.50mm_Horizontal, symbol Device:Speaker
- removed Q1, Q2: Q_PMOS_GSD, Package_TO_SOT_SMD:SOT-23, symbol Device:Q_PMOS_GSD
- removed R1, R13, R14, R15: 100K, Resistor_SMD:R_0402_1005Metric, symbol Device:R
- removed R10: 10K, Resistor_SMD:R_0402_1005Metric, symbol Device:R
- removed R12: 68K, Resistor_SMD:R_0402_1005Metric, symbol Device:R
- removed R6, R8: 560k, Resistor_SMD:R_0603_1608Metric, symbol Device:R
- removed R`1: 3.3R, Resistor_SMD:R_0805_2012Metric, symbol Device:R
- removed U1: STM32F030C8Tx, Package_QFP:LQFP-48_7x7mm_P0.5mm, symbol MCU_ST_STM32F0:STM32F030C8Tx
- removed U10: ME6216A28XG, Package_TO_SOT_SMD:TSOT-23, symbol cacophony-symbols:ME6216A28XG
- removed U11: Flir_LEPTON, libraries:MOLEX_105028-1001, symbol Sensor_Optical:Flir_LEPTON
- removed U12: 3N25000G33YC, Oscillator:Oscillator_SMD_Abracon_ASE-4Pin_3.2x2.5mm, symbol cacophony-symbols:3N25000G33YC
- removed U13, U14: TD6810, Package_TO_SOT_SMD:TSOT-23-5, symbol cacophony-symbols:TD6810
- removed U3: ATtiny85-20P, Package_DIP:DIP-8_W7.62mm, symbol MCU_Microchip_ATtiny:ATtiny85-20P
- removed U4: LMR16030S, Package_SO:TI_SO-PowerPAD-8, symbol cacophony-symbols:LMR16030S
- removed U5, U8: XC6206PxxxMR, Package_TO_SOT_SMD:SOT-23, symbol Regulator_Linear:XC6206PxxxMR
- added C38: 220nF, Capacitor_SMD:C_0402_1005Metric, symbol Device:C_Small
- added D2: LED_RGB, cacophony-footprints:LED_RGB, symbol cacophony-symbols:LED_RGB
- added D3, D4: D, Diode_SMD:D_SMA, symbol Device:D
- added H1, H2, H3, H4: MountingHole, MountingHole:MountingHole_3.5mm, symbol Mechanical:MountingHole
- added J2, J3: Screw_Terminal_M2_L10, cacophony-footprints:SMD_M2_nut, symbol Connector:Screw_Terminal_01x01
- added J4: Conn_01x05, cacophony-footprints:JST_XA_B05B-XASK-1-A_1x05_P2.50mm_Vertical, symbol Connector_Generic:Conn_01x05
- added J7, J8: Conn_01x02, Connector_PinHeader_1.00mm:PinHeader_1x02_P1.00mm_Vertical, symbol Connector_Generic:Conn_01x02
- added R21: 100k, Resistor_SMD:R_0402_1005Metric, symbol Device:R
- added R22, R23, R24, R25, R26, R27, R29, R30, R31, R32, R33: 22ohm, Resistor_SMD:R_0402_1005Metric, symbol Device:R
- added R28, R34: 10k, Resistor_SMD:R_0402_1005Metric, symbol Device:R
- added RF1: KH-IPEX-4-K501-29, cacophony-footprints:IPEX4-SMD_4P-L1.8-W1.7-LS2.0-L_KH-IPEX4-2020, symbol cacophony-symbols:KH-IPEX-4-K501-29
- added TP10, TP5, TP6, TP7, TP8, TP9: TestPoint, Connector_PinHeader_1.00mm:PinHeader_1x01_P1.00mm_Vertical, symbol Connector:TestPoint
- added U1: ATtiny1616-M, Package_DFN_QFN:VQFN-20-1EP_3x3mm_P0.4mm_EP1.7x1.7mm, symbol MCU_Microchip_ATtiny:ATtiny1616-M
- BZ1: footprint Buzzer_Beeper:MagneticBuzzer_PUI_AT-0927-TT-6-R -> cacophony-footprints:MagneticBuzzer_PUI_AT-0927-TT-6-R
- C1: value 220uF -> 220nF; footprint Capacitor_SMD:CP_Elec_8x10 -> Capacitor_SMD:C_0402_1005Metric; LCSC C2895286 -> C16772
- C2: value 1uF -> 220nF; LCSC C52923 -> C16772
- C21: value 4.7uF -> 220nF; LCSC C23733 -> C16772
- C3: value 10nF -> 220nF; LCSC C15195 -> C16772
- C5: value 1uF -> 10uF; footprint Capacitor_SMD:C_0402_1005Metric -> Capacitor_SMD:C_0603_1608Metric; LCSC C52923 -> C19702
- C7: footprint Capacitor_SMD:C_0805_2012Metric -> Capacitor_SMD:C_0603_1608Metric; LCSC C45783 -> C86295
- C8: value 100nF -> 220nF; LCSC C1525 -> C16772
- J1: footprint Connector_PinSocket_2.54mm:PinSocket_2x20_P2.54mm_Vertical -> cacophony-footprints:RPi_SMD; LCSC C2897421 -> C3975165
- R11: value 330K -> 10k; LCSC C25778 -> C25744
- R2: value 47K -> 180R; footprint Resistor_SMD:R_0402_1005Metric -> Resistor_SMD:R_0603_1608Metric; LCSC C25792 -> C22828
- R3: footprint R_0603_1608Metric -> Resistor_SMD:R_0603_1608Metric
- R4: value 100k -> 180R; LCSC C25803 -> C22828
- R5: value 6.8k -> 180R; LCSC C23212 -> C22828
- R7: value 68k -> 1M; LCSC C23231 -> C22935
- R9: footprint Resistor_SMD:R_0603_1608Metric -> Resistor_SMD:R_0402_1005Metric; LCSC C25803 -> C25741
- U15: LCSC (none) -> C404328
- U16: footprint RF_Module:Ai-Thinker-Ra-01-LoRa -> cacophony-footprints:Ai-Thinker-Ra-01-LoRa; LCSC (none) -> C503593
- U6: LCSC (none) -> C2686054
Connections:
- net I2S_DOUT is gone; now on net I2S_DOUT/SCLK1: U9.1 (DIN)
- net I2S_LRCLK is gone; now on net I2S_LRCLK/MISO1: U9.14 (LRCLK)
- net +3V3: now also C2.2, C3.2, R11.1, C38.2, D3.2 (A), R21.2, R28.1, U1.4 (VCC)
- net +5V: now also J1.2 (5V), J1.4 (5V); no longer R7.1
- net BUZZER: now also J1.22 (GPIO25)
- net GND: now also C1.1, C2.1, C21.1, C3.1, U16.16 (GND), U16.2 (GND), U16.9 (GND), U6.2 (SEL), C38.1, D2.4 (BK), D2.5 (GK), D2.6 (RK), J4.1 (Pin_1), RF1.2 (GND), RF1.3 (GND), RF1.4 (GND), U1.21 (GND), U1.3 (GND); no longer C1.2, C2.2, C21.2, C3.2, R2.2, R4.2
- net I2S_BCLK: now also U6.4 (BCLK), R24.1
- net SCL: now also J1.5 (SCL/GPIO3), R28.2, U1.14 (PB0)
- net SDA: now also J1.3 (SDA/GPIO2), R11.2, U1.13 (PB1)
- net ~{RTC_INT}: now also U1.15 (PC0)
- net LED_B: now reaches R5.1
- net LED_B: now also U1.8 (PA7); no longer R4.1
- net at R5.2: now also D2.3 (BA)
- net LED_R: now reaches R2.1
- net LED_R: now also U1.6 (PA5)
- net RTC_BT_SENSE: now reaches BT1.1 (+)
- net RTC_BT_SENSE: now also D4.2 (A), R34.2, U1.16 (PC1)
- net SPEAKER_-: now reaches U9.10 (OUTN)
- net SPEAKER_-: now also J4.3 (Pin_3)
- net SPEAKER_+: now reaches U9.9 (UOTP)
- net SPEAKER_+: now also J4.4 (Pin_4)
- net at J1.10 (GPIO15/RXD): now also J7.1 (Pin_1)
- net at J1.11 (GPIO17): now also R23.2
- net at J1.12 (GPIO18/PWM0): now also R24.2
- net at J1.13 (GPIO27): now also R33.2
- net at J1.15 (GPIO22): now also TP9.1
- net ~{LORA_RESET}: now reaches J1.16 (GPIO23)
- net ~{LORA_RESET}: now also U16.4 (~{RESET})
- net at J1.18 (GPIO24): now also TP10.1
- net at J1.19 (MOSI0/GPIO10): now also R31.1
- net MISO_0: now reaches J1.21 (MISO0/GPIO9)
- net MISO_0: now also R29.2
- net at J1.23 (SCLK0/GPIO11): now also R32.1
- net at J1.24 (~{CE0}/GPIO8): now also R30.1
- net LEPTON_POWER_EN: now reaches J1.26 (~{CE1}/GPIO7)
- net at J1.27 (ID_SD/GPIO0): now also J8.1 (Pin_1)
- net at J1.28 (ID_SC/GPIO1): now also J8.2 (Pin_2)
- net LEPTON_VSYNC: now reaches J1.29 (GCLK1/GPIO5)
- net LEPTON_CLK_EN: now reaches J1.31 (GCLK2/GPIO6)
- net LEPTON_PWR_DWN_L: now reaches J1.32 (PWM0/GPIO12)
- net LEPTON_RESET_L: now reaches J1.33 (PWM1/GPIO13)
- net at J1.35 (GPIO19/MISO1): now also R25.2
- net 4G_POWER_ON: now reaches J1.36 (GPIO16)
- net ~{W_DISABLE1}: now reaches J1.37 (GPIO26)
- net I2S_DIN/MOSI1: now reaches J1.38 (GPIO20/MOSI1)
- net I2S_DIN/MOSI1: now also U16.14 (MOSI), R27.2
- net at J1.40 (GPIO21/SCLK1): now also R26.2
- net SPEAKER_SD_MODE: now reaches J1.7 (GCLK0/GPIO4)
- net SPEAKER_SD_MODE: now also R7.1
- net at J1.8 (GPIO14/TXD): now also J7.2 (Pin_2)
- net at C5.1, U7.8 (VDD): now also D3.1 (K), D4.1 (K)
- net at U16.1 (ANT): now also RF1.1 (SIG)
- net I2S_DOUT/SCLK1: now reaches U16.12 (SCK)
- net I2S_DOUT/SCLK1: now also R26.1
- net at U16.13 (MISO): now also R22.2
- net LORA_CS: now reaches U16.15 (~{NSS})
- net LORA_CS: now also R23.1
- net +3V3_Lin: now reaches U16.3 (VDD)
- net +3V3_Lin: now also C1.2, C21.2, U6.5 (VDD)
- net at R7.2: now also U9.4 (~{SD_MODE})
- net I2S_LRCLK/MISO1: now reaches U6.1 (WS)
- net I2S_LRCLK/MISO1: now also R22.1, R25.1
- net at U6.6 (DATA): now also R27.1
- removed net +3V0: C21.1, R11.1
- new net: TP5.1, U1.18 (PC3)
- new net: R29.1, U1.1 (PA2)
- new net: TP7.1, U1.11 (PB3)
- new net: TP6.1, U1.12 (PB2)
- new net: TP8.1, U1.9 (PB5)
- new net: D2.2 (GA), R4.2
- new net: D2.1 (RA), R2.2
- new net 5V_EN: R21.1, U1.5 (PA4)
- new net ATtiny_RESET: R33.1, U1.19 (~{RESET}/PA0)
- new net BATT_SENSE: J4.5 (Pin_5), U1.10 (PB4)
- new net LED_G: R4.1, U1.7 (PA6)
- new net LEPTON_CS: R30.2
- new net MOSI_0: R31.2, U1.20 (PA1)
- new net RTC_BT_LOAD: R34.1, U1.17 (PC2)
- new net SCLK_0: R32.2, U1.2 (PA3)
- new net VIN: J4.2 (Pin_2)
- no-connect marks 16 -> 17
Other:
- added sheet Antennas (antennas.kicad_sch)
- added sheet Lepton (lepton.kicad_sch)
- added sheet Power (power.kicad_sch)
- added sheet SIM7600G_M.2 (SIM7600G_M.2.kicad_sch)
- note added: "- 3.3V x - 5V x - Audio x - RTC x - Buzzer x - ATtiny x - Humidity x - Mic x - Modem x - RGB LED x - LORA x - FLIR x - Compas (C404328) - Accel - USB plug (C879731)"
- note added: "DIG: 343-ANT-8/9-PW-LPN-ND DIG: 939-1072-1-ND"
- note added: "Magnetic Sensor"
- note added: "Microphone"
- note added: "RTC"
- note added: "Speaker"
- note added: "Status LED"
- note added: "TODO: - Change to ipex-4 C530666"
- note added: "TODO: - Check programming ATTiny1616 - Check how to keep Pi powered when rebooting STM32 - Check Microphone and LORA interferance."
- note added: "Temp and Humidity Sensor"
- note removed: "- 3.3V x - 5V x - Audio x - RTC x - Buzzer x - ATtiny x - Humidity x - Mic x - Modem x - RGB LED x - LORA x - FLIR x - Compas (C404328) - GPS - Accel"
- note removed: "140mW typical power usage ~800mW during shutter event"
- note removed: "VDD, Sensor voltage Voltage: (2.72,2.80,2.88)V Ripple: 30mV Current: (12,14,16)mA"
- note removed: "VDDC, Core voltage Voltage: (1.14,1.2,1.26)V Ripple: 50mV Current: (76,84,110)mA"
- note removed: "VDDIO, IO voltage Voltage: (2.5,2.8,3.1)V Ripple: 50mV Current: (1, 235, 310)mA FLIR recommends utilizing two separate power supplies rather than a common supply for VDD and VDDIO due to noise considerations"
- moved on the sheet: BT1, BZ1, C5, C7, C8, J1, R3, R9, U15, U16, U2, U6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

Commit message: WIP
Parts:
- removed H1: MountingHole, MountingHole:MountingHole_3.5mm, symbol Mechanical:MountingHole
- removed J4: Conn_01x05, cacophony-footprints:JST_XA_B05B-XASK-1-A_1x05_P2.50mm_Vertical, symbol Connector_Generic:Conn_01x05
- removed J7, J8: Conn_01x02, Connector_PinHeader_1.00mm:PinHeader_1x02_P1.00mm_Vertical, symbol Connector_Generic:Conn_01x02
- removed R29, R33: 22ohm, Resistor_SMD:R_0402_1005Metric, symbol Device:R
- added C4, C6: 10uF, Capacitor_SMD:C_0603_1608Metric, symbol Device:C_Small
- added D1, D5: D, Diode_SMD:D_SOD-523, symbol Device:D
- added J4: Conn_02x04_Odd_Even, cacophony-library:power-pcb, symbol Connector_Generic:Conn_02x04_Odd_Even
- added R1: 1k, Resistor_SMD:R_0402_1005Metric, symbol Device:R
- added TP11, TP13, TP14, TP15, TP16, TP17: TestPoint, cacophony-library:TP, symbol Connector:TestPoint
- added U4: ME6211, Package_TO_SOT_SMD:SOT-23-5, symbol cacophony-symbols:ME6211
- BZ1: footprint cacophony-footprints:MagneticBuzzer_PUI_AT-0927-TT-6-R -> cacophony-footprints:BUZ-TH_BD9.0-P5.00-D0.6-FD; LCSC C96256 -> C96102
- D2: footprint cacophony-footprints:LED_RGB -> cacophony-library:LED-SMD_6PIN-L1.60-W1.50-BL-RD
- D3, D4: footprint Diode_SMD:D_SMA -> Diode_SMD:D_SOD-523; LCSC C95872 -> C668989
- H2, H3, H4: footprint MountingHole:MountingHole_3.5mm -> cacophony-library:Mouning_Hole_M3
- J1: footprint cacophony-footprints:RPi_SMD -> cacophony-footprints:RPi_2_W_SMD
- J2, J3: footprint cacophony-footprints:SMD_M2_nut -> cacophony-library:SMD_NUT_D5.6-HD3.6-L10.0
- R2, R3, R4, R5: footprint Resistor_SMD:R_0603_1608Metric -> Resistor_SMD:R_0402_1005Metric; LCSC C22828 -> C38941
- TP10, TP5, TP6, TP7, TP8, TP9: footprint Connector_PinHeader_1.00mm:PinHeader_1x01_P1.00mm_Vertical -> cacophony-library:TP
- U16: footprint cacophony-footprints:Ai-Thinker-Ra-01-LoRa -> cacophony-library:WIRELM-SMD_RA-01H
- U9: footprint Package_DFN_QFN:TQFN-16-1EP_3x3mm_P0.5mm_EP1.23x1.23mm -> Package_DFN_QFN:TQFN-16-1EP_3x3mm_P0.5mm_EP1.6x1.6mm
Connections:
- net ATtiny_RESET is gone; now on net ATtiny_RESET_UPDI: U1.19 (~{RESET}/PA0)
- net +3V3: now also J4.6 (Pin_6)
- net +3V3_Lin: now also C6.1, U4.5 (Vout)
- net +5V: now also C4.1, J4.4 (Pin_4), U4.1 (Vin), U4.3 (CE)
- net 5V_EN: now also J4.5 (Pin_5)
- net BATT_SENSE: now also J4.7 (Pin_7)
- net GND: now also C4.2, C6.2, J4.2 (Pin_2), J4.8 (Pin_8), U4.2 (Vss)
- net LED_B: now also D2.3 (BA), R2.2; no longer R5.1, U1.8 (PA7)
- net LED_G: now also D2.1 (RA), R5.2; no longer R4.1, U1.7 (PA6)
- net LED_R: now also D2.2 (GA), R4.2; no longer R2.1, U1.6 (PA5)
- net MOSI_0: no longer U1.20 (PA1)
- net SCLK_0: no longer U1.2 (PA3)
- net SPEAKER_+: now also J4.1 (Pin_1)
- net SPEAKER_-: now also J4.3 (Pin_3)
- net at TP5.1: now also J1.15 (GPIO22); no longer U1.18 (PC3)
- net at U1.1 (PA2): now also TP6.1
- net at TP7.1: now also U1.2 (PA3); no longer U1.11 (PB3)
- net at U1.12 (PB2): now also TP8.1; no longer TP6.1
- net at U1.9 (PB5): now also TP16.1; no longer TP8.1
- net ATtiny_RESET_UPDI: now reaches J1.10 (GPIO15/RXD)
- net ATtiny_RESET_UPDI: now also R1.1
- net at J1.8 (GPIO14/TXD): now also R1.2
- net at J1.13 (GPIO27): now also TP10.1
- net at TP9.1: now also J1.18 (GPIO24); no longer J1.15 (GPIO22)
- net at J1.27 (ID_SD/GPIO0): now also TP11.1
- net at J1.28 (ID_SC/GPIO1): now also TP13.1
- net at U2.6 (~{RESET}): now also TP17.1
- net BUZZER: no longer names the net of R3.1
- net BUZZER: now also D1.1 (K), D5.1 (K); no longer J1.22 (GPIO25)
- new net: TP15.1, U1.11 (PB3)
- new net: R5.1, U1.6 (PA5)
- new net: R4.1, U1.7 (PA6)
- new net: TP14.1, U1.20 (PA1)
- new net: R2.1, U1.8 (PA7)
- new net ATTiny_BUZZER: D5.2 (A), U1.18 (PC3)
- new net PI_BUZZER: D1.2 (A), J1.22 (GPIO25)
Other:
- removed sheet Antennas
- removed sheet Power
- note added: "TODO: - ~ Remove copper around magnet sensor ~ - Capacitors on RTC crystal? - Fix height of M.2 standoff"
- note added: "USB micro B plugs - C2833885 - C283546"
- note removed: "- 3.3V x - 5V x - Audio x - RTC x - Buzzer x - ATtiny x - Humidity x - Mic x - Modem x - RGB LED x - LORA x - FLIR x - Compas (C404328) - Accel - USB plug (C879731)"
- note removed: "Status LED"
- note removed: "TODO: - Check programming ATTiny1616 - Check how to keep Pi powered when rebooting STM32 - Check Microphone and LORA interferance."

Commit message: WIP 2
Parts:
- removed TP14, TP16, TP17: TestPoint, cacophony-library:TP, symbol Connector:TestPoint
- added TP12: TestPoint, cacophony-library:TP, symbol Connector:TestPoint
- TP10, TP13, TP15, TP5, TP6, TP7, TP8, TP9: footprint cacophony-library:TP -> cacophony-library:TP_PAD
Connections:
- net +3V3: now also J4.4 (Pin_4); no longer J4.6 (Pin_6)
- net +5V: now also J4.6 (Pin_6); no longer J4.4 (Pin_4)
- net 5V_EN: now also J4.3 (Pin_3); no longer J4.5 (Pin_5)
- net ATTiny_BUZZER: now also U1.2 (PA3); no longer U1.18 (PC3)
- net BATT_SENSE: now also J4.1 (Pin_1), U1.6 (PA5); no longer J4.7 (Pin_7), U1.10 (PB4)
- net LED_B: now also R2.1, U1.18 (PC3); no longer D2.3 (BA), R2.2
- net LED_G: now also R5.1, U1.1 (PA2); no longer D2.1 (RA), R5.2
- net LED_R: now also R4.1, U1.20 (PA1); no longer D2.2 (GA), R4.2
- net LEPTON_CLK_EN: now also J1.13 (GPIO27); no longer J1.31 (GCLK2/GPIO6)
- net LEPTON_POWER_EN: now also J1.22 (GPIO25); no longer J1.26 (~{CE1}/GPIO7)
- net LEPTON_PWR_DWN_L: now also J1.15 (GPIO22); no longer J1.32 (PWM0/GPIO12)
- net LEPTON_RESET_L: now also J1.16 (GPIO23); no longer J1.33 (PWM1/GPIO13)
- net LEPTON_VSYNC: now also J1.18 (GPIO24); no longer J1.29 (GCLK1/GPIO5)
- net PI_BUZZER: now also J1.37 (GPIO26); no longer J1.22 (GPIO25)
- net SPEAKER_+: now also J4.7 (Pin_7); no longer J4.1 (Pin_1)
- net SPEAKER_-: now also J4.5 (Pin_5); no longer J4.3 (Pin_3)
- net ~{LORA_RESET}: now also J1.33 (PWM1/GPIO13); no longer J1.16 (GPIO23)
- net ~{W_DISABLE1}: now also J1.32 (PWM0/GPIO12); no longer J1.37 (GPIO26)
- net at TP10.1: now also U1.9 (PB5); no longer J1.13 (GPIO27)
- net at U2.6 (~{RESET}): now also TP13.1
- net at U1.12 (PB2): now also TP7.1; no longer TP8.1
- net at TP9.1: now also U1.10 (PB4); no longer J1.18 (GPIO24)
- net at U2.3 (ALERT): now also TP15.1
- net at U1.11 (PB3): now also TP8.1; no longer TP15.1
- net at U1.7 (PA6): now also TP5.1; no longer R4.1
- net at J1.28 (ID_SC/GPIO1): now also TP12.1; no longer TP13.1
- net at TP6.1: now also U1.8 (PA7); no longer U1.1 (PA2)
- new net: D2.1 (RA), R5.2
- new net: D2.2 (GA), R4.2
- new net: D2.3 (BA), R2.2
- no-connect marks 17 -> 19
Other:
- note added: "TODO:"
- note removed: "TODO: - ~ Remove copper around magnet sensor ~ - Capacitors on RTC crystal? - Fix height of M.2 standoff"
- moved on the sheet: D2, J1, J2, J3, R1, R2, R23, R24, R25, R26, R30, R31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

Commit message: WIP
Other:
- note added: "Add another cap"
Changed lines of the file:
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@@
     (effects (font (size 2 2)) (justify left bottom))
+  )
+  (text "Add another cap" (at 345.44 91.44 0)
+    (effects (font (size 1.27 1.27)) (justify left bottom))
   )
   (text "Speaker" (at 330.2 30.48 0)

Commit message: Low power version WIP
Connections:
- net I2S_LRCLK/MISO1: no longer R25.1
