File: plug-pcb/plug-pcb/plug-pcb.kicad_sch (KiCad schematic)
At the start: 6 parts, among them J1 JCON_M12_02Pin, J2 Conn_01x05, J3 JCON_M16_04Pin

Commit message: WIP
Parts:
- J1: footprint (none) -> cacophony-footprints:jcon-2pin-m12
- J2: LCSC (none) -> C265396
- J3: footprint (none) -> cacophony-footprints:jcon-4pin_m16
- R1: footprint (none) -> Resistor_SMD:R_1210_3225Metric; LCSC (none) -> C304148
- R2: footprint (none) -> Resistor_SMD:R_0805_2012Metric; LCSC (none) -> C74850
- R3: renamed from R?; footprint (none) -> Resistor_SMD:R_0805_2012Metric; LCSC (none) -> C351592
Changed lines of the file:
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@@
+    (stroke (width 0) (type default) (color 0 0 0 0))
+  )
+  (wire (pts (xy 134.62 78.74) (xy 134.62 80.01))
     (stroke (width 0) (type default) (color 0 0 0 0))
   )
@@
   )
   (wire (pts (xy 173.99 113.03) (xy 173.99 114.3))
+    (stroke (width 0) (type default) (color 0 0 0 0))
+  )
+  (wire (pts (xy 143.51 82.55) (xy 143.51 83.82))
     (stroke (width 0) (type default) (color 0 0 0 0))
   )
@@
       (effects (font (size 1.27 1.27)) hide)
     )
+    (property "LCSC" "C265396" (id 4) (at 30.48 110.49 0)
+      (effects (font (size 1.27 1.27)) hide)
+    )
     (pin "1")
     (pin "2")
@@
       (effects (font (size 1.27 1.27)) (justify left))
     )
-    (property "Footprint" "" (id 2) (at 95.25 109.22 0)
+    (property "Footprint" "cacophony-footprints:jcon-2pin-m12" (id 2) (at 95.25 109.22 0)
       (effects (font (size 1.27 1.27)) hide)
     )
@@
     (pin "2")
   )
+  (symbol (lib_id "power:GND") (at 134.62 80.01 0) (unit 1)
+    (in_bom yes) (on_board yes) (fields_autoplaced)
+    (property "Reference" "#PWR0107" (id 0) (at 134.62 86.36 0)
+      (effects (font (size 1.27 1.27)) hide)
+    )
+    (property "Value" "GND" (id 1) (at 134.62 85.09 0))
+    (property "Footprint" "" (id 2) (at 134.62 80.01 0)
+      (effects (font (size 1.27 1.27)) hide)
+    )
+    (property "Datasheet" "" (id 3) (at 134.62 80.01 0)
+      (effects (font (size 1.27 1.27)) hide)
+    )
+    (pin "1")
+  )
   (symbol (lib_id "Device:R") (at 173.99 118.11 0) (unit 1)
     (in_bom yes) (on_board yes) (fields_autoplaced)
@@
       (effects (font (size 1.27 1.27)) (justify left))
     )
-    (property "Footprint" "" (id 2) (at 172.212 118.11 90)
+    (property "Footprint" "Resistor_SMD:R_0805_2012Metric" (id 2) (at 172.212 118.11 90)
       (effects (font (size 1.27 1.27)) hide)
     )
     (property "Datasheet" "~" (id 3) (at 173.99 118.11 0)
+      (effects (font (size 1.27 1.27)) hide)
+    )
+    (property "LCSC" "C74850" (id 4) (at 173.99 118.11 0)
       (effects (font (size 1.27 1.27)) hide)
     )
@@
     (pin "1")
   )
+  (symbol (lib_id "power:PWR_FLAG") (at 143.51 83.82 180) (unit 1)
+    (in_bom yes) (on_board yes) (fields_autoplaced)
+    (property "Reference" "#FLG0102" (id 0) (at 143.51 85.725 0)
+      (effects (font (size 1.27 1.27)) hide)
+    )
+    (property "Value" "PWR_FLAG" (id 1) (at 146.05 85.0899 0)
+      (effects (font (size 1.27 1.27)) (justify right))
+    )
+    (property "Footprint" "" (id 2) (at 143.51 83.82 0)
+      (effects (font (size 1.27 1.27)) hide)
+    )
+    (property "Datasheet" "~" (id 3) (at 143.51 83.82 0)
+      (effects (font (size 1.27 1.27)) hide)
+    )
+    (pin "1")
+  )
   (symbol (lib_id "power:+12V") (at 49.53 113.03 0) (unit 1)
     (in_bom yes) (on_board yes) (fields_autoplaced)
@@
   (symbol (lib_id "Device:R") (at 173.99 127 0) (unit 1)
     (in_bom yes) (on_board yes) (fields_autoplaced)
-    (property "Reference" "R?" (id 0) (at 176.53 125.7299 0)
+    (property "Reference" "R3" (id 0) (at 176.53 125.7299 0)
       (effects (font (size 1.27 1.27)) (justify left))
     )
@@
       (effects (font (size 1.27 1.27)) (justify left))
     )
-    (property "Footprint" "" (id 2) (at 172.212 127 90)
+    (property "Footprint" "Resistor_SMD:R_0805_2012Metric" (id 2) (at 172.212 127 90)
       (effects (font (size 1.27 1.27)) hide)
     )
@@
       (effects (font (size 1.27 1.27)) hide)
     )
-    (pin "1")
-    (pin "2")
+    (property "LCSC" "C351592" (id 4) (at 173.99 127 0)
+      (effects (font (size 1.27 1.27)) hide)
+    )
+    (pin "1")
+    (pin "2")
+  )
+  (symbol (lib_id "power:+12V") (at 143.51 82.55 0) (unit 1)
+    (in_bom yes) (on_board yes) (fields_autoplaced)
+    (property "Reference" "#PWR0106" (id 0) (at 143.51 86.36 0)
+      (effects (font (size 1.27 1.27)) hide)
+    )
+    (property "Value" "+12V" (id 1) (at 143.51 77.47 0))
+    (property "Footprint" "" (id 2) (at 143.51 82.55 0)
+      (effects (font (size 1.27 1.27)) hide)
+    )
+    (property "Datasheet" "" (id 3) (at 143.51 82.55 0)
+      (effects (font (size 1.27 1.27)) hide)
+    )
+    (pin "1")
+  )
+  (symbol (lib_id "power:PWR_FLAG") (at 134.62 78.74 0) (unit 1)
+    (in_bom yes) (on_board yes) (fields_autoplaced)
+    (property "Reference" "#FLG0101" (id 0) (at 134.62 76.835 0)
+      (effects (font (size 1.27 1.27)) hide)
+    )
+    (property "Value" "PWR_FLAG" (id 1) (at 134.62 73.66 0))
+    (property "Footprint" "" (id 2) (at 134.62 78.74 0)
+      (effects (font (size 1.27 1.27)) hide)
+    )
+    (property "Datasheet" "~" (id 3) (at 134.62 78.74 0)
+      (effects (font (size 1.27 1.27)) hide)
+    )
+    (pin "1")
   )
   (symbol (lib_id "Device:R") (at 173.99 107.95 0) (unit 1)
@@
       (effects (font (size 1.27 1.27)) (justify left))
     )
-    (property "Footprint" "" (id 2) (at 172.212 107.95 90)
+    (property "Footprint" "Resistor_SMD:R_1210_3225Metric" (id 2) (at 172.212 107.95 90)
       (effects (font (size 1.27 1.27)) hide)
     )
     (property "Datasheet" "~" (id 3) (at 173.99 107.95 0)
+      (effects (font (size 1.27 1.27)) hide)
+    )
+    (property "LCSC" "C304148" (id 4) (at 173.99 107.95 0)
       (effects (font (size 1.27 1.27)) hide)
     )
@@
     (property "Reference" "J3" (id 0) (at 147.32 99.06 0))
     (property "Value" "JCON_M16_04Pin" (id 1) (at 147.32 101.6 0))
-    (property "Footprint" "" (id 2) (at 147.32 110.49 0)
+    (property "Footprint" "cacophony-footprints:jcon-4pin_m16" (id 2) (at 147.32 110.49 0)
       (effects (font (size 1.27 1.27)) hide)
     )
@@
   )
   (symbol_instances
+    (path "/dc03340c-c408-4ef7-9aa0-9d3fd2f5a1ad"
+      (reference "#FLG0101") (unit 1) (value "PWR_FLAG") (footprint "")
+    )
+    (path "/494dc53c-5b9d-4f88-a780-ac1d1fbedaeb"
+      (reference "#FLG0102") (unit 1) (value "PWR_FLAG") (footprint "")
+    )
     (path "/1e7f0642-e8b7-467b-9cc8-e6c2baa46f90"
       (reference "#PWR0101") (unit 1) (value "+12V") (footprint "")
@@
       (reference "#PWR0105") (unit 1) (value "+12V") (footprint "")
     )
+    (path "/aa0ea218-06c4-458d-bad5-081b15bfde23"
+      (reference "#PWR0106") (unit 1) (value "+12V") (footprint "")
+    )
+    (path "/328717f0-bfa9-4b3a-93ac-490f80c12b49"
+      (reference "#PWR0107") (unit 1) (value "GND") (footprint "")
+    )
     (path "/1fdde5ee-a840-414d-8817-7833102ccbb6"
-      (reference "J1") (unit 1) (value "JCON_M12_02Pin") (footprint "")
+      (reference "J1") (unit 1) (value "JCON_M12_02Pin") (footprint "cacophony-footprints:jcon-2pin-m12")
     )
     (path "/1f42909f-5948-4f99-a4c5-67d170866d51"
@@
     )
     (path "/e36b8bf1-a39c-40b7-8859-11056348a983"
-      (reference "J3") (unit 1) (value "JCON_M16_04Pin") (footprint "")
+      (reference "J3") (unit 1) (value "JCON_M16_04Pin") (footprint "cacophony-footprints:jcon-4pin_m16")
     )
     (path "/e26e29af-c0b7-4e16-9f97-67468309483b"
-      (reference "R1") (unit 1) (value "2M") (footprint "")
+      (reference "R1") (unit 1) (value "2M") (footprint "Resistor_SMD:R_1210_3225Metric")
     )
     (path "/334f7704-fc49-477d-b898-35fa373b0081"
-      (reference "R2") (unit 1) (value "150k") (footprint "")
+      (reference "R2") (unit 1) (value "150k") (footprint "Resistor_SMD:R_0805_2012Metric")
     )
     (path "/8c4cd8e5-35ba-4c86-9164-254b6e3c601a"
-      (reference "R?") (unit 1) (value "22k") (footprint "")
-    )
-  )
+      (reference "R3") (unit 1) (value "22k") (footprint "Resistor_SMD:R_0805_2012Metric")
+    )
+  )

Commit message: WIP
Parts:
- removed J2: Conn_01x05, Connector_JST:JST_XA_S05B-XASK-1_1x05_P2.50mm_Horizontal, symbol Connector_Generic:Conn_01x05
- added C101, C102, C103, C104, C106, C107: 22uF, Capacitor_SMD:C_0805_2012Metric, symbol Device:C
- added C105, C108: 220uF, Capacitor_SMD:CP_Elec_8x10, symbol Device:C_Polarized
- added C109, C110, C111, C112, C119, C120: 1nF, Capacitor_SMD:C_0402_1005Metric, symbol Device:C_Small
- added C113, C114: 47pF, Capacitor_SMD:C_0402_1005Metric, symbol Device:C_Small
- added C115, C116: 10nF, Capacitor_SMD:C_0402_1005Metric, symbol Device:C_Small
- added C117, C118: 100nF, Capacitor_SMD:C_0402_1005Metric, symbol Device:C_Small
- added C121, C122, C123, C124, C125, C126, C127, C128: 22uF, Capacitor_SMD:C_0603_1608Metric, symbol Device:C
- added D101: D_Zener, cacophony-footprints:LL-34_L3.5-W1.5-RD, symbol Device:D_Zener
- added D102, D103: D_Shockley, Diode_SMD:D_SMA, symbol Device:D_Shockley
- added J103: Conn_02x04_Odd_Even, cacophony-library:HDR-TH_8P-P2.54-H-F-R2-C4-S2.54-W10.2, symbol Connector_Generic:Conn_02x04_Odd_Even
- added L101, L102: 6.8uF, cacophony-footprints:IND-SMD_L8.0-W8.0_1217AS, symbol Device:L
- added Q101: Q_PMOS_GSD, Package_TO_SOT_SMD:SOT-23, symbol Device:Q_PMOS_GSD
- added R104, R110, R112: 100k, Resistor_SMD:R_0402_1005Metric, symbol Device:R
- added R105, R106: 33k, Resistor_SMD:R_0402_1005Metric, symbol Device:R
- added R107: 150k, Resistor_SMD:R_0402_1005Metric, symbol Device:R
- added R108, R111: 22k, Resistor_SMD:R_0402_1005Metric, symbol Device:R
- added R109: 10k, Resistor_SMD:R_0402_1005Metric, symbol Device:R
- added U101, U102: TPS54331, Package_SO:SO-8_3.9x4.9mm_P1.27mm, symbol cacophony-symbols:TPS54331
- renumbered J1 to J101, J3 to J102, R1 to R101, R2 to R102, R3 to R103
Connections:
- net +12V: now also C101.1, C102.1, C103.1, C104.1, C105.1, C106.1, C107.1, C108.1, C109.1, C110.1, D101.1 (K), Q101.2 (S), U101.2 (VIN), U102.2 (VIN); no longer J102.2
- net Batt_sense: now also J103.7 (Pin_7)
- net GND: now also C101.2, C102.2, C103.2, C104.2, C105.2, C106.2, C107.2, C108.2, C109.2, C110.2, C111.2, C112.2, C113.2, C114.2, C115.2, C116.2, C119.2, C120.2, C121.2, C122.2, C123.2, C124.2, C125.2, C126.2, C127.2, C128.2, D102.2 (A), D103.2 (A), J103.2 (Pin_2), J103.8 (Pin_8), R104.2, R107.1, R109.2, R111.1, U101.7 (GND), U102.7 (GND)
- net Speaker+: now also J103.1 (Pin_1)
- net Speaker-: now also J103.3 (Pin_3)
- new net: R107.2, R110.2, R111.2, U101.5 (VSENSE)
- new net: D101.2 (A), Q101.1 (G), R104.1
- new net: C117.1, U101.1 (BOOT)
- new net: C113.1, R105.1, U101.6 (COMP)
- new net: R108.2, R112.2, U102.5 (VSENSE)
- new net: C116.1, U102.4 (SS)
- new net: C114.1, R106.1, U102.6 (COMP)
- new net: C112.1, R106.2
- new net: R108.1, R109.1
- new net: C115.1, U101.4 (SS)
- new net: C111.1, R105.2
- new net: C118.1, U102.1 (BOOT)
- new net +3V3: C120.1, C122.1, C124.1, C126.1, C128.1, J103.6 (Pin_6), L102.2, R112.1
- new net +5V: C119.1, C121.1, C123.1, C125.1, C127.1, J103.4 (Pin_4), L101.2, R110.1
- new net 5V_EN: J103.5 (Pin_5), U101.3 (EN)
- new net SW_3V3: C118.2, D103.1 (K), L102.1, U102.8 (PH)
- new net SW_5V: C117.2, D102.1 (K), L101.1, U101.8 (PH)
- new net VIN: J102.2, Q101.3 (D)
- no-connect marks 0 -> 1
Other:
- note added: "- C239344, C92271: female, 2.54 - C239355: angled, female, 2.54,"
- note added: "TODO: - Check the pinout of plugs - Check size of pins on plugs - Change Capacitors to something that has smaller leakage current. - C178503"
- note removed: "TODO: - Check the pinout of plugs - Check size of pins on plugs"
- moved on the sheet: J101, J102, R101, R102, R103

Commit message: WIP 2
Connections:
- net +3V3: now also J103.4 (Pin_4); no longer J103.6 (Pin_6)
- net +5V: now also J103.6 (Pin_6); no longer J103.4 (Pin_4)
- net 5V_EN: now also J103.3 (Pin_3); no longer J103.5 (Pin_5)
- net Batt_sense: now also J103.1 (Pin_1); no longer J103.7 (Pin_7)
- net Speaker+: now also J103.7 (Pin_7); no longer J103.1 (Pin_1)
- net Speaker-: now also J103.5 (Pin_5); no longer J103.3 (Pin_3)
Changed lines of the file:
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@@
     (effects (font (size 1.27 1.27)) (justify left bottom))
   )
-  (label "Speaker+" (at 43.18 179.07 0)
+  (label "Speaker+" (at 43.18 186.69 0)
     (effects (font (size 1.27 1.27)) (justify left bottom))
   )
-  (label "Batt_sense" (at 43.18 186.69 0)
+  (label "Batt_sense" (at 43.18 179.07 0)
     (effects (font (size 1.27 1.27)) (justify left bottom))
   )
@@
     (effects (font (size 1.27 1.27)) (justify left bottom))
   )
-  (label "5V_EN" (at 43.18 184.15 0)
+  (label "5V_EN" (at 43.18 181.61 0)
     (effects (font (size 1.27 1.27)) (justify left bottom))
   )
@@
     (effects (font (size 1.27 1.27)) (justify right bottom))
   )
-  (label "Speaker-" (at 43.18 181.61 0)
+  (label "Speaker-" (at 43.18 184.15 0)
     (effects (font (size 1.27 1.27)) (justify left bottom))
   )
@@
     (pin "2")
   )
-  (symbol (lib_id "power:+5V") (at 24.13 180.34 0) (unit 1)
-    (in_bom yes) (on_board yes) (fields_autoplaced)
-    (property "Reference" "#PWR0102" (id 0) (at 24.13 184.15 0)
-      (effects (font (size 1.27 1.27)) hide)
-    )
-    (property "Value" "+5V" (id 1) (at 24.13 175.26 0))
-    (property "Footprint" "" (id 2) (at 24.13 180.34 0)
-      (effects (font (size 1.27 1.27)) hide)
-    )
-    (property "Datasheet" "" (id 3) (at 24.13 180.34 0)
+  (symbol (lib_id "power:+5V") (at 17.78 180.34 0) (unit 1)
+    (in_bom yes) (on_board yes) (fields_autoplaced)
+    (property "Reference" "#PWR0102" (id 0) (at 17.78 184.15 0)
+      (effects (font (size 1.27 1.27)) hide)
+    )
+    (property "Value" "+5V" (id 1) (at 17.78 175.26 0))
+    (property "Footprint" "" (id 2) (at 17.78 180.34 0)
+      (effects (font (size 1.27 1.27)) hide)
+    )
+    (property "Datasheet" "" (id 3) (at 17.78 180.34 0)
       (effects (font (size 1.27 1.27)) hide)
     )
@@
     (pin "2")
   )
-  (symbol (lib_id "power:+3V3") (at 17.78 180.34 0) (unit 1)
-    (in_bom yes) (on_board yes) (fields_autoplaced)
-    (property "Reference" "#PWR0104" (id 0) (at 17.78 184.15 0)
-      (effects (font (size 1.27 1.27)) hide)
-    )
-    (property "Value" "+3V3" (id 1) (at 17.78 175.26 0))
-    (property "Footprint" "" (id 2) (at 17.78 180.34 0)
-      (effects (font (size 1.27 1.27)) hide)
-    )
-    (property "Datasheet" "" (id 3) (at 17.78 180.34 0)
-      (effects (font (size 1.27 1.27)) hide)
-    )
+  (symbol (lib_id "power:+3V3") (at 24.13 180.34 0) (unit 1)
+    (in_bom yes) (on_board yes) (fields_autoplaced)
+    (property "Reference" "#PWR0104" (id 0) (at 24.13 184.15 0)
+      (effects (font (size 1.27 1.27)) hide)
+    )
+    (property "Value" "+3V3" (id 1) (at 24.13 175.26 0))
+    (property "Footprint" "" (id 2) (at 24.13 180.34 0)
+      (effects (font (size 1.27 1.27)) hide)
+    )
+    (property "Datasheet" "" (id 3) (at 24.13 180.34 0)
+      (effects (font (size 1.27 1.27)) hide)
+    )
