File: usb-adapter/usb-adapter.kicad_sch (KiCad schematic)
At the start: 2 parts

Commit message: WIP
Parts:
- removed J?: USB_A, symbol Connector:USB_A
- added J1: Conn_01x02, Connector_PinSocket_2.54mm:PinSocket_1x02_P2.54mm_Vertical, symbol Connector_Generic:Conn_01x02
- added USB1: FUS420-MSBK6M, cacophony-library:MICRO-USB-SMD_FUS420-MSBK6M, symbol cacophony-library:FUS420-MSBK6M
- J2: renamed from J?; footprint Connector_PinHeader_1.00mm:PinHeader_1x03_P1.00mm_Vertical -> Connector_PinSocket_2.54mm:PinSocket_1x03_P2.54mm_Vertical
Connections:
- net GND: now also USB1.5
- net D+: now reaches J2.2 (Pin_2)
- net D+: now also USB1.3
- net D-: now reaches J2.3 (Pin_3)
- net D-: now also USB1.2
- new net ID: J1.2 (Pin_2), USB1.4
- new net VCC: J1.1 (Pin_1), USB1.1
- no-connect marks 1 -> 4
Changed lines of the file:
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@@
 (kicad_sch (version 20211123) (generator eeschema)
   (paper "A4")
-  (junction (at 105.41 93.98) (diameter 0) (color 0 0 0 0)
-  )
-  (no_connect (at 115.57 78.74))
+  (no_connect (at 113.03 57.15))
+  (no_connect (at 113.03 59.69))
+  (no_connect (at 113.03 54.61))
+  (no_connect (at 113.03 52.07))
   (wire (pts (xy 123.19 88.9) (xy 123.19 90.17))
     (stroke (width 0) (type default) (color 0 0 0 0))
   )
-  (wire (pts (xy 105.41 95.25) (xy 105.41 93.98))
+  (wire (pts (xy 97.79 60.96) (xy 100.33 60.96))
     (stroke (width 0) (type default) (color 0 0 0 0))
   )
-  (wire (pts (xy 105.41 93.98) (xy 107.95 93.98))
+  (wire (pts (xy 97.79 62.23) (xy 97.79 60.96))
+    (stroke (width 0) (type default) (color 0 0 0 0))
+  )
+  (wire (pts (xy 99.06 58.42) (xy 100.33 58.42))
+    (stroke (width 0) (type default) (color 0 0 0 0))
+  )
+  (wire (pts (xy 99.06 50.8) (xy 100.33 50.8))
+    (stroke (width 0) (type default) (color 0 0 0 0))
+  )
+  (wire (pts (xy 99.06 53.34) (xy 100.33 53.34))
     (stroke (width 0) (type default) (color 0 0 0 0))
   )
@@
     (stroke (width 0) (type default) (color 0 0 0 0))
   )
+  (wire (pts (xy 99.06 55.88) (xy 100.33 55.88))
+    (stroke (width 0) (type default) (color 0 0 0 0))
+  )
   (wire (pts (xy 115.57 86.36) (xy 123.19 86.36))
     (stroke (width 0) (type default) (color 0 0 0 0))
   )
-  (symbol (lib_id "Connector:USB_A") (at 107.95 83.82 0) (unit 1)
+  (label "VCC" (at 95.25 102.87 180)
+    (effects (font (size 1.27 1.27)) (justify right bottom))
+  )
+  (label "D+" (at 115.57 86.36 180)
+    (effects (font (size 1.27 1.27)) (justify right bottom))
+  )
+  (label "D-" (at 115.57 83.82 180)
+    (effects (font (size 1.27 1.27)) (justify right bottom))
+  )
+  (label "ID" (at 95.25 105.41 180)
+    (effects (font (size 1.27 1.27)) (justify right bottom))
+  )
+  (label "D+" (at 99.06 55.88 180)
+    (effects (font (size 1.27 1.27)) (justify right bottom))
+  )
+  (label "D-" (at 99.06 53.34 180)
+    (effects (font (size 1.27 1.27)) (justify right bottom))
+  )
+  (label "VCC" (at 99.06 50.8 180)
+    (effects (font (size 1.27 1.27)) (justify right bottom))
+  )
+  (label "ID" (at 99.06 58.42 180)
+    (effects (font (size 1.27 1.27)) (justify right bottom))
+  )
+  (symbol (lib_name "GND_1") (lib_id "power:GND") (at 97.79 62.23 0) (unit 1)
     (in_bom yes) (on_board yes) (fields_autoplaced)
-    (property "Reference" "J?" (id 0) (at 107.95 71.12 0))
-    (property "Value" "USB_A" (id 1) (at 107.95 73.66 0))
-    (property "Footprint" "" (id 2) (at 111.76 85.09 0)
+    (property "Reference" "#PWR0101" (id 0) (at 97.79 68.58 0)
       (effects (font (size 1.27 1.27)) hide)
     )
-    (property "Datasheet" " ~" (id 3) (at 111.76 85.09 0)
+    (property "Value" "GND" (id 1) (at 97.79 67.31 0))
+    (property "Footprint" "" (id 2) (at 97.79 62.23 0)
+      (effects (font (size 1.27 1.27)) hide)
+    )
+    (property "Datasheet" "" (id 3) (at 97.79 62.23 0)
       (effects (font (size 1.27 1.27)) hide)
     )
     (pin "1")
-    (pin "2")
-    (pin "3")
-    (pin "4")
-    (pin "5")
   )
   (symbol (lib_id "power:GND") (at 123.19 90.17 0) (unit 1)
     (in_bom yes) (on_board yes) (fields_autoplaced)
-    (property "Reference" "#PWR?" (id 0) (at 123.19 96.52 0)
+    (property "Reference" "#PWR0102" (id 0) (at 123.19 96.52 0)
       (effects (font (size 1.27 1.27)) hide)
     )
@@
     (pin "1")
   )
-  (symbol (lib_id "power:GND") (at 105.41 95.25 0) (unit 1)
+  (symbol (lib_id "cacophony-library:FUS420-MSBK6M") (at 106.68 55.88 0) (unit 1)
     (in_bom yes) (on_board yes) (fields_autoplaced)
-    (property "Reference" "#PWR?" (id 0) (at 105.41 101.6 0)
+    (property "Reference" "USB1" (id 0) (at 106.68 43.18 0))
+    (property "Value" "FUS420-MSBK6M" (id 1) (at 106.68 45.72 0))
+    (property "Footprint" "cacophony-library:MICRO-USB-SMD_FUS420-MSBK6M" (id 2) (at 106.68 68.58 0)
       (effects (font (size 1.27 1.27)) hide)
     )
-    (property "Value" "GND" (id 1) (at 105.41 100.33 0))
-    (property "Footprint" "" (id 2) (at 105.41 95.25 0)
+    (property "Datasheet" "" (id 3) (at 106.68 55.88 0)
       (effects (font (size 1.27 1.27)) hide)
     )
-    (property "Datasheet" "" (id 3) (at 105.41 95.25 0)
+    (property "Manufacturer" "TXGA(特思嘉)" (id 4) (at 106.68 71.12 0)
+      (effects (font (size 1.27 1.27)) hide)
+    )
+    (property "LCSC Part" "C2833885" (id 5) (at 106.68 73.66 0)
+      (effects (font (size 1.27 1.27)) hide)
+    )
+    (property "JLC Part" "Extended Part" (id 6) (at 106.68 76.2 0)
       (effects (font (size 1.27 1.27)) hide)
     )
     (pin "1")
+    (pin "12")
+    (pin "13")
+    (pin "2")
+    (pin "3")
+    (pin "4")
+    (pin "5")
+    (pin "8")
+    (pin "9")
   )
   (symbol (lib_id "Connector_Generic:Conn_01x03") (at 128.27 86.36 0) (mirror x) (unit 1)
     (in_bom yes) (on_board yes) (fields_autoplaced)
-    (property "Reference" "J?" (id 0) (at 130.81 87.6301 0)
+    (property "Reference" "J2" (id 0) (at 130.81 87.6301 0)
       (effects (font (size 1.27 1.27)) (justify left))
     )
@@
       (effects (font (size 1.27 1.27)) (justify left))
     )
-    (property "Footprint" "Connector_PinHeader_1.00mm:PinHeader_1x03_P1.00mm_Vertical" (id 2) (at 128.27 86.36 0)
+    (property "Footprint" "Connector_PinSocket_2.54mm:PinSocket_1x03_P2.54mm_Vertical" (id 2) (at 128.27 86.36 0)
       (effects (font (size 1.27 1.27)) hide)
     )
@@
     (pin "3")
   )
+  (symbol (lib_id "Connector_Generic:Conn_01x02") (at 100.33 102.87 0) (unit 1)
+    (in_bom yes) (on_board yes) (fields_autoplaced)
+    (property "Reference" "J1" (id 0) (at 102.87 102.8699 0)
+      (effects (font (size 1.27 1.27)) (justify left))
+    )
+    (property "Value" "Conn_01x02" (id 1) (at 102.87 105.4099 0)
+      (effects (font (size 1.27 1.27)) (justify left))
+    )
+    (property "Footprint" "Connector_PinSocket_2.54mm:PinSocket_1x02_P2.54mm_Vertical" (id 2) (at 100.33 102.87 0)
+      (effects (font (size 1.27 1.27)) hide)
+    )
+    (property "Datasheet" "~" (id 3) (at 100.33 102.87 0)
+      (effects (font (size 1.27 1.27)) hide)
+    )
+    (pin "1")
+    (pin "2")
+  )
   (sheet_instances
     (path "/" (page "1"))
   )
   (symbol_instances
+    (path "/37e139ac-81ed-40ee-87f6-97ccf04a4efa"
+      (reference "#PWR0101") (unit 1) (value "GND") (footprint "")
+    )
     (path "/65262092-5ba5-4f90-93d8-e8a529b0c7de"
-      (reference "#PWR?") (unit 1) (value "GND") (footprint "")
+      (reference "#PWR0102") (unit 1) (value "GND") (footprint "")
     )
-    (path "/8012604c-7d40-44ac-bb83-566ca31a2b69"
-      (reference "#PWR?") (unit 1) (value "GND") (footprint "")
-    )
-    (path "/4fd563b1-8bba-454c-bb2d-cb692d1b4429"
-      (reference "J?") (unit 1) (value "USB_A") (footprint "")
+    (path "/c73cdd4f-072d-4769-8d9f-072202583139"
+      (reference "J1") (unit 1) (value "Conn_01x02") (footprint "Connector_PinSocket_2.54mm:PinSocket_1x02_P2.54mm_Vertical")
     )
     (path "/bbd3bb83-d701-4961-80de-d4cc4d63997d"
-      (reference "J?") (unit 1) (value "Conn_01x03") (footprint "Connector_PinHeader_1.00mm:PinHeader_1x03_P1.00mm_Vertical")
+      (reference "J2") (unit 1) (value "Conn_01x03") (footprint "Connector_PinSocket_2.54mm:PinSocket_1x03_P2.54mm_Vertical")
+    )
+    (path "/70ea6019-3ebb-40d9-a001-2a00af2c4eb4"
+      (reference "USB1") (unit 1) (value "FUS420-MSBK6M") (footprint "cacophony-library:MICRO-USB-SMD_FUS420-MSBK6M")
     )
   )
