File: tc2-main-pcb/tc2-main-pcb.kicad_pcb (KiCad board)
At the start: 4 copper layers, 57.5 x 70.4 mm, 139 parts, among them J1 Screw_Terminal_01x01, J3 Conn_02x04_Odd_Even, J4 Raspberry_Pi_2_3, J5 Screw_Terminal_01x01, J6 Screw_Terminal_01x01, J7 Screw_Terminal_01x01, J8 Conn_01x03, SW2 K2-6639SP-M4SC-04, U1 ATtiny1616-M, U10 TD6810, U11 TD6810, U12 SIM7600G-H-M.2, U13 MAX98357, U14 SPH0645LM4H, U15 ME6211, U2 W25Q128JVS, U3 RP2040, U4 MT29F2G01ABAGDWB-IT, U5 SHT30-DIS, U6 PCF8563T, U7 ME6216A28XG, U8 Flir_LEPTON, U9 3N25000G33YC, Y1 Crystal_GND24, Y2 Crystal

Commit message: Clean up of files and updated drawings for PCBs
Parts:
- removed ?: , 
- removed the J7 at (137.9, 83.3)
- removed the J7 at (106.0, 70.9)
- removed the J7 at (117.0, 71.0)
- added H2: MountingHole, cacophony-library:Mouning_Hole_M3, F.Cu at (92.4, 54.9)
- added J7: Screw_Terminal_01x01, cacophony-library:SMD_BD4.4-L4.4-D2.8, F.Cu at (136.8, 74.9)
- added J9: Conn_02x03_Odd_Even, cacophony-library:mic-pcb, F.Cu at (110.9, 66.5)
- added REF**: MountingHole_2.1mm, MountingHole:MountingHole_2.1mm, F.Cu at (93.8, 62.1)
- added REF**: MountingHole_2.1mm, MountingHole:MountingHole_2.1mm, F.Cu at (116.9, 66.7)
- J3: footprint cacophony-library:power-pcb -> cacophony-library:power-pcb-3
- moved J3 10.8 mm to (123.1, 135.2), turned to 0 degrees
Connections:
- net Net-(J4-MOSI0/GPIO10) renamed /Raspberry_Pi/RPI_SPI_MOSI_
- net Net-(J4-SCLK0/GPIO11) renamed /Raspberry_Pi/RPI_SPI_SCLK_
- net Net-(J4-~{CE0}/GPIO8) renamed /Raspberry_Pi/RPI_SPI_CS_
Routing:
- net 5V_EN: track 31.4 -> 11.4 mm
- net BATT_SENSE: track 33.2 -> 15.3 mm
- net SPEAKER_-: track 16.9 -> 0.00 mm
- net SPEAKER_+: track 14.3 -> 1.55 mm
Other:
- board size 57.5 x 70.4 mm -> 64.5 x 88.7 mm

Commit message: Version 2 WIP
Parts:
- removed C38: 220nF, Capacitor_SMD:C_0402_1005Metric
- removed C39: 12pF, Capacitor_SMD:C_0402_1005Metric
- removed C43: 1uF, Capacitor_SMD:C_0402_1005Metric
- removed the H2 at (92.4, 54.9)
- removed REF** (x2): MountingHole_2.1mm, MountingHole:MountingHole_2.1mm
- removed TP10, TP11, TP4: TestPoint, cacophony-library:TP
- removed U14: SPH0645LM4H, cacophony-library:MIC_SPH0645LM4H-B
- removed U15: ME6211, Package_TO_SOT_SMD:SOT-23-5
- added H4: MountingHole, cacophony-library:Mouning_Hole_M3, F.Cu at (92.0, 53.9)
- added H5: MountingHole, MountingHole:MountingHole_2.2mm_M2, F.Cu at (92.0, 61.0)
- added H6: MountingHole, MountingHole:MountingHole_2.2mm_M2, F.Cu at (115.0, 67.0)
- added R35: 100k, Resistor_SMD:R_0402_1005Metric, F.Cu at (106.4, 78.1)
- added TP18: TestPoint, cacophony-library:TP, F.Cu at (142.1, 83.4)
- added TP19: TestPoint, cacophony-library:TP, F.Cu at (142.1, 85.1)
- added TP20: TestPoint, cacophony-library:TP, F.Cu at (142.1, 86.9)
- J3, R32: moved to B.Cu
- R28, TP7: moved to F.Cu
- moved R28 40.0 mm to (107.4, 78.2), turned to 90 degrees
- moved TP14 30.5 mm to (142.1, 81.6), turned to 0 degrees
- moved R31 15.9 mm to (97.3, 96.2)
- moved TP13 13.1 mm to (107.4, 79.5), turned to 90 degrees
- moved TP47 12.5 mm to (115.5, 73.9), turned to 90 degrees
- moved TP9 12.5 mm to (117.2, 73.9), turned to 90 degrees
- moved TP46 12.4 mm to (116.4, 73.9), turned to 90 degrees
- moved TP44 12.3 mm to (107.7, 82.2), turned to 90 degrees
- moved TP12 12.2 mm to (108.4, 79.3), turned to 90 degrees
- moved C12 11.9 mm to (109.8, 77.4), turned to 90 degrees
- moved C3 11.4 mm to (110.2, 87.7), turned to 90 degrees
- moved R2 10.8 mm to (109.5, 79.4), turned to -90 degrees
- moved R9 10.8 mm to (108.8, 82.9), turned to 180 degrees
- moved R34 10.8 mm to (97.9, 111.1), turned to 90 degrees
- moved SW2 10.8 mm to (133.7, 126.5)
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Connections:
- net Net-(U3-GPIO16) renamed /GPIO16
- net Net-(U3-GPIO17) renamed /GPIO17
- net Net-(U3-GPIO2) renamed /GPIO2
- net Net-(U3-GPIO3) renamed /GPIO3
- J3 pad 5: SPEAKER_- -> SPEAKER_+
- J3 pad 7: SPEAKER_+ -> SPEAKER_-
- J4 pad 36: unconnected-(J4-GPIO16-Pad36) -> ~{WAKEUP_PING}
- J4 pad 38: I2S_DIN -> unconnected-(J4-GPIO20/MOSI1-Pad38)
- J9 pad 1: unconnected-(J9-Pin_1-Pad1) -> PDM_CLOCK
- J9 pad 2: unconnected-(J9-Pin_2-Pad2) -> GND
- J9 pad 3: unconnected-(J9-Pin_3-Pad3) -> GND
- J9 pad 4: unconnected-(J9-Pin_4-Pad4) -> +3V3
- J9 pad 5: unconnected-(J9-Pin_5-Pad5) -> PDM_DATA
- J9 pad 6: unconnected-(J9-Pin_6-Pad6) -> GND
- R28 pad 1: Net-(U14-DATA) -> /PDM_CLOCK_
- R28 pad 2: I2S_DIN -> PDM_CLOCK
- R3 pad 1: Net-(U1-PA3) -> Net-(U1-PA4)
- R4 pad 1: Net-(U1-PA4) -> Net-(U1-PA3)
- SW2 pad 1: Net-(U1-PA7) -> Net-(U1-PA6)
- TP14 pad 1: Net-(U3-GPIO4) -> GND
- TP6 pad 1: Net-(U1-PB4) -> Net-(U1-PA7)
- TP7 pad 1: Net-(U1-PB5) -> Net-(U1-PC0)
- U1 pad 10: Net-(U1-PB4) -> RTC_BT_SENSE
- U1 pad 12: Net-(U1-PB2) -> ~{WAKEUP_PING}
- U1 pad 15: BATT_SENSE -> Net-(U1-PC0)
- U1 pad 7: RTC_BT_SENSE -> Net-(U1-PA6)
- U1 pad 9: Net-(U1-PB5) -> BATT_SENSE
- U3 pad 2: Net-(U3-GPIO0) -> PDM_DATA
- U3 pad 3: Net-(U3-GPIO1) -> /PDM_CLOCK_
- U3 pad 39: LEPTON_PWR_DWN_L -> LEPTON_CLK_EN
- U3 pad 40: LEPTON_RESET_L -> LEPTON_PWR_DWN_L
- U3 pad 41: LEPTON_CLK_EN -> LEPTON_RESET_L
- U3 pad 6: Net-(U3-GPIO4) -> ~{WAKEUP_PING}
Routing:
- net ~{WAKEUP_PING}: track 0.00 -> 67.1 mm, vias 0 -> 4
- net I2S_DIN: track 54.8 -> 0.00 mm, vias 2 -> 0
- net Net-(U1-PA5): track 39.2 -> 62.1 mm, vias 0 -> 2
- net Net-(U1-PA6): track 0.00 -> 22.7 mm, vias 0 -> 1
- net Net-(U1-PA4): track 38.5 -> 58.9 mm
- net SPEAKER_-: track 0.00 -> 19.5 mm, vias 0 -> 4
- net 5V_EN: track 11.4 -> 30.3 mm, vias 3 -> 2
- net Net-(U1-PA3): track 36.6 -> 54.9 mm
- net LEPTON_CLK_EN: track 35.0 -> 17.3 mm
- net LEPTON_MASTER_CLK: track 35.8 -> 18.8 mm
- net SPEAKER_+: track 1.55 -> 17.3 mm, vias 0 -> 4
- net LEPTON_PWR_DWN_L: track 38.9 -> 23.5 mm
- net LEPTON_I2C_SCL: track 36.1 -> 20.9 mm
- net LEPTON_I2C_SDA: track 35.0 -> 20.0 mm
- net LEPTON_RESET_L: track 39.9 -> 25.1 mm
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- added copper zone on F.Cu, net +5V
- added copper zone on F.Cu, net SPEAKER_+
- added copper zone on F.Cu, net SPEAKER_-
Other:
- board size 64.5 x 88.7 mm -> 64.5 x 89 mm

Commit message: Thermal camera V2 WIP
Parts:
- removed R13: 100k, Resistor_SMD:R_0402_1005Metric
- removed U13: MAX98357, Package_DFN_QFN:TQFN-16-1EP_3x3mm_P0.5mm_EP1.6x1.6mm
- added U14: MAX98357AEWL+T, cacophony-library:WLP-9_L1.4-W1.3-P0.40-R3-C3-BR, F.Cu at (112.7, 127.1)
- moved C29 2.30 mm to (110.9, 126.8), turned to 0 degrees
- moved R12 1.71 mm to (110.4, 125.5), turned to 0 degrees
- moved C28 1.06 mm to (110.4, 128.0)
Connections:
- C29 pad 1: +5V -> GND
- C29 pad 2: GND -> +5V
- J3 pad 5: SPEAKER_+ -> SPEAKER_-
- J3 pad 7: SPEAKER_- -> SPEAKER_+
Routing:
- net GND: track 80.8 -> 73.5 mm, vias 115 -> 121
- net I2S_BCLK: track 24.3 -> 30.9 mm, vias 2 -> 4
- net SPEAKER_+: track 17.3 -> 23.4 mm
- net I2S_DOUT: track 62.9 -> 68.9 mm, vias 2 -> 4
- net I2S_LRCLK: track 50.7 -> 55.2 mm, vias 2 -> 4
- net Net-(U14-~{SD_MODE}): track 1.60 -> 4.28 mm, vias 0 -> 2
- net +5V: track 0.00 -> 2.17 mm, vias 4 -> 6
- net Net-(U13-GAIN_SLOT): track 1.45 -> 0.00 mm
- net SPEAKER_-: track 19.5 -> 20.4 mm
- net SPEAKER_SD_MODE: track 16.3 -> 15.4 mm
- removed copper zone on F.Cu, net SPEAKER_+
- removed copper zone on F.Cu, net SPEAKER_-

Commit message: P2 milestone
Parts:
- removed Card1: SIM-Nano, cacophony-library:SIM-SMD_SMN-304
- removed D4: SMF05CT1G, cacophony-library:SOT-363_L2.0-W1.3-P0.65-LS2.1-BR
- removed H2: MountingHole, cacophony-library:Mouning_Hole_M3
- removed TP15, TP16, TP2, TP3, TP44, TP5, TP7: TestPoint, cacophony-library:TP
- removed U5: SHT30-DIS, Sensor_Humidity:Sensirion_DFN-8-1EP_2.5x2.5mm_P0.5mm_EP1.1x1.7mm
- added C38: 10uF, Capacitor_SMD:C_0603_1608Metric, F.Cu at (25.1, -23.3)
- added C39: 10uF, Capacitor_SMD:C_0603_1608Metric, B.Cu at (7.83, 6.35)
- added C43: 10uF, Capacitor_SMD:C_0603_1608Metric, F.Cu at (27.7, -24.2)
- added J10: Conn_02x06_Odd_Even, cacophony-library:power-pcb-3.1, B.Cu at (24.3, 35.3)
- added J11: Conn_01x08, cacophony-library:sim-usb-pcb, B.Cu at (51.7, -11.0)
- added J2: Conn_01x03, Connector_PinHeader_2.54mm:PinHeader_1x03_P2.54mm_Vertical, B.Cu at (-7.00, -0.87)
- added Q1: Q_PMOS_GSD, Package_TO_SOT_SMD:SOT-23, F.Cu at (27.7, -21.8)
- added R13: 100k, Resistor_SMD:R_0402_1005Metric, B.Cu at (32.8, -8.85)
- added R36: 100k, Resistor_SMD:R_0402_1005Metric, B.Cu at (32.8, -7.81)
- added R37: 1k, Resistor_SMD:R_0402_1005Metric, B.Cu at (-5.70, 16.6)
- added R38: 100k, Resistor_SMD:R_0402_1005Metric, F.Cu at (30.1, -21.8)
- added R39: 180R, Resistor_SMD:R_0402_1005Metric, B.Cu at (10.9, 6.22)
- added TP24: TestPoint_2Pole, cacophony-library:test-point-2p, F.Cu at (39.2, 30.3)
- added TP25: TestPoint_2Pole, cacophony-library:test-point-2p, F.Cu at (32.7, -6.68)
- added TP28: TestPoint_2Pole, cacophony-library:test-point-2p, F.Cu at (14.1, 29.1)
- added TP4: TestPoint_2Pole, cacophony-library:test-point-2p, F.Cu at (32.7, -2.88)
- added U13: AHT21, cacophony-library:SENSOR-SMD_L3.0-W3.0-P1.00-BR, B.Cu at (10.1, 3.46)
- added U15: 74HC4052, cacophony-library:SOP-16_L10.0-W3.9-P1.27-LS6.0-BL, F.Cu at (-7.46, 16.9)
- C17: value 220nF -> 1u
- C37: value 220nF -> 10uF; footprint Capacitor_SMD:C_0402_1005Metric -> Capacitor_SMD:C_0603_1608Metric; moved to F.Cu
- J3: value Conn_02x04_Odd_Even -> Conn_01x03; footprint cacophony-library:power-pcb-3 -> cacophony-library:JST_SH_BM03B-SRSS-TB_1x03-1MP_P1.00mm_Vertical
- J8: value Conn_01x03 -> Screw_Terminal_01x01; footprint Connector_PinHeader_2.54mm:PinHeader_1x03_P2.54mm_Vertical -> cacophony-library:SMTSO25
- R15: value 1k -> 100k; moved to B.Cu
- R3, R4, R5, TP1: moved to F.Cu
- SW2: footprint cacophony-library:KEY-SMD_4P-L6.0-W6.0-P3.90-LS9.0 -> cacophony-library:KEY-SMD_4P-L6.0-W6.0-P3.90_K2-6639SP-K4SC-04
- TP6: value TestPoint -> TestPoint_2Pole; footprint cacophony-library:TP -> cacophony-library:test-point-2p; moved to F.Cu
- TP8: value TestPoint -> TestPoint_2Pole; footprint cacophony-library:TP -> cacophony-library:test-point-2p
- moved J3 183.3 mm to (-8.30, 8.80)
- moved TP6 167.1 mm to (23.6, -23.3), turned to -90 degrees
- moved C37 164.5 mm to (-9.61, 23.2)
- moved H3 144.6 mm to (19.3, 21.2)
- moved R11 144.0 mm to (7.49, 5.12), turned to 180 degrees
- moved R25 143.5 mm to (32.9, 9.92), turned to 45 degrees
- moved C32 143.2 mm to (24.6, 11.1)
- moved C33 143.2 mm to (26.2, 11.1)
- moved C34 143.2 mm to (41.1, 11.1)
- moved C35 143.2 mm to (42.7, 11.1)
- moved C36 143.2 mm to (44.3, 11.1)
- moved R24 143.2 mm to (28.0, 12.2)
- moved U12 143.2 mm to (34.2, 17.5)
- moved J7 143.2 mm to (34.1, -24.3)
- moved R26 143.2 mm to (33.5, 10.7), turned to 45 degrees
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Connections:
- C10 pad 1: +3V3 -> +3V3_rp2040
- C11 pad 1: +3V3 -> +3V3_rp2040
- C12 pad 1: +3V3 -> +3V3_rp2040
- C13 pad 1: +3V3 -> +3V3_rp2040
- C14 pad 1: +3V3 -> +3V3_rp2040
- C15 pad 1: +3V3 -> +3V3_rp2040
- C16 pad 1: +3V3 -> +3V3_rp2040
- C17 pad 1: GND -> +3V3
- C17 pad 2: +3V3 -> GND
- C2 pad 1: +3V3 -> +3V3_rp2040
- C37 pad 1: GND -> +5V
- C37 pad 2: Net-(Card1-VCC) -> GND
- C8 pad 1: +3V3 -> +3V3_rp2040
- C9 pad 1: +3V3 -> +3V3_rp2040
- J3 pad 1: BATT_SENSE -> SW_CLK
- J3 pad 3: 5V_EN -> SWD
- J4 pad 10: ATtiny_RESET_UPDI -> RPI_RX
- J4 pad 13: unconnected-(J4-GPIO27-Pad13) -> ~{PI_SHUTDOWN}
- J4 pad 31: unconnected-(J4-GCLK2/GPIO6-Pad31) -> MUL_S0
- J4 pad 32: unconnected-(J4-PWM0/GPIO12-Pad32) -> MUL_S1
- J8 pad 1: GND -> unconnected-(J8-Pin_1-Pad1)
- R15 pad 1: ATtiny_RESET_UPDI -> ATTINY_TX
- R15 pad 2: Net-(J4-GPIO14/TXD) -> Net-(U1-PB2)
- R2 pad 1: +3V3 -> +3V3_rp2040
- R25 pad 2: Net-(Card1-RST) -> USIM_RST
- R26 pad 2: Net-(Card1-CLK) -> USIM_CLK
- R27 pad 2: Net-(Card1-I/O) -> USIM_DATA
- R9 pad 2: +3V3 -> +3V3_rp2040
- SW2 pad 2: GND -> unconnected-(SW2-Pad2)
- SW2 pad 4: unconnected-(SW2-Pad4) -> GND
- TP1 pad 1: Net-(U1-PC2) -> Net-(U1-PC3)
- TP6 pad 1: Net-(U1-PA7) -> GND
- TP8 pad 1: RUN -> GND
- U1 pad 11: Net-(U1-PB3) -> ATTINY_RX
- U1 pad 12: ~{WAKEUP_PING} -> Net-(U1-PB2)
- U1 pad 15: Net-(U1-PC0) -> ~{WAKEUP_PING}
- U1 pad 17: Net-(U1-PC2) -> EN_PERIPH_POWER
- U1 pad 20: Net-(U1-PA1) -> ~{EN_RP2040_POWER}
- U1 pad 8: Net-(U1-PA7) -> ~{PI_SHUTDOWN}
- U12 pad 36: Net-(Card1-VCC) -> USIM_VDD
- U2 pad 8: +3V3 -> +3V3_rp2040
- U3 pad 1: +3V3 -> +3V3_rp2040
- U3 pad 10: +3V3 -> +3V3_rp2040
- U3 pad 22: +3V3 -> +3V3_rp2040
- U3 pad 33: +3V3 -> +3V3_rp2040
- U3 pad 42: +3V3 -> +3V3_rp2040
- U3 pad 43: +3V3 -> +3V3_rp2040
- U3 pad 44: +3V3 -> +3V3_rp2040
- U3 pad 48: +3V3 -> +3V3_rp2040
- U3 pad 49: +3V3 -> +3V3_rp2040
- U4 pad 8: +3V3 -> +3V3_rp2040
Routing:
- net +3V3_rp2040: track 0.00 -> 78.6 mm, vias 0 -> 6
- net ~{EN_RP2040_POWER}: track 0.00 -> 55.3 mm, vias 0 -> 1
- net OUT_RX: track 0.00 -> 38.3 mm, vias 0 -> 1
- net EN_PERIPH_POWER: track 0.00 -> 38.1 mm, vias 0 -> 2
- net OUT_TX: track 0.00 -> 37.5 mm, vias 0 -> 1
- net MUL_S0: track 0.00 -> 37.0 mm, vias 0 -> 3
- net MUL_S1: track 0.00 -> 36.2 mm, vias 0 -> 3
- net Net-(Card1-VCC): track 35.5 -> 0.00 mm
- net Net-(Card1-CLK): track 35.3 -> 0.00 mm
- net ATTINY_RX: track 0.00 -> 34.7 mm, vias 0 -> 3
- net ATTINY_TX: track 0.00 -> 32.9 mm, vias 0 -> 3
- net USIM_RST: track 0.00 -> 28.4 mm
- net Net-(Card1-RST): track 28.1 -> 0.00 mm
- net USIM_CLK: track 0.00 -> 26.1 mm
- net USIM_VDD: track 0.00 -> 24.5 mm
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- added copper zone on F.Cu, net +3V3_rp2040
Other:
- board size 64.5 x 89 mm -> 65 x 89 mm
- board text added: "1V2"
- board text added: "2V8"
- board text added: "3V0"
- board text added: "3V3"
- board text added: "5V0"
- board text added: "CLK"
- board text added: "GND"
- board text added: "SWD"
- board text removed: "D+"
- board text removed: "D-"

Commit message: P3-Nov release
Parts:
- removed TP24, TP25, TP28: TestPoint_2Pole, cacophony-library:test-point-2p
- added C40: 12pF, Capacitor_SMD:C_0402_1005Metric, B.Cu at (41.5, 11.8)
- added C44: 12pF, Capacitor_SMD:C_0402_1005Metric, F.Cu at (18.5, 17.0)
- added C45: 220nF, Capacitor_SMD:C_0402_1005Metric, F.Cu at (34.7, 16.8)
- added C46: 12pF, Capacitor_SMD:C_0402_1005Metric, F.Cu at (29.9, 16.8)
- added C47: 220nF, Capacitor_SMD:C_0402_1005Metric, F.Cu at (29.0, 16.8)
- added C48: 220nF, Capacitor_SMD:C_0402_1005Metric, F.Cu at (16.2, 7.74)
- added C49: 22uF, Capacitor_SMD:C_0603_1608Metric, F.Cu at (35.9, 16.7)
- added C50: 220nF, Capacitor_SMD:C_0402_1005Metric, F.Cu at (3.68, 22.6)
- added C51: 220nF, Capacitor_SMD:C_0402_1005Metric, B.Cu at (24.3, 11.8)
- added C52: 22uF, Capacitor_SMD:C_0603_1608Metric, F.Cu at (37.3, 16.7)
- added C53: 22uF, Capacitor_SMD:C_0603_1608Metric, F.Cu at (38.8, 16.7)
- added C54: 22uF, Capacitor_SMD:C_0603_1608Metric, F.Cu at (26.4, 16.7)
- added C55: 22uF, Capacitor_SMD:C_0603_1608Metric, F.Cu at (27.8, 16.7)
- added C56: 12pF, Capacitor_SMD:C_0402_1005Metric, B.Cu at (21.0, 13.1)
- added C57: 22uF, Capacitor_SMD:C_0603_1608Metric, B.Cu at (27.8, 11.3)
- added C58: 22uF, Capacitor_SMD:C_0603_1608Metric, B.Cu at (25.4, 11.3)
- added C59: 22uF, Capacitor_SMD:C_0603_1608Metric, B.Cu at (23.1, 11.3)
- added C60: 22uF, Capacitor_SMD:C_0603_1608Metric, F.Cu at (40.2, 16.7)
- added C62: 22uF, Capacitor_SMD:C_0603_1608Metric, B.Cu at (17.1, 30.1)
- added C64: 22uF, Capacitor_SMD:C_0603_1608Metric, F.Cu at (23.1, 30.3)
- added C65: 22uF, Capacitor_SMD:C_0603_1608Metric, F.Cu at (30.1, 29.8)
- added C66: 22uF, Capacitor_SMD:C_0603_1608Metric, F.Cu at (30.1, 28.4)
- added FB1: FerriteBead, Inductor_SMD:L_0805_2012Metric, F.Cu at (41.8, 16.4)
- added L3: INDUCTOR, Inductor_SMD:L_1008_2520Metric, F.Cu at (32.3, 14.0)
- added R40: 10k, Resistor_SMD:R_0402_1005Metric, F.Cu at (18.5, 15.2)
- added R42: 1M, Resistor_SMD:R_0402_1005Metric, F.Cu at (35.1, 18.8)
- added R43: 1M, Resistor_SMD:R_0402_1005Metric, F.Cu at (37.5, 19.3)
- added R44: 100k, Resistor_SMD:R_0402_1005Metric, F.Cu at (29.9, 19.3)
- added R45: 150k, Resistor_SMD:R_0402_1005Metric, F.Cu at (35.1, 19.8)
- added R46: 1k, Resistor_SMD:R_0402_1005Metric, B.Cu at (18.2, 5.60)
- added R49: 10k, Resistor_SMD:R_0402_1005Metric, B.Cu at (21.0, 11.2)
- added TP10: TP_2P, cacophony-library:test-point-2p, F.Cu at (40.3, 27.1)
- added TP2: TestPoint, cacophony-library:TP, F.Cu at (22.9, 7.75)
- added TP3: TP_2P, cacophony-library:test-point-2p, F.Cu at (24.6, -23.6)
- added TP5: TP_2P, cacophony-library:test-point-2p, F.Cu at (38.2, -6.46)
- added U16: M24C02-WMN, Package_SO:SOIC-8_3.9x4.9mm_P1.27mm, F.Cu at (13.0, 6.46)
- added U17: PCA9515ADP,118, Package_SO:TSSOP-8_3x3mm_P0.65mm, F.Cu at (4.61, 20.2)
- added U5: TPS6302x, cacophony-library:VSON-14_L4.0-W3.0-P0.50-BL-EP_TI_DSJ, F.Cu at (32.3, 17.7)
- C32: value 10uF -> 12pF; footprint Capacitor_SMD:C_0603_1608Metric -> Capacitor_SMD:C_0402_1005Metric
- C33, C34, C35: value 10uF -> 22uF
- C36: value 10uF -> 220nF; footprint Capacitor_SMD:C_0603_1608Metric -> Capacitor_SMD:C_0402_1005Metric
- H1, H3, H4: footprint cacophony-library:Mouning_Hole_M3 -> cacophony-library:MountingHole_3.2mm_M3
- J2: value Conn_01x03 -> Screw_Terminal_01x01; footprint Connector_PinHeader_2.54mm:PinHeader_1x03_P2.54mm_Vertical -> cacophony-library:SMTSO25
- J4: footprint cacophony-library:RPI_HDR-SMD_40P-P2.54-V-F-R2-C20-S8.7-EH -> cacophony-library:HDR-SMD_40P-P2.54-V-F-R2-C20-LS8.2-EH
- J7: footprint cacophony-library:SMD_BD4.4-L4.4-D2.8 -> cacophony-library:M2_modem_mount_screw
- R15: value 100k -> 1k
- R35: value 100k -> 1k; moved to B.Cu
- TP1: value TestPoint -> TP_2P; footprint cacophony-library:TP -> cacophony-library:test-point-2p
- TP4, TP6, TP8: value TestPoint_2Pole -> TP_2P
- U15: footprint cacophony-library:SOP-16_L10.0-W3.9-P1.27-LS6.0-BL -> Package_SO:SOP-16_3.9x9.9mm_P1.27mm
- moved TP6 56.0 mm to (40.3, 30.1), turned to 180 degrees
- moved R5 39.1 mm to (21.7, 21.7), turned to -90 degrees
- moved R3 38.7 mm to (19.8, 21.7), turned to -90 degrees
- moved LED1 38.1 mm to (20.6, 23.9), turned to -90 degrees
- moved R4 38.0 mm to (20.8, 21.7), turned to -90 degrees
- moved R35 29.0 mm to (18.2, 4.66), turned to 180 degrees
- moved J2 29.0 mm to (0.00, -29.0)
- moved H3 27.6 mm to (-8.20, 24.0)
- moved H4 22.1 mm to (-8.20, -24.0)
- moved TP1 21.0 mm to (38.1, 14.4)
- moved C33 18.9 mm to (45.1, 11.3)
- moved R24 9.50 mm to (20.9, 18.5), turned to 90 degrees
- moved R36 8.25 mm to (29.0, -15.2)
- moved R13 8.16 mm to (29.0, -16.1)
- moved H5 6.02 mm to (-8.20, -33.0)
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Connections:
- net /PDM_CLOCK_ renamed /PDM_CLOCK_PHY
- net LED_B renamed ~{LED_B}
- net LED_G renamed ~{LED_G}
- net LED_R renamed ~{LED_R}
- net Net-(BT1-+) renamed /RTC_BATTERY
- net Net-(D3-K) renamed /RTC_VDD
- net Net-(U1-PA5) renamed /ATtiny1616/~{LED_R_PHY}
- net Net-(U13-VDD) renamed /AHT21_VDD
- net Net-(U4-~{HOLD}/IO3) renamed /MEM_~{HOLD}/IO3
- net Net-(U4-~{WP}/IO2) renamed /MEM_~{WP}/IO2
- net Net-(U6-CLKO) renamed /RTC_CLKO
- net Net-(U6-OSCI) renamed /RTC_OSCI
- net Net-(U6-OSCO) renamed /RTC_OSCO
- net RTC_BT_SENSE renamed RTC_BT_SENSE_PHY
- C32 pad 1: +3V3 -> GND
- C32 pad 2: GND -> +3V8
- C33 pad 1: +3V3 -> +3V8
- C34 pad 1: +3V3 -> +3V8
- C35 pad 1: +3V3 -> +3V8
- C36 pad 1: +3V3 -> GND
- C36 pad 2: GND -> +3V8
- J10 pad 1: GND -> 5V_EN
- J10 pad 10: OUT_TX -> +3V3
- J10 pad 12: OUT_RX -> GND
- J10 pad 2: BATT_SENSE -> OUT_RX
- J10 pad 3: +3V3 -> BATT_SENSE_HV
- J10 pad 4: 5V_EN -> OUT_TX
- J10 pad 5: +5V -> BATT_SENSE_LV
- J10 pad 6: SPEAKER_+ -> GND
- J10 pad 7: GND -> SPEAKER_-
- J10 pad 8: SPEAKER_- -> +5V
- J10 pad 9: unconnected-(J10-Pin_9-Pad9) -> SPEAKER_+
- J2 pad 1: SW_CLK -> unconnected-(J2-Pin_1-Pad1)
- J4 pad 13: ~{PI_SHUTDOWN} -> ~{PI_POWERED_OFF}
- J4 pad 3: SDA -> RPI_SDA
- J4 pad 36: ~{WAKEUP_PING} -> ~{READ_ATTINY_CMD_REG}
- J4 pad 37: unconnected-(J4-GPIO26-Pad37) -> ~{PI_SHUTDOWN}
- J4 pad 38: unconnected-(J4-GPIO20/MOSI1-Pad38) -> MODEM_POWER_EN
- J4 pad 5: SCL -> RPI_SCL
- R15 pad 1: ATTINY_TX -> /ATtiny1616/~{READ_ATTINY_CMD_REG_PHY}
- R15 pad 2: Net-(U1-PB2) -> ~{READ_ATTINY_CMD_REG}
- R3 pad 1: Net-(U1-PA4) -> /ATtiny1616/~{LED_G_PHY}
- R35 pad 1: +3V3 -> /ATtiny1616/~{PI_SHUTDOWN_PHY}
- R35 pad 2: ~{WAKEUP_PING} -> ~{PI_SHUTDOWN}
- R4 pad 1: Net-(U1-PA3) -> /ATtiny1616/~{LED_B_PHY}
- SW2 pad 1: Net-(U1-PA6) -> /ATtiny1616/ATtiny_SW
- SW2 pad 2: unconnected-(SW2-Pad2) -> /ATtiny1616/ATtiny_SW
- SW2 pad 3: unconnected-(SW2-Pad3) -> GND
- TP1 pad 1: Net-(U1-PC3) -> GND
- TP6 pad 2: +3V3_rp2040 -> +3V3
- U1 pad 11: ATTINY_RX -> /ATtiny1616/~{LED_B_PHY}
- U1 pad 12: Net-(U1-PB2) -> /ATtiny1616/~{LED_G_PHY}
- U1 pad 15: ~{WAKEUP_PING} -> /ATtiny1616/~{READ_ATTINY_CMD_REG_PHY}
- U1 pad 17: EN_PERIPH_POWER -> /ATtiny1616/EN_PERIPH_POWER_PHY
- U1 pad 18: Net-(U1-PC3) -> /ATtiny1616/~{PI_SHUTDOWN_PHY}
- U1 pad 2: Net-(U1-PA3) -> /ATtiny1616/ATTINY_PA3
- U1 pad 5: Net-(U1-PA4) -> BATT_SENSE_LOW_VOLTAGE_PHY
- U1 pad 7: Net-(U1-PA6) -> /ATtiny1616/ATtiny_SW
- U1 pad 8: ~{PI_SHUTDOWN} -> ~{PI_POWERED_OFF}
- U1 pad 9: BATT_SENSE -> BATT_SENSE_HIGH_VOLTAGE_PHY
- U12 pad 2: +3V3 -> +3V8
- U12 pad 4: +3V3 -> +3V8
- U12 pad 70: +3V3 -> +3V8
- U12 pad 72: +3V3 -> +3V8
- U12 pad 74: +3V3 -> +3V8
- U15 pad 15: ATTINY_TX -> unconnected-(U15-1Y2-Pad15)
- U15 pad 2: ATTINY_RX -> unconnected-(U15-2Y2-Pad2)
- U3 pad 6: ~{WAKEUP_PING} -> ~{READ_ATTINY_CMD_REG}
Routing:
- net MODEM_POWER_EN: track 0.00 -> 70.3 mm, vias 0 -> 5
- net ~{WAKEUP_PING}: track 69.6 -> 0.00 mm, vias 4 -> 0
- net ~{READ_ATTINY_CMD_REG}: track 0.00 -> 62.7 mm, vias 0 -> 2
- net Net-(U1-PA4): track 57.4 -> 0.00 mm, vias 3 -> 0
- net Net-(U1-PA3): track 53.7 -> 0.00 mm, vias 3 -> 0
- net /ATtiny1616/~{LED_R_PHY}: track 60.1 -> 12.2 mm, vias 3 -> 1
- net ATTINY_RX: track 34.7 -> 0.00 mm, vias 3 -> 0
- net ATTINY_TX: track 32.9 -> 0.00 mm, vias 3 -> 0
- net +5V: track 13.9 -> 41.9 mm, vias 7 -> 14
- net BATT_SENSE: track 27.7 -> 0.00 mm, vias 2 -> 0
- net /ATtiny1616/ATtiny_SW: track 0.00 -> 27.5 mm, vias 0 -> 5
- net BATT_SENSE_LV: track 0.00 -> 23.4 mm, vias 0 -> 2
- net 5V_EN: track 30.5 -> 52.7 mm, vias 2 -> 5
- net Net-(U1-PA6): track 20.2 -> 0.00 mm, vias 1 -> 0
- net BATT_SENSE_HV: track 0.00 -> 20.0 mm, vias 0 -> 1
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- added copper zone on B.Cu, net +3V8
- added copper zone on F.Cu, net +3V8
- added copper zone on F.Cu, net /modem/3V3_L1
- added copper zone on F.Cu, net /modem/3V3_L2
- added copper zone on F.Cu, net /modem/MODEM_3V8
Other:
- board size 65 x 89 mm -> 65 x 75.5 mm
- board text added: "3V8"
- board text removed: "CLK"
- board text removed: "GND"
- board text removed: "SWD"
