File: tc2-main-pcb/tc2-main-pcb.kicad_pcb (KiCad board)
At the start: 4 copper layers, 65 x 75.5 mm, 177 parts, among them J1 Screw_Terminal_01x01, J10 Conn_02x06_Odd_Even, J11 Conn_01x08, J2 Screw_Terminal_01x01, J3 Conn_01x03, J4 Raspberry_Pi_2_3, J5 Screw_Terminal_01x01, J6 Screw_Terminal_01x01, J7 Screw_Terminal_01x01, J8 Screw_Terminal_01x01, J9 Conn_02x03_Odd_Even, Q1 Q_PMOS_GSD, SW2 K2-6639SP-M4SC-04, U1 ATtiny1616-M, U10 TD6810, U11 TD6810, U12 SIM7600G-H-M.2, U13 AHT21, U14 MAX98357AEWL+T, U15 74HC4052, U16 M24C02-WMN, U17 PCA9515ADP,118, U2 W25Q128JVS, U3 RP2040, U4 MT29F2G01ABAGDWB-IT, U5 TPS6302x, U6 PCF8563T, U7 ME6216A28XG, U8 Flir_LEPTON, U9 3N25000G33YC, Y1 Crystal_GND24, Y2 Crystal

Commit message: v0.4.0
Parts:
- removed SW2: K2-6639SP-M4SC-04, cacophony-library:KEY-SMD_4P-L6.0-W6.0-P3.90_K2-6639SP-K4SC-04
- removed TP46, TP47, TP9: TestPoint, cacophony-library:TP
- removed U17: PCA9515ADP,118, Package_SO:TSSOP-8_3x3mm_P0.65mm
- added C61: 22pF, Capacitor_SMD:C_0402_1005Metric, B.Cu at (14.9, 2.41)
- added C63: 22pF, Capacitor_SMD:C_0402_1005Metric, B.Cu at (13.1, 2.41)
- added H2: MountingHole, cacophony-library:MountingHole_3.2mm_M3, F.Cu at (56.8, 18.0)
- added J12: USB_B_Micro, cacophony-library:MICRO-USB-TH_MICRO-USB-A14, F.Cu at (34.8, -33.6)
- added R41: 100k, Resistor_SMD:R_0402_1005Metric, F.Cu at (-3.15, 11.0)
- added R47: 100k, Resistor_SMD:R_0402_1005Metric, F.Cu at (-9.93, 7.59)
- added R48: 22ohm, Resistor_SMD:R_0402_1005Metric, F.Cu at (12.6, -11.4)
- added R50: 22ohm, Resistor_SMD:R_0402_1005Metric, B.Cu at (18.8, -26.0)
- added R51: 22ohm, Resistor_SMD:R_0402_1005Metric, B.Cu at (19.8, -26.0)
- added R52: 100k, Resistor_SMD:R_0402_1005Metric, F.Cu at (4.33, 24.7)
- added SW1: SW_Push, Button_Switch_THT:SW_PUSH_6mm, F.Cu at (27.4, 22.7)
- added TP11: TestPoint, cacophony-library:TP, F.Cu at (-4.13, 7.46)
- added TP15: TestPoint, cacophony-library:TP, F.Cu at (-7.63, 19.0)
- added TP16: TestPoint, cacophony-library:TP, F.Cu at (-3.27, 17.5)
- added TP21: TestPoint, cacophony-library:TP, F.Cu at (-3.23, 15.1)
- added TP22: TestPoint, cacophony-library:TP, F.Cu at (6.27, -15.3)
- added TP7: TestPoint, cacophony-library:TP, F.Cu at (-4.16, 5.28)
- added U18: TCA4311ADGKR, Package_SO:MSOP-8_3x3mm_P0.65mm, F.Cu at (5.67, 21.1)
- H5, H6: footprint MountingHole:MountingHole_2.2mm_M2 -> cacophony-library:MountingHole_2.2mm_M2
- J1, J2, J5, J6, J8: footprint cacophony-library:SMTSO25 -> cacophony-library:smd_nut_SMTSO25
- R24: moved to F.Cu
- TP13: value TestPoint -> TP_2P; footprint cacophony-library:TP -> cacophony-library:test-point-2p
- U10, U11: footprint Package_TO_SOT_SMD:TSOT-23-5 -> cacophony-library:TSOT-23-5
- U13: value AHT21 -> AHT20_C2757850
- U6: footprint Package_SO:SOIC-8_3.9x4.9mm_P1.27mm -> cacophony-library:SOIC-8_3.9x4.9mm_P1.27mm
- moved TP13 39.8 mm to (12.2, 20.9), turned to 180 degrees
- moved R24 19.1 mm to (3.38, 11.0), turned to -90 degrees
- moved TP3 13.2 mm to (11.4, -23.0), turned to 90 degrees
- moved TP19 12.6 mm to (42.1, -1.90)
- moved C65 6.48 mm to (36.4, 31.4)
- moved C66 6.48 mm to (36.4, 29.9)
- moved TP20 4.73 mm to (41.2, -8.00)
- moved C50 3.23 mm to (6.17, 24.7), turned to 0 degrees
- moved R38 2.33 mm to (29.4, -21.2)
- moved Q1 1.81 mm to (27.0, -22.2)
- moved C38 1.81 mm to (24.4, -23.7)
- moved C43 1.81 mm to (27.0, -24.7)
- moved R44 1.48 mm to (29.9, 17.9)
- moved R34 1.31 mm to (1.09, 12.7)
- moved C49 1.18 mm to (35.8, 15.5)
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Connections:
- C37 pad 1: +5V -> +3V3
- J4 pad 32: MUL_S1 -> /Raspberry_Pi/GPIO12
- J4 pad 33: unconnected-(J4-PWM1/GPIO13-Pad33) -> I2C_BUS_LOCK
- TP13 pad 1: /GPIO3 -> GND
- U15 pad 11: unconnected-(U15-1Y3-Pad11) -> Net-(U15-1Y3)
- U15 pad 15: unconnected-(U15-1Y2-Pad15) -> Net-(U15-1Y2)
- U15 pad 16: +5V -> +3V3
- U15 pad 2: unconnected-(U15-2Y2-Pad2) -> Net-(U15-2Y2)
- U15 pad 4: unconnected-(U15-2Y3-Pad4) -> Net-(U15-2Y3)
- U15 pad 6: GND -> /Raspberry_Pi/~{UART_MULTIPLEX_EN}
- U15 pad 9: MUL_S1 -> Net-(U15-S1)
- U16 pad 5: SCL -> SDA
- U16 pad 6: SDA -> SCL
- U3 pad 18: RPI_SPI_MISO -> /RPI_SPI_MISO_PHY
- U3 pad 46: /USB_D- -> /USB_D-_PHY
- U3 pad 47: /USB_D+ -> /USB_D+_PHY
- U3 pad 5: /GPIO3 -> I2C_BUS_LOCK
Routing:
- net MUL_S1: track 34.1 -> 0.00 mm, vias 3 -> 0
- net USB_D+: track 0.00 -> 22.7 mm
- net USB_D-: track 0.00 -> 21.1 mm
- net I2C_BUS_LOCK: track 0.00 -> 12.8 mm, vias 0 -> 1
- net /Raspberry_Pi/GPIO12: track 0.00 -> 9.62 mm
- net Net-(U15-S1): track 0.00 -> 9.42 mm
- net Net-(U15-1Y3): track 0.00 -> 8.41 mm
- net +5V: track 41.9 -> 34.4 mm, vias 14 -> 13
- net ~{EN_RP2040_POWER}: track 64.0 -> 57.2 mm
- net RPI_SPI_MISO: track 25.0 -> 18.6 mm
- net GND: track 99.6 -> 105.6 mm, vias 182 -> 183
- net /GPIO3: track 6.07 -> 0.00 mm
- net SDA: track 74.6 -> 79.9 mm, vias 4 -> 7
- net /RPI_SPI_MISO_PHY: track 0.00 -> 5.26 mm
- net /USB_D-_PHY: track 0.00 -> 4.91 mm, vias 0 -> 1
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- removed copper zone on In2.Cu, net GND
Other:
- board size 65 x 75.5 mm -> 73 x 75.5 mm
- board text added: "V0.4.0"
