File: tc2-main-pcb/tc2-main-pcb.kicad_pcb (KiCad board)
At the start: 6 copper layers, 73 x 75.5 mm, 215 parts, among them J101 Conn_02x03_Odd_Even, J102 USB_B_Micro, J103 Conn_01x03, J104 Conn_02x06_Odd_Even, J105 Screw_Terminal_01x01, J106 Screw_Terminal_01x01, J107 Screw_Terminal_01x01, J108 Screw_Terminal_01x01, J109 Screw_Terminal_01x01, J110 Raspberry_Pi_2_3, J111 Conn_01x08, J112 Screw_Terminal_01x01, Q101 Q_PMOS_GSD, SW101 SW_Push, U101 W25Q128JVS, U102 RP2040, U103 MT29F2G01ABAGDWB-IT, U104 AHT20_C2757850, U105 PCF8563T, U106 M24C02-WMN, U107 MAX98357AEWL+T, U108 TCA4311ADGKR, U109 74HC4052, U110 TD6810, U111 TD6810, U112 ME6216A28XG, U113 3N25000G33YC, U114 Flir_LEPTON, U115 TPS6302x, U116 SIM7600G-H-M.2, U117 ATtiny1616-M, Y101 Crystal_GND24, Y102 Crystal

Commit message: Fix library
Parts:
- C112, C113, C118: value 1u -> 1uF
- R102, R103, R104, R110, R119, R120, R121, R122, R123, R124, R135, R143, R144, R145: value 22ohm -> 22Ω
- R112, R157, R158, R159: value 180R -> 180Ω
- U101: footprint Package_SO:SOIC-8_5.23x5.23mm_P1.27mm -> Package_SO:SOIC-8_5.3x5.3mm_P1.27mm
- U109: footprint Package_SO:SOP-16_3.9x9.9mm_P1.27mm -> cacophony-library:SOP-16_L10.0-W3.9-P1.27-LS6.0-BL
- turned U109 to 90 degrees

Commit message: Add JLPCPCB 2D barcode to PCBs
Parts:
- added U1: ~, cacophony-library:JLCPCB_QR_8mm, F.Cu at (-41.4, 25.6)
Changed lines of the file:
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@@
 		)
 		(embedded_fonts no)
-		(model "${KICAD6_3DMODEL_DIR}/Connector_JST.3dshapes/JST_SH_BM03B-SRSS-TB_1x03-1MP_P1.00mm_Vertical.wrl"
+		(model "${KICAD10_3DMODEL_DIR}/Connector_JST.3dshapes/JST_SH_BM03B-SRSS-TB_1x03-1MP_P1.00mm_Vertical.step"
 			(offset
 				(xyz 0 0 0)
@@
 		)
 		(embedded_fonts no)
-		(model "${KICAD8_3DMODEL_DIR}/Connector_PinSocket_2.54mm.3dshapes/PinSocket_2x20_P2.54mm_Vertical.wrl"
+		(model "${KICAD10_3DMODEL_DIR}/Connector_PinSocket_2.54mm.3dshapes/PinSocket_2x20_P2.54mm_Vertical.step"
 			(offset
 				(xyz 0 0 0)
@@
 		)
 	)
+	(footprint "cacophony-library:JLCPCB_QR_8mm"
+		(layer "F.Cu")
+		(at -41.375 25.625)
+		(property "Reference" "U1"
+			(at 0 -0.5 0)
+			(unlocked yes)
+			(layer "F.SilkS")
+			(hide yes)
+			(effects
+				(font
+					(size 1 1)
+					(thickness 0.1)
+				)
+			)
+		)
+		(property "Value" "~"
+			(at 0 1 0)
+			(unlocked yes)
+			(layer "F.Fab")
+			(effects
+				(font
+					(size 1 1)
+					(thickness 0.15)
+				)
+			)
+		)
+		(property "Datasheet" ""
+			(at 0 0 0)
+			(unlocked yes)
+			(layer "F.Fab")
+			(hide yes)
+			(effects
+				(font
+					(size 1 1)
+					(thickness 0.15)
+				)
+			)
+		)
+		(property "Description" ""
+			(at 0 0 0)
+			(unlocked yes)
+			(layer "F.Fab")
+			(hide yes)
+			(effects
+				(font
+					(size 1 1)
+					(thickness 0.15)
+				)
+			)
+		)
+		(sheetname "/")
+		(sheetfile "tc2-main-pcb.kicad_sch")
+		(attr exclude_from_pos_files exclude_from_bom)
+		(duplicate_pad_numbers_are_jumpers no)
+		(fp_rect
+			(start -4 -4)
+			(end 4 4)
+			(stroke
+				(width 0)
+				(type solid)
+			)
+			(fill yes)
+			(layer "F.SilkS")
+		)
+		(fp_text user "${REFERENCE}"
+			(at 0 2.5 0)
+			(unlocked yes)
+			(layer "F.Fab")
+			(effects
+				(font
+					(size 1 1)
+					(thickness 0.15)
+				)
+			)
+		)
+		(embedded_fonts no)
+	)
 	(footprint "Resistor_SMD:R_0402_1005Metric"
 		(layer "F.Cu")
@@
 		)
 		(embedded_fonts no)
-		(model "${KICAD8_3DMODEL_DIR}/Package_SO.3dshapes/SOIC-8_3.9x4.9mm_P1.27mm.wrl"
+		(model "${KICAD10_3DMODEL_DIR}/Package_SO.3dshapes/SOIC-8_3.9x4.9mm_P1.27mm.step"
 			(offset
 				(xyz 0 0 0)
@@
 		)
 		(embedded_fonts no)
-		(model "${KICAD8_3DMODEL_DIR}/Connector_PinSocket_2.54mm.3dshapes/PinSocket_1x08_P2.54mm_Vertical.wrl"
+		(model "${KICAD10_3DMODEL_DIR}/Connector_PinSocket_2.54mm.3dshapes/PinSocket_1x08_P2.54mm_Vertical.step"
 			(offset
 				(xyz 0 0 0)
@@
 		)
 		(embedded_fonts no)
-		(model "${KICAD6_3DMODEL_DIR}/Connector_PinSocket_1.27mm.3dshapes/PinSocket_2x03_P1.27mm_Vertical_SMD.wrl"
+		(model "${KICAD10_3DMODEL_DIR}/Connector_PinSocket_1.27mm.3dshapes/PinSocket_2x03_P1.27mm_Vertical_SMD.step"
 			(offset
 				(xyz 0 0 0)
@@
 		)
 		(embedded_fonts no)
-		(model "${KICAD8_3DMODEL_DIR}/Package_TO_SOT_SMD.3dshapes/TSOT-23-5.wrl"
+		(model "${KICAD10_3DMODEL_DIR}/Package_TO_SOT_SMD.3dshapes/TSOT-23-5.step"
 			(offset
 				(xyz 0 0 0)
@@
 			)
 		)
-		(property "JLCPCB" ""
-			(at 0 0 90)
-			(layer "B.Fab")
-			(hide yes)
-			(effects
-				(font
-					(size 1 1)
-					(thickness 0.15)
-				)
-				(justify mirror)
-			)
-		)
 		(property "LCSC Part" "C16510"
 			(at 0 0 270)
@@
 		)
 		(embedded_fonts no)
-		(model "${KICAD8_3DMODEL_DIR}/Package_TO_SOT_SMD.3dshapes/TSOT-23-5.wrl"
+		(model "${KICAD10_3DMODEL_DIR}/Package_TO_SOT_SMD.3dshapes/TSOT-23-5.step"
 			(offset
 				(xyz 0 0 0)
@@
 		)
 		(embedded_fonts no)
-		(model "${KISYS3DMOD}/Package_DFN_QFN.3dshapes/QFN-56-1EP_7x7mm_P0.4mm_EP5.6x5.6mm.wrl"
+		(model "${KICAD10_3DMODEL_DIR}/Package_DFN_QFN.3dshapes/QFN-56-1EP_7x7mm_P0.4mm_EP5.6x5.6mm.step"
 			(offset
 				(xyz 0 0 0)
@@
 	)
 	(gr_circle
-		(center -43.6 24.92)
-		(end -42.4 24.92)
-		(stroke
-			(width 0.15)
-			(type default)
-		)
-		(fill no)
-		(layer "User.4")
-	)
-	(gr_circle
 		(center -41.8 -29)
 		(end -43.55 -29)
@@
 		(layer "User.4")
 	)
-	(gr_circle
-		(center -30.6 24.92)
-		(end -23.6 24.92)
-		(stroke
-			(width 0.15)
-			(type default)
-		)
-		(fill no)
-		(layer "User.4")
-	)
 	(gr_line
 		(start -27.6 20.92)
@@
 		)
 		(fill no)
-		(layer "User.4")
-	)
-	(gr_circle
-		(center -17.6 24.92)
-		(end -16.4 24.92)
-		(stroke
-			(width 0.15)
-			(type default)
-		)
-		(fill no)

Commit message: Update layout
Parts:
- removed C133, C135, C136, C137, C138, C140: 10uF, Capacitor_SMD:C_0603_1608Metric
- removed C134, C139, C149: 12pF, Capacitor_SMD:C_0402_1005Metric
- removed C146, C147, C151, C152, C153, C154: 22uF, Capacitor_SMD:C_0603_1608Metric
- removed C148, C150: 220nF, Capacitor_SMD:C_0402_1005Metric
- removed D102: D, Diode_SMD:D_SOD-523
- removed FB101: FerriteBead, Inductor_SMD:L_0805_2012Metric
- removed L101, L102: 4.7uH, cacophony-library:IND-SMD_L4.0-W4.0_SWPA4018S
- removed L103: INDUCTOR, Inductor_SMD:L_1008_2520Metric
- removed R113: 1k, Resistor_SMD:R_0402_1005Metric
- removed R137, R141: 100k, Resistor_SMD:R_0402_1005Metric
- removed R138, R139: 1M, Resistor_SMD:R_0402_1005Metric
- removed R140: 150k, Resistor_SMD:R_0402_1005Metric
- removed TP105, TP122, TP135: TestPoint, cacophony-library:TP
- removed TP117: TestPoint, TestPoint:TestPoint_Pad_D1.0mm
- removed TP131, TP132, TP133, TP134: TP_2P, cacophony-library:test-point-2p
- removed U108: TCA4311ADGKR, Package_SO:MSOP-8_3x3mm_P0.65mm
- removed U110, U111: TD6810, cacophony-library:TSOT-23-5
- removed U112: ME6216A28XG, Package_TO_SOT_SMD:TSOT-23
- removed U115: TPS6302x, cacophony-library:VSON-14_L4.0-W3.0-P0.50-BL-EP_TI_DSJ
- added C168: 2.2uF, Capacitor_SMD:C_0402_1005Metric, F.Cu at (-32.4, -3.13)
- added C169: 2.2uF, Capacitor_SMD:C_0402_1005Metric, F.Cu at (-30.3, -4.68)
- added C170: 2.2uF, Capacitor_SMD:C_0402_1005Metric, F.Cu at (-37.9, -2.75)
- added C171: 22pF, Capacitor_SMD:C_0402_1005Metric, F.Cu at (-25.1, 2.32)
- added C172: 2.2uF, Capacitor_SMD:C_0402_1005Metric, F.Cu at (-35.8, -4.29)
- added C173: 22uF, Capacitor_SMD:C_0603_1608Metric, F.Cu at (-30.4, 2.63)
- added C174: 22uF, Capacitor_SMD:C_0603_1608Metric, F.Cu at (-31.8, 2.63)
- added C175: 22uF, Capacitor_SMD:C_0603_1608Metric, F.Cu at (-23.9, 2.58)
- added C176: 22uF, Capacitor_SMD:C_0603_1608Metric, B.Cu at (-30.5, 16.7)
- added C177: 22uF, Capacitor_SMD:C_0603_1608Metric, B.Cu at (-29.1, 16.7)
- added C178: 22pF, Capacitor_SMD:C_0402_1005Metric, B.Cu at (-35.4, 17.8)
- added C179: 22uF, Capacitor_SMD:C_0603_1608Metric, B.Cu at (-37.0, 16.8)
- added FB103: FerriteBead, Inductor_SMD:L_0805_2012Metric, B.Cu at (-37.1, 14.4)
- added FB104: FerriteBead, Inductor_SMD:L_0805_2012Metric, F.Cu at (-24.9, -0.65)
- added H1: MountingHole, cacophony-library:MountingHole_1.8mm_M1.6, F.Cu at (-22.6, -3.58)
- added H2: MountingHole, cacophony-library:MountingHole_1.8mm_M1.6, F.Cu at (-38.6, -10.6)
- added H3: Key Hole, cacophony-library:KeyHole_1.8mm, F.Cu at (-38.6, -7.58)
- added H4: Key Hole, cacophony-library:KeyHole_1.8mm, F.Cu at (-22.6, -7.58)
- added J1901: TC2030, cacophony-library:Tag-Connect_TC2030-IDC-NL_2x03_P1.27mm_Vertical, B.Cu at (-46.2, -13.7)
- added L104: 1uH, Inductor_SMD:L_1008_2520Metric, B.Cu at (-33.4, 14.1)
- added L105: INDUCTOR, Inductor_SMD:L_1008_2520Metric, F.Cu at (-27.7, 0.05)
- added R1: 10M, Resistor_SMD:R_0402_1005Metric, F.Cu at (-12.8, 11.0)
- added R148: 100k, Resistor_SMD:R_0402_1005Metric, F.Cu at (-27.0, 2.34)
- added R161: 100k, Resistor_SMD:R_0402_1005Metric, B.Cu at (-31.3, 18.6)
- added R162: 470k, Resistor_SMD:R_0402_1005Metric, B.Cu at (-35.8, 16.4)
- added R163: 100k, Resistor_SMD:R_0402_1005Metric, F.Cu at (-26.0, 2.33)
- added R164: 68k, Resistor_SMD:R_0402_1005Metric, B.Cu at (-34.9, 16.4)
- added R165: 100k, Resistor_SMD:R_0402_1005Metric, B.Cu at (-33.9, 16.4)
- added R166: 10k, Resistor_SMD:R_0402_1005Metric, F.Cu at (-29.0, -15.2)
- added R167: 10k, Resistor_SMD:R_0402_1005Metric, F.Cu at (-29.0, -16.1)
- added R168: 100k, Resistor_SMD:R_0402_1005Metric, F.Cu at (-29.5, 4.58)
- added TP136: TP_2P, cacophony-library:test-point-2p, B.Cu at (-35.2, 1.27)
- added TP137: TP_2P, cacophony-library:test-point-2p, B.Cu at (-21.5, -0.11)
- added TP138: TP_2P, cacophony-library:test-point-2p, B.Cu at (-39.9, -0.97)
- added TP139: TP_2P, cacophony-library:test-point-2p, B.Cu at (-26.0, 6.89)
- added U118: TLV75530PDRV, Package_SON:WSON-6-1EP_2x2mm_P0.65mm_EP1x1.6mm, F.Cu at (-30.6, -2.96)
- added U119: TLV75528PDRV, Package_SON:WSON-6-1EP_2x2mm_P0.65mm_EP1x1.6mm, F.Cu at (-37.6, -4.46)
- added U120: TPS62A02DRLR, cacophony-library:SOT-563, F.Cu at (-28.5, 2.76)
- added U121: TPS62A02DRLR, cacophony-library:SOT-563, B.Cu at (-32.3, 16.8)
- added U2: PCA9517ADP,118, Package_SO:MSOP-8_3x3mm_P0.65mm, B.Cu at (-5.78, 21.6)
- BT101: value Battery_Cell -> MS621FE-FL11E
- C123: value 22pF -> 220nF
- C145, R133, R134: moved to F.Cu
- R105, R107: moved to B.Cu
- R117, R129, R136: value 100k -> 10k
- R128: value 390k -> 10k
- R131: value 100k -> 10k; moved to F.Cu
- TP104, TP106, TP107: footprint cacophony-library:TP -> TestPoint:TestPoint_Loop_D2.54mm_Drill1.5mm_Beaded
- TP120: footprint cacophony-library:TP -> TestPoint:TestPoint_Pad_D1.0mm
- U109: footprint cacophony-library:SOP-16_L10.0-W3.9-P1.27-LS6.0-BL -> Package_SO:SOIC-16_3.9x9.9mm_P1.27mm
- moved R117 55.1 mm to (-28.1, -25.0), turned to 180 degrees
- moved TP106 54.8 mm to (5.48, -29.2)
- moved TP120 51.7 mm to (-51.4, -14.2)
- moved TP107 49.9 mm to (-8.10, 29.3)
- moved TP121 45.7 mm to (-46.2, -10.6)
- moved R128 41.7 mm to (-5.09, 26.4), turned to -90 degrees
- moved R127 41.5 mm to (-6.09, 26.4), turned to -90 degrees
- moved TP104 38.5 mm to (-50.8, 14.4)
- moved R107 36.6 mm to (-29.6, -24.0), turned to 135 degrees
- moved R105 33.2 mm to (-29.9, -22.4), turned to 180 degrees
- moved R129 30.5 mm to (-25.8, -25.6), turned to 90 degrees
- moved R136 29.4 mm to (-8.61, 5.11)
- moved R130 27.8 mm to (4.36, 2.61), turned to 180 degrees
- moved R131 15.2 mm to (-8.30, 4.13), turned to 0 degrees
- moved R115 11.9 mm to (-46.7, -8.70), turned to 0 degrees
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Connections:
- net Net-(U114-SPI_MISO) renamed /Lepton/LEPTON_SPI_MISO_PIN
- net Net-(U116-USIM_CLK) renamed /modem/USIM_CLK_PIN
- net Net-(U116-USIM_DATA) renamed /modem/USIM_DATA_PIN
- net Net-(U116-USIM_RST) renamed /modem/USIM_RST_PIN
- net Net-(U117-PA6) renamed /ATtiny1616/BUTTON
- C123 pad 1: /RTC_OSCO -> RTC_BT_SENSE_PHY
- R105 pad 1: +3V3 -> +3V3_rp2040
- R107 pad 1: +3V3 -> +3V3_rp2040
- R117 pad 1: GND -> +3V3_rp2040
- R117 pad 2: Net-(U108-READY) -> SDA
- R127 pad 1: Net-(R127-Pad1) -> RPI_SCL
- R127 pad 2: +3V0 -> +3V3
- R128 pad 1: /Lepton/FB_3V0 -> RPI_SDA
- R128 pad 2: Net-(R127-Pad1) -> +3V3
- R129 pad 1: /Lepton/FB_3V0 -> +3V3_rp2040
- R129 pad 2: GND -> SCL
- R130 pad 1: /Lepton/FB_1V2 -> GND
- R130 pad 2: +1V2 -> MUL_S0
- R131 pad 1: /Lepton/FB_1V2 -> +3V3
- R131 pad 2: GND -> SDA
- R136 pad 1: +3V0 -> +3V3
- R136 pad 2: LEPTON_I2C_SDA -> SCL
- TP120 pad 1: SPEAKER_+ -> Net-(J1901-Pad6)
- TP121 pad 1: 5V_EN -> Net-(J1901-Pad3)
- U117 pad 2: /ATtiny1616/ATTINY_PA3 -> EN_RPI_I2C
Routing:
- net EN_RPI_I2C: track 0.00 -> 42.5 mm, vias 0 -> 3
- net +3V0: track 43.4 -> 26.1 mm, vias 8 -> 4
- net GND: track 91.6 -> 76.8 mm, vias 177 -> 134
- net 5V_EN: track 48.7 -> 35.3 mm, vias 5 -> 4
- net /EEPROM_~{WC}: track 7.45 -> 19.5 mm
- net SCL: track 120.9 -> 130.0 mm
- net +3V3_rp2040: track 75.0 -> 84.1 mm
- net Net-(U115-PG): track 8.26 -> 0.00 mm
- net +3V3: track 20.6 -> 26.1 mm
- net /modem/3V8_FB: track 0.00 -> 5.38 mm
- net MODEM_POWER_EN: track 73.4 -> 68.1 mm
- net RPI_SCL: track 5.49 -> 10.4 mm, vias 1 -> 0
- net /Lepton/1V2_FB: track 0.00 -> 4.66 mm
- net Net-(J1901-Pad6): track 0.00 -> 4.36 mm, vias 0 -> 1
- net SDA: track 122.7 -> 126.7 mm, vias 7 -> 8
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- added copper zone on F.Cu, net /Lepton/1V2_PHY
- added copper zone on B.Cu, net /modem/3V8_PHY
- removed copper zone on B.Cu, net +1V2
- removed copper zone on F.Cu, net +1V2
- removed copper zone on B.Cu, net +3V0
- removed copper zone on F.Cu, net +3V0
- removed copper zone on B.Cu, net +3V3
- removed copper zone on B.Cu, net /Lepton/SW_1V2
- removed copper zone on B.Cu, net /Lepton/SW_3V0
- removed copper zone on B.Cu, net /modem/3V3_L1
- removed copper zone on B.Cu, net /modem/3V3_L2
- removed copper zone on B.Cu, net /modem/MODEM_3V8
Other:
- board text removed: "1V2"
- board text removed: "~{WC}"
