File: tc2-main-pcb/tc2-main-pcb.kicad_sch (KiCad schematic)
At the start: 77 parts, among them J10 Conn_02x06_Odd_Even, J12 USB_B_Micro, J3 Conn_01x03, J9 Conn_02x03_Odd_Even, Q1 Q_PMOS_GSD, U13 AHT20_C2757850, U16 M24C02-WMN, U2 W25Q128JVS, U3 RP2040, U4 MT29F2G01ABAGDWB-IT, U6 PCF8563T, Y1 Crystal_GND24, Y2 Crystal

Commit message: Update to use touch sensor
Parts:
- added H107, H108: MountingHole, cacophony-library:MountingHole_2.2mm_M2, symbol Mechanical:MountingHole
- added R115: 100k, Resistor_SMD:R_0402_1005Metric, symbol Device:R
- added TP101, TP102, TP108, TP110, TP117: TestPoint, TestPoint:TestPoint_Pad_D1.0mm, symbol Connector:TestPoint
- R108: renamed from R2; now not fitted
- renumbered BT1 to BT101, C5 to C101, C6 to C102, C8 to C103, C10 to C104, C11 to C105, C12 to C106, C13 to C107, C14 to C108, C15 to C109, C38 to C110, C43 to C111, C7 to C112, C9 to C113, C2 to C114, C3 to C115, C4 to C116, C16 to C117, C17 to C118, C39 to C119, C18 to C120, C48 to C121, C63 to C122, C61 to C123, C65 to C124, C66 to C125, C62 to C126, C64 to C127, D3 to D101, D2 to D102, H5 to H101, H6 to H102, H1 to H103, H3 to H104, H4 to H105, H2 to H106, J9 to J101, J12 to J102, J3 to J103, J10 to J104, Q1 to Q101, R38 to R101, R50 to R102, R51 to R103, R28 to R104, R10 to R105, R53 to R106, R11 to R107, R1 to R109, R48 to R110, R9 to R111, R39 to R112, R7 to R113, R8 to R114, TP3 to TP103, TP14 to TP104, TP18 to TP105, TP19 to TP106, TP20 to TP107, TP12 to TP109, TP26 to TP111, TP27 to TP112, TP41 to TP113, TP40 to TP114, TP13 to TP115, TP17 to TP116, TP6 to TP118, TP10 to TP119, U2 to U101, U3 to U102, U4 to U103, U13 to U104, U6 to U105, U16 to U106, Y1 to Y101, Y2 to Y102
Connections:
- net +3V3: now also R115.2
- net PDM_CLOCK: now also TP101.1
- net PDM_DATA: now also TP102.1
- net SCL: now also TP110.1
- net SDA: now also TP108.1
- net SPEAKER_+: now also J104.7 (Pin_7); no longer J104.9 (Pin_9)
- net SPEAKER_-: now also J104.9 (Pin_9); no longer J104.7 (Pin_7)
- net EEPROM_~{WC}: now reaches U106.7 (~{WC})
- net EEPROM_~{WC}: now also R115.1, TP117.1
- net BATT_SENSE_HV renamed BATTERY_HV
- net BATT_SENSE_LV renamed BATTERY_LV
- no-connect marks 10 -> 9

Commit message: Change to through hole connector and add simcard PCB to pannel
Parts:
- removed H107, H108: MountingHole, cacophony-library:MountingHole_2.2mm_M2, symbol Mechanical:MountingHole
Other:
- note added: "C3975170"
Changed lines of the file:
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@@
 		)
 	)
+	(text "C3975170"
+		(exclude_from_sim no)
+		(at 48.26 238.76 0)
+		(effects
+			(font
+				(size 1.27 1.27)
+			)
+		)
+	)
 	(text "Always double check \nallignemnt with plug PCB"
 		(exclude_from_sim no)
@@
 	)
 	(symbol
-		(lib_id "Mechanical:MountingHole")
-		(at 115.57 234.95 0)
-		(unit 1)
-		(exclude_from_sim no)
-		(in_bom no)
-		(on_board yes)
-		(dnp no)
-		(fields_autoplaced yes)
-		(property "Reference" "H108"
-			(at 118.11 234.315 0)
-			(effects
-				(font
-					(size 1.27 1.27)
-				)
-				(justify left)
-			)
-		)
-		(property "Value" "MountingHole"
-			(at 118.11 236.855 0)
-			(effects
-				(font
-					(size 1.27 1.27)
-				)
-				(justify left)
-			)
-		)
-		(property "Footprint" "cacophony-library:MountingHole_2.2mm_M2"
-			(at 115.57 234.95 0)
-			(effects
-				(font
-					(size 1.27 1.27)
-				)
-				(hide yes)
-			)
-		)
-		(property "Datasheet" "~"
-			(at 115.57 234.95 0)
-			(effects
-				(font
-					(size 1.27 1.27)
-				)
-				(hide yes)
-			)
-		)
-		(property "Description" ""
-			(at 115.57 234.95 0)
-			(effects
-				(font
-					(size 1.27 1.27)
-				)
-				(hide yes)
-			)
-		)
-		(instances
-			(project "tc2-main-pcb"
-				(path "/0662f88c-5300-4b75-bef3-048a3227af84"
-					(reference "H108")
-					(unit 1)
-				)
-			)
-		)
-	)
-	(symbol
 		(lib_id "Device:R")
 		(at 236.22 127 90)
@@
 					(unit 1)
 				)
-			)
-		)
-	)
-	(symbol
-		(lib_id "Mechanical:MountingHole")
-		(at 115.57 229.87 0)
-		(unit 1)
-		(exclude_from_sim no)
-		(in_bom no)
-		(on_board yes)
-		(dnp no)
-		(fields_autoplaced yes)
-		(property "Reference" "H107"
-			(at 118.11 229.235 0)
-			(effects
-				(font
-					(size 1.27 1.27)
-				)
-				(justify left)
-			)
-		)
-		(property "Value" "MountingHole"
-			(at 118.11 231.775 0)
-			(effects
-				(font
-					(size 1.27 1.27)
-				)
-				(justify left)
-			)
-		)
-		(property "Footprint" "cacophony-library:MountingHole_2.2mm_M2"
-			(at 115.57 229.87 0)
-			(effects
-				(font
-					(size 1.27 1.27)
-				)
-				(hide yes)
-			)
-		)
-		(property "Datasheet" "~"
-			(at 115.57 229.87 0)
-			(effects
-				(font
-					(size 1.27 1.27)
-				)
-				(hide yes)
-			)
-		)
-		(property "Description" ""
-			(at 115.57 229.87 0)
-			(effects
-				(font
-					(size 1.27 1.27)
-				)
-				(hide yes)
-			)
-		)
-		(instances
-			(project "tc2-main-pcb"
-				(path "/0662f88c-5300-4b75-bef3-048a3227af84"
-					(reference "H107")
-					(unit 1)
-				)

Commit message: Version v0.7.0
Parts:
- BT101: now left out of the parts list
Changed lines of the file:
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@@
 		(unit 1)
 		(exclude_from_sim no)
-		(in_bom yes)
+		(in_bom no)
 		(on_board yes)
 		(dnp no)
 		(property "Reference" "BT101"
-			(at 311.15 229.87 0)
+			(at 308.61 229.87 0)
 			(effects
 				(font

Commit message: version v0.7.1
Changed lines of the file:
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@@
-	(wire
-		(pts
-			(xy 298.45 226.06) (xy 297.18 226.06)
-		)
-		(stroke
-			(width 0)
-			(type default)
-		)
-	)
 	(wire
 		(pts
@@
 		)
 		(stroke
+			(width 0)
+			(type default)
+		)
+	)
+	(wire
+		(pts
+			(xy 297.18 226.06) (xy 298.45 226.06)
+		)
+		(stroke

Commit message: v0.7.2 panelise microphone boards
Parts:
- removed J104: Conn_02x06_Odd_Even, cacophony-library:power-pcb-3.1, symbol Connector_Generic:Conn_02x06_Odd_Even
- removed TP112: TestPoint, cacophony-library:TP, symbol Connector:TestPoint
- added C134: 220uF, symbol Device:C_Small
- added C177: 22pF, Capacitor_SMD:C_0402_1005Metric, symbol Device:C_Small
- added J113: Conn_02x07_Odd_Even, cacophony-library:power-pcb-0.7, symbol Connector_Generic:Conn_02x07_Odd_Even
- added R127: 22ohm, Resistor_SMD:R_0402_1005Metric, symbol Device:R
- added U121, U122, U123, U124: ICSRC3908SFR, cacophony-library:CONN-SMD_L3.9-W0.8, symbol cacophony-library:ICSRC3908SFR
Connections:
- net +3V3: now also C134.1, J113.10 (Pin_10)
- net +5V: now also J113.8 (Pin_8)
- net 5V_EN: now also J113.1 (Pin_1)
- net BATTERY_HV: now also J113.3 (Pin_3)
- net BATTERY_LV: now also J113.5 (Pin_5)
- net EN_PERIPH_POWER: now also J113.11 (Pin_11)
- net GND: now also C134.2, C177.2, J113.12 (Pin_12), J113.6 (Pin_6), U121.1, U122.1, U123.1, U124.1
- net OUT_RX: now also J113.2 (Pin_2)
- net OUT_TX: now also J113.4 (Pin_4)
- net RTC_BT_SENSE_PHY: now also C177.1
- net SPEAKER_+: now also J113.7 (Pin_7)
- net SPEAKER_-: now also J113.9 (Pin_9)
- net GPIO17 renamed BUCK_BOOST_FPWM_PHY
- net BUCK_BOOST_FPWM_PHY: now also R127.1
- new net BUCK_BOOST_FPWM: J113.13 (Pin_13), R127.2
- no-connect marks 9 -> 10
Other:
- note added: "Mounting holes for Microphone PCB"
- moved on the sheet: H101, H102, TP101, TP102, TP113

Commit message: v0.7.3
Parts:
- removed TP117: TestPoint, TestPoint:TestPoint_Pad_D1.0mm, symbol Connector:TestPoint
- added J114: Conn_01x02, cacophony-library:test_pads_2, symbol Connector_Generic:Conn_01x02
- BT101, J113: now not fitted
- C112, C113, C118: value 1u -> 1uF
- C134: value 220uF -> 220nF; footprint (none) -> Capacitor_SMD:C_0402_1005Metric
- H103, H104, H105, H106: footprint cacophony-library:MountingHole_3.2mm_M3 -> cacophony-library:MountingHole_3.5mm_M3
- U121, U122, U123, U124: LCSC (none) -> C238203
Connections:
- net EEPROM_~{WC}: now also J114.1 (Pin_1)
- net GND: now also J114.2 (Pin_2)

Commit message: 0.8.0 WIP
Parts:
- R102, R103, R104, R110, R127: value 22ohm -> 22Ω
- R112: value 180R -> 180Ω
Changed lines of the file:
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@@
 	(label "RTC_CLKO"
 		(at 383.54 240.03 0)
-		(fields_autoplaced yes)
 		(effects
 			(font
@@
 	(label "QSPI_SCLK"
 		(at 54.61 123.19 0)
-		(fields_autoplaced yes)
 		(effects
 			(font
@@
 	(label "QSPI_SS"
 		(at 54.61 118.11 0)
-		(fields_autoplaced yes)
 		(effects
 			(font
@@
 	(label "RTC_OSCO"
 		(at 351.79 242.57 0)
-		(fields_autoplaced yes)
 		(effects
 			(font
@@
 	(label "USB_D-_PHY"
 		(at 208.28 81.28 0)
-		(fields_autoplaced yes)
 		(effects
 			(font
@@
 	(label "I2C_BUS_LOCK_PHY"
 		(at 208.28 96.52 0)
-		(fields_autoplaced yes)
 		(effects
 			(font
@@
 	(label "PDM_CLOCK_PHY"
 		(at 208.28 91.44 0)
-		(fields_autoplaced yes)
 		(effects
 			(font
@@
 	(label "RTC_VDD"
 		(at 375.92 218.44 0)
-		(fields_autoplaced yes)
 		(effects
 			(font
@@
 	(label "BUCK_BOOST_FPWM_PHY"
 		(at 208.28 132.08 0)
-		(fields_autoplaced yes)
 		(effects
 			(font
@@
 	(label "USB_D+_PHY"
 		(at 208.28 78.74 0)
-		(fields_autoplaced yes)
 		(effects
 			(font
@@
 	(label "RPI_SPI_MISO_PHY"
 		(at 208.28 127 0)
-		(fields_autoplaced yes)
 		(effects
 			(font
@@
 	(label "RTC_OSCI"
 		(at 351.79 232.41 0)
-		(fields_autoplaced yes)
 		(effects
 			(font
@@
 	(label "MEM_~{WP}{slash}IO2"
 		(at 350.52 146.05 180)
-		(fields_autoplaced yes)
 		(effects
 			(font
@@
 	(label "RTC_BATTERY"
 		(at 323.85 226.06 0)
-		(fields_autoplaced yes)
 		(effects
 			(font
@@
 	(label "EEPROM_~{WC}"
 		(at 226.06 248.92 0)
-		(fields_autoplaced yes)
 		(effects
 			(font
@@
 	(label "AHT21_VDD"
 		(at 365.76 185.42 0)
-		(fields_autoplaced yes)
 		(effects
 			(font
@@
 	(label "MEM_~{HOLD}{slash}IO3"
 		(at 387.35 143.51 0)
-		(fields_autoplaced yes)
 		(effects
 			(font
@@
 	(label "GPIO16"
 		(at 208.28 129.54 0)
-		(fields_autoplaced yes)
 		(effects
 			(font
@@
 	(label "GPIO2"
 		(at 208.28 93.98 0)
-		(fields_autoplaced yes)
 		(effects
 			(font
@@
 			)
 		)
-		(property "Value" "22ohm"
+		(property "Value" "22Ω"
 			(at 242.57 77.47 90)
 			(effects
@@
 			)
 		)
-		(property "Value" "22ohm"
+		(property "Value" "22Ω"
 			(at 242.57 90.17 90)
 			(effects
@@
 			)
 		)
-		(property "Value" "22ohm"
+		(property "Value" "22Ω"
 			(at 247.65 130.81 90)
 			(effects
@@
 			)
 		)
-		(property "Value" "22ohm"
+		(property "Value" "22Ω"
 			(at 242.57 125.73 90)
 			(effects
@@
 			)
 		)
-		(property "Value" "22ohm"
+		(property "Value" "22Ω"
 			(at 242.57 80.01 90)
 			(effects
@@
 			)
 		)
-		(property "Value" "180R"
+		(property "Value" "180Ω"
 			(at 360.68 180.34 90)
 			(effects

Commit message: Updated to use field LCSC Part instead of LCSC for the JLCPCB part number
Parts:
- BT101: LCSC C80909 -> (none); LCSC Part (none) -> C80909
- C101, C102, C103, C104, C105, C106, C107, C108, C109, C114, C117, C121, C134: LCSC C16772 -> (none); LCSC Part (none) -> C16772
- C110, C111, C119, C120: LCSC C19702 -> (none); LCSC Part (none) -> C19702
- C112, C113, C118: LCSC C52923 -> (none); LCSC Part (none) -> C52923
- C115, C116: LCSC C1547 -> (none); LCSC Part (none) -> C1547
- C122, C123, C177: LCSC C1555 -> (none); LCSC Part (none) -> C1555
- C124, C125, C126, C127: LCSC C86295 -> (none); LCSC Part (none) -> C86295
- D101, D102: LCSC C668989 -> (none); LCSC Part (none) -> C668989
- J101: LCSC C3975129 -> (none); LCSC Part (none) -> C3975129
- J102: LCSC C145795 -> (none); LCSC Part (none) -> C145795
- J103: LCSC C160389 -> (none); LCSC Part (none) -> C160389
- Q101: LCSC C15127 -> (none); LCSC Part (none) -> C15127
- R101, R111, R115: LCSC C25741 -> (none); LCSC Part (none) -> C25741
- R102, R103, R104, R110, R127: LCSC C25092 -> (none); LCSC Part (none) -> C25092
- R105, R107: LCSC C25744 -> (none); LCSC Part (none) -> C25744
- R106, R109, R113, R114: LCSC C11702 -> (none); LCSC Part (none) -> C11702
- R112: LCSC C38941 -> (none); LCSC Part (none) -> C38941
- U101: LCSC C97521 -> (none); LCSC Part (none) -> C97521
- U102: LCSC C2040 -> (none); LCSC Part (none) -> C2040
- U103: LCSC C410863 -> (none); LCSC Part (none) -> C410863
- U104: LCSC C2757850 -> (none); LCSC Part (none) -> C2757850
- U105: LCSC C7440 -> (none); LCSC Part (none) -> C7440
- U106: LCSC C7562 -> (none); LCSC Part (none) -> C7562
- U121, U122, U123, U124: LCSC C238203 -> (none)
- Y101: LCSC C9002 -> (none); LCSC Part (none) -> C9002
- Y102: LCSC C32346 -> (none); LCSC Part (none) -> C32346
Changed lines of the file:
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@@
 			)
 		)
-		(property "LCSC" "C25741"
+		(property "LCSC Part" "C25741"
 			(at 58.42 58.42 0)
 			(effects
@@
 			)
 		)
-		(property "LCSC" "C238203"
+		(property "LCSC Part" "C238203"
 			(at 48.26 205.74 0)
 			(effects
@@
 			)
 		)
-		(property "LCSC" "C25092"
+		(property "LCSC Part" "C25092"
 			(at 236.22 78.74 0)
 			(effects
@@
 			)
 		)
-		(property "LCSC" "C15127"
+		(property "LCSC Part" "C15127"
 			(at 64.77 55.88 0)
 			(effects
@@
 			)
 		)
-		(property "LCSC" "C86295"
+		(property "LCSC Part" "C86295"
 			(at 97.79 267.97 0)
 			(effects
@@
 			)
 		)
-		(property "LCSC" "C16772"
+		(property "LCSC Part" "C16772"
 			(at 269.24 43.18 0)
 			(effects
@@
 			)
 		)
-		(property "LCSC" "C16772"
+		(property "LCSC Part" "C16772"
 			(at 257.81 43.18 0)
 			(effects
@@
 			)
 		)
-		(property "LCSC" "C32346"
+		(property "LCSC Part" "C32346"
 			(at 349.25 237.49 90)
 			(effects
@@
 			)
 		)
-		(property "LCSC" "C16772"
+		(property "LCSC Part" "C16772"
 			(at 203.2 233.68 0)
 			(effects
@@
 			)
 		)
-		(property "LCSC" "C11702"
+		(property "LCSC Part" "C11702"
 			(at 355.6 226.06 0)
 			(effects
@@
 			)
 		)
-		(property "LCSC" "C16772"
+		(property "LCSC Part" "C16772"
 			(at 246.38 43.18 0)
 			(effects
@@
 			)
 		)
-		(property "LCSC" "C25092"
+		(property "LCSC Part" "C25092"
 			(at 236.22 91.44 0)
 			(effects
@@
 			)
 		)
-		(property "LCSC" "C7440"
+		(property "LCSC Part" "C7440"
 			(at 372.11 237.49 0)
 			(effects
@@
 			)
 		)
-		(property "LCSC" "C19702"
+		(property "LCSC Part" "C19702"
 			(at 363.22 190.5 0)
 			(effects
@@
 			)
 		)
-		(property "LCSC" "C25092"
+		(property "LCSC Part" "C25092"
 			(at 241.3 132.08 0)
 			(effects
@@
 			)
 		)
-		(property "LCSC" "C1555"
+		(property "LCSC Part" "C1555"
 			(at 339.09 246.38 0)
 			(effects
@@
 			)
 		)
-		(property "LCSC" "C16772"
+		(property "LCSC Part" "C16772"
 			(at 234.95 43.18 0)
 			(effects
@@
 			)
 		)
-		(property "LCSC" "C1547"
+		(property "LCSC Part" "C1547"
 			(at 121.92 129.54 0)
 			(effects
@@
 			)
 		)
-		(property "LCSC" "C25092"
+		(property "LCSC Part" "C25092"
 			(at 236.22 127 0)
 			(effects
@@
 			)
 		)
-		(property "LCSC" "C25092"
+		(property "LCSC Part" "C25092"
 			(at 236.22 81.28 0)
 			(effects
@@
 			)
 		)
-		(property "LCSC" "C11702"
+		(property "LCSC Part" "C11702"
 			(at 311.15 226.06 0)
 			(effects
@@
 			)
 		)
-		(property "LCSC" "C160389"
+		(property "LCSC Part" "C160389"
 			(at 46.99 161.29 0)
 			(effects
@@
 			)
 		)
-		(property "LCSC" "C86295"
+		(property "LCSC Part" "C86295"
 			(at 107.95 267.97 0)
 			(effects
@@
 			)
 		)
-		(property "LCSC" "C1547"
+		(property "LCSC Part" "C1547"
 			(at 121.92 119.38 0)
 			(effects
@@
 			)
 		)
-		(property "LCSC" "C25741"
+		(property "LCSC Part" "C25741"
 			(at 349.25 135.89 0)
 			(effects
@@
 			)
 		)
-		(property "Description" ""
+		(property "Description" "128Mb Serial Flash Memory, Standard/Dual/Quad SPI, SOIC-8"
 			(at 78.74 120.65 0)
 			(effects
@@
 			)
 		)
-		(property "LCSC" "C97521"
+		(property "LCSC Part" "C97521"
 			(at 78.74 120.65 0)
 			(effects
@@
 			)
 		)
+		(property "JLCPCB" ""
+			(at 78.74 120.65 0)
+			(effects
+				(font
+					(size 1.27 1.27)
+				)
+				(hide yes)
+			)
+		)
 		(pin "1"
 		)
@@
 			)
 		)
-		(property "LCSC" "C9002"
+		(property "LCSC Part" "C9002"
 			(at 134.62 124.46 0)
 			(effects
@@
 			)
 		)
-		(property "LCSC" "C145795"
+		(property "LCSC Part" "C145795"
 			(at 308.61 81.28 0)
 			(effects
@@
 			)
 		)
-		(property "LCSC" "C16772"
+		(property "LCSC Part" "C16772"
 			(at 394.97 36.83 0)
 			(effects
@@
 			)
 		)
-		(property "LCSC" "C25744"
+		(property "LCSC Part" "C25744"
 			(at 382.27 99.06 0)
 			(effects
@@
 			)
 		)
-		(property "LCSC" "C238203"
+		(property "LCSC Part" "C238203"
 			(at 48.26 199.39 0)
 			(effects
@@
 			)
 		)
-		(property "LCSC" "C19702"
+		(property "LCSC Part" "C19702"
 			(at 44.45 58.42 0)
 			(effects
@@
 			)
 		)
-		(property "LCSC" "C16772"
+		(property "LCSC Part" "C16772"
 			(at 223.52 43.18 0)
 			(effects
@@
 			)
 		)
-		(property "LCSC" "C52923"
+		(property "LCSC Part" "C52923"
 			(at 200.66 58.42 0)
 			(effects
@@
 			)
 		)
-		(property "LCSC" "C668989"
+		(property "LCSC Part" "C668989"
 			(at 302.26 226.06 0)
 			(effects
@@
 			)
 		)
-		(property "LCSC" "C16772"
+		(property "LCSC Part" "C16772"
 			(at 85.09 99.06 0)
 			(effects
@@
 			)
 		)
-		(property "LCSC" "C1555"
+		(property "LCSC Part" "C1555"
 			(at 349.25 246.38 0)
 			(effects
@@
 			)
 		)
-		(property "LCSC" "C238203"
+		(property "LCSC Part" "C238203"
 			(at 48.26 193.04 0)
 			(effects
@@
 			)
 		)
-		(property "LCSC" "C16772"
+		(property "LCSC Part" "C16772"
 			(at 134.62 43.18 0)
 			(effects
@@
 			)
 		)
-		(property "LCSC" "C86295"
+		(property "LCSC Part" "C86295"
 			(at 140.97 267.97 0)
 			(effects
@@
 			)
 		)
-		(property "LCSC" "C19702"
+		(property "LCSC Part" "C19702"
 			(at 383.54 222.25 0)
 			(effects
@@
 			)
 		)
-		(property "LCSC" "C1555"
+		(property "LCSC Part" "C1555"
 			(at 292.1 229.87 0)
 			(effects
@@
 			)
 		)
-		(property "LCSC" "C52923"
+		(property "LCSC Part" "C52923"
 			(at 146.05 58.42 0)
 			(effects
@@
 			)
 		)
-		(property "LCSC" "C11702"
+		(property "LCSC Part" "C11702"
 			(at 236.22 96.52 0)
 			(effects
@@
 			)
 		)
-		(property "LCSC" "C86295"
+		(property "LCSC Part" "C86295"
 			(at 130.81 267.97 0)
 			(effects
@@
 			)
 		)
-		(property "LCSC" "C3975129"
+		(property "LCSC Part" "C3975129"
 			(at 382.27 33.02 0)
 			(effects
@@
 			)
 		)
-		(property "LCSC" "C2040"
+		(property "LCSC Part" "C2040"
 			(at 175.26 121.92 0)
 			(effects
@@
 			)
 		)
-		(property "LCSC" "C80909"
+		(property "LCSC Part" "C80909"
 			(at 317.5 232.41 0)
 			(effects
@@
 			)
 		)
-		(property "LCSC" "C52923"
+		(property "LCSC Part" "C52923"
 			(at 353.06 190.5 0)
 			(effects
@@
 			)
 		)
-		(property "LCSC" "C7562"
+		(property "LCSC Part" "C7562"
 			(at 207.01 246.38 0)
 			(effects
@@
 			)
 		)
-		(property "LCSC" "C410863"
+		(property "LCSC Part" "C410863"
 			(at 368.3 144.78 0)
 			(effects
@@
 			)
 		)
-		(property "LCSC" "C25744"
+		(property "LCSC Part" "C25744"
 			(at 382.27 93.98 0)
 			(effects
@@
 			)
 		)
-		(property "LCSC" "C16772"
+		(property "LCSC Part" "C16772"
 			(at 212.09 43.18 0)
 			(effects
@@
 			)
 		)
-		(property "LCSC" "C16772"
+		(property "LCSC Part" "C16772"
 			(at 393.7 132.08 0)
 			(effects
@@
 			)
 		)
-		(property "LCSC" "C16772"
+		(property "LCSC Part" "C16772"
 			(at 200.66 43.18 0)
 			(effects
@@
 			)
 		)
-		(property "LCSC" "C25741"
+		(property "LCSC Part" "C25741"
 			(at 242.57 243.84 0)
 			(effects
@@
 			)
 		)
-		(property "LCSC" "C19702"
+		(property "LCSC Part" "C19702"
 			(at 72.39 57.15 0)
 			(effects
@@
 			)
 		)
-		(property "LCSC" "C11702"
+		(property "LCSC Part" "C11702"
 			(at 48.26 118.11 0)
 			(effects
@@
 			)
 		)
-		(property "LCSC" "C668989"
+		(property "LCSC Part" "C668989"
 			(at 365.76 218.44 0)
 			(effects
@@
 			)
 		)
-		(property "LCSC" "C16772"
+		(property "LCSC Part" "C16772"
 			(at 146.05 43.18 0)
 			(effects
@@
 			)
 		)
-		(property "LCSC" "C2757850"
+		(property "LCSC Part" "C2757850"
 			(at 386.08 185.42 0)
 			(effects
@@
 			)
 		)
-		(property "LCSC" "C38941"
+		(property "LCSC Part" "C38941"
 			(at 358.14 185.42 0)
 			(effects
@@
 			)
 		)
-		(property "LCSC" "C238203"
+		(property "LCSC Part" "C238203"
 			(at 48.26 212.09 0)
 			(effects
