File: tc2-main-pcb/tc2-main-pcb.kicad_sch (KiCad schematic)
At the start: 83 parts, among them J101 Conn_02x03_Odd_Even, J102 USB_B_Micro, J103 Conn_01x03, J104 Conn_02x06_Odd_Even, Q101 Q_PMOS_GSD, U101 W25Q128JVS, U102 RP2040, U103 MT29F2G01ABAGDWB-IT, U104 AHT20_C2757850, U105 PCF8563T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

Commit message: Tidy up for making an order for v0.7.3
Parts:
- BT101: LCSC C80909 -> (none); LCSC Part (none) -> C80909
- C101, C102, C103, C104, C105, C106, C107, C108, C109, C114, C117, C121: LCSC C16772 -> (none); LCSC Part (none) -> C16772
- C110, C111, C119, C120: LCSC C19702 -> (none); LCSC Part (none) -> C19702
- C112, C113, C118: value 1u -> 1uF; LCSC C52923 -> (none); LCSC Part (none) -> C52923
- C115, C116: LCSC C1547 -> (none); LCSC Part (none) -> C1547
- C122, C123: LCSC C1555 -> (none); LCSC Part (none) -> C1555
- C124, C125, C126, C127: LCSC C86295 -> (none); LCSC Part (none) -> C86295
- D101, D102: LCSC C668989 -> (none); LCSC Part (none) -> C668989
- J101: LCSC C3975129 -> (none); LCSC Part (none) -> C3975129
- J102: LCSC C145795 -> (none); LCSC Part (none) -> C145795
- J103: LCSC C160389 -> (none); LCSC Part (none) -> C160389
- J104: LCSC C6470934 -> (none); LCSC Part (none) -> C6470934
- Q101: LCSC C15127 -> (none); LCSC Part (none) -> C15127
- R101, R111, R115: LCSC C25741 -> (none); LCSC Part (none) -> C25741
- R102, R103, R104, R110: value 22ohm -> 22Ω; LCSC C25092 -> (none); LCSC Part (none) -> C25092
- R105, R107: LCSC C25744 -> (none); LCSC Part (none) -> C25744
- R106, R109, R113, R114: LCSC C11702 -> (none); LCSC Part (none) -> C11702
- R112: value 180R -> 180Ω; LCSC C38941 -> (none); LCSC Part (none) -> C38941
- U101: LCSC C97521 -> (none)
- U102: LCSC C2040 -> (none)
- U103: LCSC C410863 -> (none); LCSC Part (none) -> C410863
- U104: LCSC C2757850 -> (none); LCSC Part (none) -> C2757850
- U105: LCSC C7440 -> (none); LCSC Part (none) -> C7440
- U106: LCSC C7562 -> (none); LCSC Part (none) -> C7562
- Y101: LCSC C9002 -> (none); LCSC Part (none) -> C9002
- Y102: LCSC C32346 -> (none); LCSC Part (none) -> C32346
Changed lines of the file:
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@@
 			)
 		)
-		(property "LCSC" "C25741"
+		(property "LCSC Part" "C25741"
 			(at 58.42 58.42 0)
 			(effects
@@
 			)
 		)
-		(property "LCSC" "C6470934"
+		(property "LCSC Part" "C6470934"
 			(at 46.99 267.97 0)
 			(effects
@@
 			)
 		)
-		(property "Value" "22ohm"
+		(property "Value" "22Ω"
 			(at 242.57 77.47 90)
 			(effects
@@
 			)
 		)
-		(property "LCSC" "C25092"
+		(property "LCSC Part" "C25092"
 			(at 236.22 78.74 0)
 			(effects
@@
 			)
 		)
-		(property "LCSC" "C15127"
+		(property "LCSC Part" "C15127"
 			(at 64.77 55.88 0)
 			(effects
@@
 			)
 		)
-		(property "LCSC" "C86295"
+		(property "LCSC Part" "C86295"
 			(at 97.79 267.97 0)
 			(effects
@@
 			)
 		)
-		(property "LCSC" "C16772"
+		(property "LCSC Part" "C16772"
 			(at 269.24 43.18 0)
 			(effects
@@
 			)
 		)
-		(property "LCSC" "C16772"
+		(property "LCSC Part" "C16772"
 			(at 257.81 43.18 0)
 			(effects
@@
 			)
 		)
-		(property "LCSC" "C32346"
+		(property "LCSC Part" "C32346"
 			(at 349.25 237.49 90)
 			(effects
@@
 			)
 		)
-		(property "LCSC" "C16772"
+		(property "LCSC Part" "C16772"
 			(at 203.2 233.68 0)
 			(effects
@@
 			)
 		)
-		(property "LCSC" "C11702"
+		(property "LCSC Part" "C11702"
 			(at 355.6 226.06 0)
 			(effects
@@
 			)
 		)
-		(property "LCSC" "C16772"
+		(property "LCSC Part" "C16772"
 			(at 246.38 43.18 0)
 			(effects
@@
 			)
 		)
-		(property "Value" "22ohm"
+		(property "Value" "22Ω"
 			(at 242.57 90.17 90)
 			(effects
@@
 			)
 		)
-		(property "LCSC" "C25092"
+		(property "LCSC Part" "C25092"
 			(at 236.22 91.44 0)
 			(effects
@@
 			)
 		)
-		(property "LCSC" "C7440"
+		(property "LCSC Part" "C7440"
 			(at 372.11 237.49 0)
 			(effects
@@
 			)
 		)
-		(property "LCSC" "C19702"
+		(property "LCSC Part" "C19702"
 			(at 363.22 190.5 0)
 			(effects
@@
 			)
 		)
-		(property "LCSC" "C1555"
+		(property "LCSC Part" "C1555"
 			(at 339.09 246.38 0)
 			(effects
@@
 			)
 		)
-		(property "LCSC" "C16772"
+		(property "LCSC Part" "C16772"
 			(at 234.95 43.18 0)
 			(effects
@@
 			)
 		)
-		(property "LCSC" "C1547"
+		(property "LCSC Part" "C1547"
 			(at 121.92 129.54 0)
 			(effects
@@
 			)
 		)
-		(property "Value" "22ohm"
+		(property "Value" "22Ω"
 			(at 242.57 125.73 90)
 			(effects
@@
 			)
 		)
-		(property "LCSC" "C25092"
+		(property "LCSC Part" "C25092"
 			(at 236.22 127 0)
 			(effects
@@
 			)
 		)
-		(property "Value" "22ohm"
+		(property "Value" "22Ω"
 			(at 242.57 80.01 90)
 			(effects
@@
 			)
 		)
-		(property "LCSC" "C25092"
+		(property "LCSC Part" "C25092"
 			(at 236.22 81.28 0)
 			(effects
@@
 			)
 		)
-		(property "LCSC" "C11702"
+		(property "LCSC Part" "C11702"
 			(at 311.15 226.06 0)
 			(effects
@@
 			)
 		)
-		(property "LCSC" "C160389"
+		(property "LCSC Part" "C160389"
 			(at 46.99 161.29 0)
 			(effects
@@
 			)
 		)
-		(property "LCSC" "C86295"
+		(property "LCSC Part" "C86295"
 			(at 107.95 267.97 0)
 			(effects
@@
 			)
 		)
-		(property "LCSC" "C1547"
+		(property "LCSC Part" "C1547"
 			(at 121.92 119.38 0)
 			(effects
@@
 			)
 		)
-		(property "LCSC" "C25741"
+		(property "LCSC Part" "C25741"
 			(at 349.25 135.89 0)
 			(effects
@@
 			)
 		)
-		(property "LCSC" "C97521"
+		(property "LCSC Part" "C97521"
 			(at 78.74 120.65 0)
 			(effects
@@
 			)
 		)
-		(property "LCSC" "C9002"
+		(property "LCSC Part" "C9002"
 			(at 134.62 124.46 0)
 			(effects
@@
 			)
 		)
-		(property "LCSC" "C145795"
+		(property "LCSC Part" "C145795"
 			(at 308.61 81.28 0)
 			(effects
@@
 			)
 		)
-		(property "LCSC" "C25744"
+		(property "LCSC Part" "C25744"
 			(at 382.27 99.06 0)
 			(effects
@@
 			)
 		)
-		(property "LCSC" "C19702"
+		(property "LCSC Part" "C19702"
 			(at 44.45 58.42 0)
 			(effects
@@
 			)
 		)
-		(property "LCSC" "C16772"
+		(property "LCSC Part" "C16772"
 			(at 223.52 43.18 0)
 			(effects
@@
 			)
 		)
-		(property "Value" "1u"
+		(property "Value" "1uF"
 			(at 203.581 59.563 0)
 			(effects
@@
 			)
 		)
-		(property "LCSC" "C52923"
+		(property "LCSC Part" "C52923"
 			(at 200.66 58.42 0)
 			(effects
@@
 			)
 		)
-		(property "LCSC" "C668989"
+		(property "LCSC Part" "C668989"
 			(at 302.26 226.06 0)
 			(effects
@@
 			)
 		)
-		(property "LCSC" "C16772"
+		(property "LCSC Part" "C16772"
 			(at 85.09 99.06 0)
 			(effects
@@
 			)
 		)
-		(property "LCSC" "C1555"
+		(property "LCSC Part" "C1555"
 			(at 349.25 246.38 0)
 			(effects
@@
 			)
 		)
-		(property "LCSC" "C16772"
+		(property "LCSC Part" "C16772"
 			(at 134.62 43.18 0)
 			(effects
@@
 			)
 		)
-		(property "LCSC" "C86295"
+		(property "LCSC Part" "C86295"
 			(at 140.97 267.97 0)
 			(effects
@@
 			)
 		)
-		(property "LCSC" "C19702"
+		(property "LCSC Part" "C19702"
 			(at 383.54 222.25 0)
 			(effects
@@
 			)
 		)
-		(property "Value" "1u"
+		(property "Value" "1uF"
 			(at 148.971 59.563 0)
 			(effects
@@
 			)
 		)
-		(property "LCSC" "C52923"
+		(property "LCSC Part" "C52923"
 			(at 146.05 58.42 0)
 			(effects
@@
 			)
 		)
-		(property "LCSC" "C11702"
+		(property "LCSC Part" "C11702"
 			(at 236.22 96.52 0)
 			(effects
@@
 			)
 		)
-		(property "LCSC" "C86295"
+		(property "LCSC Part" "C86295"
 			(at 130.81 267.97 0)
 			(effects
@@
 			)
 		)
-		(property "LCSC" "C3975129"
+		(property "LCSC Part" "C3975129"
 			(at 382.27 33.02 0)
 			(effects
@@
 			)
 		)
-		(property "LCSC" "C2040"
+		(property "LCSC Part" "C2040"
 			(at 175.26 121.92 0)
 			(effects
@@
 			)
 		)
-		(property "LCSC" "C80909"
+		(property "LCSC Part" "C80909"
 			(at 317.5 232.41 0)
 			(effects
@@
 			)
 		)
-		(property "Value" "1u"
+		(property "Value" "1uF"
 			(at 355.981 191.643 0)
 			(effects
@@
 			)
 		)
-		(property "LCSC" "C52923"
+		(property "LCSC Part" "C52923"
 			(at 353.06 190.5 0)
 			(effects
@@
 			)
 		)
-		(property "LCSC" "C7562"
+		(property "LCSC Part" "C7562"
 			(at 207.01 246.38 0)
 			(effects
@@
 			)
 		)
-		(property "LCSC" "C410863"
+		(property "LCSC Part" "C410863"
 			(at 368.3 144.78 0)
 			(effects
@@
 			)
 		)
-		(property "LCSC" "C25744"
+		(property "LCSC Part" "C25744"
 			(at 382.27 93.98 0)
 			(effects
@@
 			)
 		)
-		(property "LCSC" "C16772"
+		(property "LCSC Part" "C16772"
 			(at 212.09 43.18 0)
 			(effects
@@
 			)
 		)
-		(property "LCSC" "C16772"
+		(property "LCSC Part" "C16772"
 			(at 393.7 132.08 0)
 			(effects
@@
 			)
 		)
-		(property "LCSC" "C16772"
+		(property "LCSC Part" "C16772"
 			(at 200.66 43.18 0)
 			(effects
@@
 			)
 		)
-		(property "LCSC" "C25741"
+		(property "LCSC Part" "C25741"
 			(at 242.57 243.84 0)
 			(effects
@@
 			)
 		)
-		(property "LCSC" "C19702"
+		(property "LCSC Part" "C19702"
 			(at 72.39 57.15 0)
 			(effects
@@
 			)
 		)
-		(property "LCSC" "C11702"
+		(property "LCSC Part" "C11702"
 			(at 48.26 118.11 0)
 			(effects
@@
 			)
 		)
-		(property "LCSC" "C668989"
+		(property "LCSC Part" "C668989"
 			(at 365.76 218.44 0)
 			(effects
@@
 			)
 		)
-		(property "LCSC" "C16772"
+		(property "LCSC Part" "C16772"
 			(at 146.05 43.18 0)
 			(effects
@@
 			)
 		)
-		(property "LCSC" "C2757850"
+		(property "LCSC Part" "C2757850"
 			(at 386.08 185.42 0)
 			(effects
@@
 			)
 		)
-		(property "Value" "180R"
+		(property "Value" "180Ω"
 			(at 360.68 180.34 90)
 			(effects
@@
 			)
 		)
-		(property "LCSC" "C38941"
+		(property "LCSC Part" "C38941"
 			(at 358.14 185.42 0)
 			(effects
