File: tc2-main-pcb/raspberry_pi.kicad_sch (KiCad schematic)
At the start: 36 parts, among them J105 Screw_Terminal_01x01, J106 Screw_Terminal_01x01, J107 Screw_Terminal_01x01, J108 Screw_Terminal_01x01, J109 Screw_Terminal_01x01, J110 Raspberry_Pi_2_3, U107 MAX98357AEWL+T, U108 TCA4311ADGKR, U109 74HC4052

Commit message: Tidy up for making an order for v0.7.3
Parts:
- C128, C132: LCSC C19702 -> (none); LCSC Part (none) -> C19702
- C129, C130: LCSC C16772 -> (none); LCSC Part (none) -> C16772
- C131: LCSC C86295 -> (none); LCSC Part (none) -> C86295
- J105, J106, J107, J108, J109: LCSC C2915630 -> (none); LCSC Part (none) -> C2915630
- J110: LCSC C350295 -> (none); LCSC Part (none) -> C350295
- R116: LCSC C326730 -> (none); LCSC Part (none) -> C326730
- R117, R125, R126: LCSC C25741 -> (none); LCSC Part (none) -> C25741
- R118: LCSC C11702 -> (none); LCSC Part (none) -> C11702
- R119, R120, R121, R122, R123, R124: value 22ohm -> 22Ω; LCSC C25092 -> (none); LCSC Part (none) -> C25092
- U107: LCSC C2682619 -> (none); LCSC Part (none) -> C2682619
- U108: LCSC C130025 -> (none); LCSC Part (none) -> C130025
- U109: LCSC C111594 -> (none); LCSC Part (none) -> C111594
Changed lines of the file:
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@@
 			)
 		)
-		(property "LCSC Part" ""
-			(at 93.98 60.96 0)
-			(effects
-				(font
-					(size 1.27 1.27)
-				)
-				(hide yes)
-			)
-		)
 		(property "JLC Part" "Extended Part"
 			(at 93.98 63.5 0)
@@
 			)
 		)
-		(property "LCSC" "C2682619 "
+		(property "LCSC Part" "C2682619 "
 			(at 93.98 40.64 0)
 			(effects
@@
 			)
 		)
-		(property "LCSC" "C2915630"
+		(property "LCSC Part" "C2915630"
 			(at 276.86 82.55 0)
 			(effects
@@
 			)
 		)
-		(property "Value" "22ohm"
+		(property "Value" "22Ω"
 			(at 139.7 121.92 90)
 			(effects
@@
 			)
 		)
-		(property "LCSC" "C25092"
+		(property "LCSC Part" "C25092"
 			(at 133.35 123.19 0)
 			(effects
@@
 			)
 		)
-		(property "LCSC" "C16772"
+		(property "LCSC Part" "C16772"
 			(at 191.77 26.67 0)
 			(effects
@@
 			)
 		)
-		(property "LCSC" "C25741"
+		(property "LCSC Part" "C25741"
 			(at 189.23 53.34 0)
 			(effects
@@
 			)
 		)
-		(property "LCSC" "C11702"
+		(property "LCSC Part" "C11702"
 			(at 143.51 100.33 0)
 			(effects
@@
 			)
 		)
-		(property "LCSC Part" ""
-			(at 172.72 59.69 0)
-			(effects
-				(font
-					(size 1.27 1.27)
-				)
-				(hide yes)
-			)
-		)
-		(property "LCSC" "C130025"
+		(property "LCSC Part" "C130025"
 			(at 172.72 40.64 0)
 			(effects
@@
 			)
 		)
-		(property "LCSC" "C25741"
+		(property "LCSC Part" "C25741"
 			(at 31.75 170.18 0)
 			(effects
@@
 			)
 		)
-		(property "Value" "22ohm"
+		(property "Value" "22Ω"
 			(at 219.71 132.08 90)
 			(effects
@@
 			)
 		)
-		(property "LCSC" "C25092"
+		(property "LCSC Part" "C25092"
 			(at 213.36 133.35 0)
 			(effects
@@
 			)
 		)
-		(property "LCSC" "C2915630"
+		(property "LCSC Part" "C2915630"
 			(at 248.92 78.74 0)
 			(effects
@@
 			)
 		)
-		(property "LCSC" "C326730"
+		(property "LCSC Part" "C326730"
 			(at 68.58 35.56 90)
 			(effects
@@
 			)
 		)
-		(property "LCSC" "C86295"
+		(property "LCSC Part" "C86295"
 			(at 153.67 82.55 0)
 			(effects
@@
 			)
 		)
-		(property "LCSC" "C2915630"
+		(property "LCSC Part" "C2915630"
 			(at 276.86 46.99 0)
 			(effects
@@
 			)
 		)
-		(property "Value" "22ohm"
+		(property "Value" "22Ω"
 			(at 139.7 116.84 90)
 			(effects
@@
 			)
 		)
-		(property "LCSC" "C25092"
+		(property "LCSC Part" "C25092"
 			(at 133.35 118.11 0)
 			(effects
@@
 			)
 		)
-		(property "LCSC" "C19702"
+		(property "LCSC Part" "C19702"
 			(at 24.13 43.18 0)
 			(effects
@@
 			)
 		)
-		(property "LCSC" "C2915630"
+		(property "LCSC Part" "C2915630"
 			(at 262.89 46.99 0)
 			(effects
@@
 			)
 		)
-		(property "LCSC" "C350295"
+		(property "LCSC Part" "C350295"
 			(at 168.91 123.19 0)
 			(effects
@@
 			)
 		)
-		(property "LCSC" "C16772"
+		(property "LCSC Part" "C16772"
 			(at 31.75 43.18 0)
 			(effects
@@
 			)
 		)
-		(property "Value" "22ohm"
+		(property "Value" "22Ω"
 			(at 139.7 111.76 90)
 			(effects
@@
 			)
 		)
-		(property "LCSC" "C25092"
+		(property "LCSC Part" "C25092"
 			(at 133.35 113.03 0)
 			(effects
@@
 			)
 		)
-		(property "Value" "22ohm"
+		(property "Value" "22Ω"
 			(at 219.71 127 90)
 			(effects
@@
 			)
 		)
-		(property "LCSC" "C25092"
+		(property "LCSC Part" "C25092"
 			(at 213.36 128.27 0)
 			(effects
@@
 			)
 		)
-		(property "LCSC" "C19702"
+		(property "LCSC Part" "C19702"
 			(at 92.71 142.24 0)
 			(effects
@@
 			)
 		)
-		(property "LCSC" "C25741"
+		(property "LCSC Part" "C25741"
 			(at 87.63 175.26 0)
 			(effects
@@
 			)
 		)
-		(property "LCSC Part" ""
-			(at 73.66 182.88 0)
-			(effects
-				(font
-					(size 1.27 1.27)
-				)
-				(hide yes)
-			)
-		)
-		(property "LCSC" "C111594"
+		(property "LCSC Part" "C111594"
 			(at 73.66 161.29 0)
 			(effects
@@
 			)
 		)
-		(property "Value" "22ohm"
+		(property "Value" "22Ω"
 			(at 219.71 134.62 90)
 			(effects
@@
 			)
 		)
-		(property "LCSC" "C25092"
+		(property "LCSC Part" "C25092"
 			(at 213.36 135.89 0)
 			(effects
@@
 			)
 		)
-		(property "LCSC" "C2915630"
+		(property "LCSC Part" "C2915630"
 			(at 248.92 46.99 0)
 			(effects
