File: tc2-main-pcb/raspberry_pi.kicad_sch (KiCad schematic)
At the start: 36 parts, among them J105 Screw_Terminal_01x01, J106 Screw_Terminal_01x01, J107 Screw_Terminal_01x01, J108 Screw_Terminal_01x01, J109 Screw_Terminal_01x01, J110 Raspberry_Pi_2_3, U107 MAX98357AEWL+T, U108 TCA4311ADGKR, U109 74HC4052

Commit message: Fix library
Parts:
- U109: footprint Package_SO:SOP-16_3.9x9.9mm_P1.27mm -> cacophony-library:SOP-16_L10.0-W3.9-P1.27-LS6.0-BL
Changed lines of the file:
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@@
 			)
 		)
-		(property "Footprint" "Package_SO:SOP-16_3.9x9.9mm_P1.27mm"
+		(property "Footprint" "cacophony-library:SOP-16_L10.0-W3.9-P1.27-LS6.0-BL"
 			(at 73.66 177.8 0)
 			(hide yes)

Commit message: Update schematic
Parts:
- removed R117: 100k, Resistor_SMD:R_0402_1005Metric, symbol Device:R
- removed TP120, TP122: TestPoint, cacophony-library:TP, symbol Connector:TestPoint
- removed TP121: TestPoint, TestPoint:TestPoint_Pad_D1.0mm, symbol Connector:TestPoint
- removed U108: TCA4311ADGKR, Package_SO:MSOP-8_3x3mm_P0.65mm, symbol cacophony-library:TCA4311ADGKR
- added R127, R128: 10k, Resistor_SMD:R_0402_1005Metric, symbol Device:R
- added R130: 100k, Resistor_SMD:R_0402_1005Metric, symbol Device:R
- added U2: PCA9517ADP,118, Package_SO:MSOP-8_3x3mm_P0.65mm, symbol cacophony-library:PCA9517ADP,118
- U107: LCSC Part C2682619 -> C2682619
- U109: footprint cacophony-library:SOP-16_L10.0-W3.9-P1.27-LS6.0-BL -> Package_SO:SOIC-16_3.9x9.9mm_P1.27mm; LCSC Part C111594 -> C11350
Connections:
- net +3V3: now also R127.2, R128.2, U2.1 (VCCA), U2.8 (VCCB)
- net GND: now also R130.1, U2.4 (GND)
- net MUL_S0: now also R130.2
- net RPI_SCL: now also R127.1, U2.7 (SCLB)
- net RPI_SDA: now also R128.1, U2.6 (SDAB)
- net SCL: now also U2.2 (SCLA)
- net SDA: now also U2.3 (SDAA)
- new net EN_RPI_I2C: U2.5 (EN)
Other:
- moved on the sheet: C128, C129, C130, C132, J105, J106, J107, J108, J109, R116, R125, R126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
