File: tc2-mic-pcb/tc2-mic-pcb.kicad_pcb (KiCad board)
At the start: 2 copper layers, 31 x 13.5 mm, 9 parts, among them J1 Screw_Terminal_01x01, J2 Screw_Terminal_01x01, J4 Conn_02x03_Odd_Even, U1 ME6211, U2 SPH0645LM4H

Commit message: Version 2 WIP
Parts:
- removed U1: ME6211, Package_TO_SOT_SMD:SOT-23-5
- added C4: 1uF, Capacitor_SMD:C_0402_1005Metric, F.Cu at (111.7, 107.1)
- added C5: 1uF, Capacitor_SMD:C_0402_1005Metric, F.Cu at (108.2, 107.1)
- added MK1: SPH0641LU4H-1, Sensor_Audio:Knowles_LGA-5_3.5x2.65mm, F.Cu at (112.8, 110.0)
- added R2: 22R, Resistor_SMD:R_0402_1005Metric, F.Cu at (125.0, 110.8)
- added R3: 22R, Resistor_SMD:R_0402_1005Metric, F.Cu at (118.0, 109.2)
- added U3: AP7335-18SNG-7, cacophony-library:U-DFN2020-6_L2.0-W2.0-P0.65-BL-EP, F.Cu at (109.9, 107.0)
- C1: value 1uF -> 100nF
- C2: value 220nF -> 100nF; footprint Capacitor_SMD:C_0402_1005Metric -> Capacitor_SMD:C_1206_3216Metric
- C3: value 12pF -> 100nF
- R1: value 22ohm -> 22R
- U2: value SPH0645LM4H -> TXS0102DCT; footprint cacophony-library:MIC_SPH0645LM4H-B -> Package_SO:SSOP-8_2.95x2.8mm_P0.65mm
- moved U2 39.6 mm to (124.5, 108.7), turned to 0 degrees
- moved C3 39.5 mm to (127.7, 108.7)
- moved R1 32.1 mm to (120.8, 107.1), turned to 180 degrees
- moved C1 28.8 mm to (121.3, 108.5), turned to 90 degrees
- moved J4 27.4 mm to (120.7, 104.0), turned to 180 degrees
- moved J1 27.3 mm to (127.0, 104.0)
- moved J2 27.3 mm to (104.0, 110.0)
- moved C2 26.8 mm to (115.9, 109.3), turned to 90 degrees
Connections:
- C1 pad 1: GND -> +1V8
- C1 pad 2: +5V -> GND
- C2 pad 1: GND -> +1V8
- C2 pad 2: +3V3_Lin -> GND
- C3 pad 1: GND -> +3V3
- C3 pad 2: +3V3_Lin -> GND
- J1 pad 1: unconnected-(J1-Pin_1-Pad1) -> GND
- J2 pad 1: unconnected-(J2-Pin_1-Pad1) -> GND
- J4 pad 1: I2S_LRCLK -> PDM_CLOCK
- J4 pad 2: +5V -> GND
- J4 pad 4: I2S_DIN -> +3V3
- J4 pad 5: I2S_BCLK -> PDM_DATA
- R1 pad 1: Net-(U2-DATA) -> /PDM_DATA_
- R1 pad 2: I2S_DIN -> PDM_DATA
- U2 pad 1: I2S_LRCLK -> /PDM_DATA_
- U2 pad 3: GND -> +1V8
- U2 pad 4: I2S_BCLK -> /DATA
- U2 pad 5: +3V3_Lin -> /CLOCK_
- U2 pad 6: Net-(U2-DATA) -> +3V3
Routing:
- net +1V8: track 0.00 -> 24.7 mm
- net +3V3: track 0.00 -> 24.4 mm
- net I2S_BCLK: track 19.4 -> 0.00 mm
- net /CLOCK: track 0.00 -> 12.4 mm
- net I2S_LRCLK: track 12.0 -> 0.00 mm
- net +5V: track 11.0 -> 0.00 mm
- net I2S_DIN: track 6.48 -> 0.00 mm
- net PDM_DATA: track 0.00 -> 6.14 mm
- net PDM_CLOCK: track 0.00 -> 5.11 mm
- net /DATA: track 0.00 -> 4.57 mm
- net +3V3_Lin: track 3.53 -> 0.00 mm
- net /DATA_: track 0.00 -> 3.46 mm
- net /PDM_DATA_: track 0.00 -> 1.73 mm
- net /CLOCK_: track 0.00 -> 1.60 mm
- net Net-(U2-DATA): track 1.55 -> 0.00 mm
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- added copper zone on F.Cu, net +3V3
Other:
- board size 31 x 13.5 mm -> 38 x 17.5 mm

Commit message: Thermal camera V2 WIP
Parts:
- MK1: footprint Sensor_Audio:Knowles_LGA-5_3.5x2.65mm -> cacophony-library:Knowles_LGA-5_3.5x2.65mm_0.6mm_NPTH
Other:
- board text added: "CAC_MIC 0.6mm NPTH"
Changed lines of the file:
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@@
     (fp_line (start 1.6 0.8) (end -1.6 0.8)
       (stroke (width 0.1) (type solid)) (layer "F.Fab"))
-    (pad "1" smd roundrect (at -1.475 0 90) (size 1.15 1.8) (layers "F.Cu" "F.Paste" "F.Mask") (roundrect_rratio 0.217391)
+    (pad "1" smd roundrect (at -1.475 0 90) (size 1.15 1.8) (layers "F.Cu" "F.Paste" "F.Mask") (roundrect_rratio 0.2173913043)
       (net 2 "+1V8") (pintype "passive"))
-    (pad "2" smd roundrect (at 1.475 0 90) (size 1.15 1.8) (layers "F.Cu" "F.Paste" "F.Mask") (roundrect_rratio 0.217391)
+    (pad "2" smd roundrect (at 1.475 0 90) (size 1.15 1.8) (layers "F.Cu" "F.Paste" "F.Mask") (roundrect_rratio 0.2173913043)
       (net 1 "GND") (pintype "passive"))
     (model "${KICAD6_3DMODEL_DIR}/Capacitor_SMD.3dshapes/C_1206_3216Metric.wrl"
@@
     )
   )
-  (footprint "Sensor_Audio:Knowles_LGA-5_3.5x2.65mm" (layer "F.Cu")
+  (footprint "cacophony-library:Knowles_LGA-5_3.5x2.65mm_0.6mm_NPTH" (layer "F.Cu")
     (at 112.768 109.9925 -90)
     (descr "https://www.knowles.com/docs/default-source/model-downloads/sph0641lu4h-1-revb.pdf")
@@
     (property "ki_keywords" "Microphone MEMS")
     (attr smd)
-    (fp_text reference "MK1" (at 2.2755 -0.008 -180) (layer "F.SilkS")
+    (fp_text reference "MK1" (at 2.2755 -0.008) (layer "F.SilkS")
         (effects (font (size 0.5 0.5) (thickness 0.1)))
     )
@@
     (fp_arc (start 0.6 1.05) (mid 0.464769 1.241582) (end 0.271239 1.374011)
       (stroke (width 0.3) (type solid)) (layer "F.Paste"))
+    (fp_circle (center 0 0.77) (end 3 0.77)
+      (stroke (width 0.12) (type default)) (fill none) (layer "B.SilkS"))
     (fp_line (start -1.44 1.36) (end -1.44 1.86)
       (stroke (width 0.12) (type solid)) (layer "F.SilkS"))
@@
     (fp_line (start 1.325 1.75) (end -1.325 1.75)
       (stroke (width 0.1) (type solid)) (layer "F.Fab"))
-    (pad "" np_thru_hole circle (at 0 0.77 270) (size 0.5 0.5) (drill 0.5) (layers "*.Cu" "*.Mask"))
+    (pad "" np_thru_hole circle (at 0 0.77 270) (size 0.6 0.6) (drill 0.6) (layers "F&B.Cu" "*.Mask"))
     (pad "1" smd rect (at -0.8375 -1.304 270) (size 0.725 0.522) (layers "F.Cu" "F.Paste" "F.Mask")
       (net 8 "/DATA_") (pinfunction "DATA") (pintype "output"))
@@
   (gr_circle (center 104 110) (end 106.6 110)
     (stroke (width 0.2) (type solid)) (fill none) (layer "User.5"))
+  (gr_text "CAC_MIC \n0.6mm NPTH" (at 130.49 111.17) (layer "B.SilkS")
+    (effects (font (size 1.5 1.5) (thickness 0.3) bold) (justify left bottom mirror))
+  )
   (segment (start 109.12 106.91) (end 109.2 106.99) (width 0.37) (layer "F.Cu") (net 1))
   (segment (start 108.175 106.6) (end 108.485 106.91) (width 0.37) (layer "F.Cu") (net 1))
   (segment (start 124.235 104.135) (end 124.235 105) (width 0.37) (layer "F.Cu") (net 1))
-  (segment (start 112 109.3425) (end 112 108.8) (width 0.3) (layer "F.Cu") (net 1))
-  (segment (start 110.7225 109.9925) (end 110.72 109.99) (width 0.3) (layer "F.Cu") (net 1))
   (segment (start 122.8 108.385) (end 121.925 108.385) (width 0.3) (layer "F.Cu") (net 1))
   (segment (start 121.925 108.385) (end 121.77 108.23) (width 0.3) (layer "F.Cu") (net 1))
   (segment (start 122.65 104) (end 124.1 104) (width 0.37) (layer "F.Cu") (net 1))
   (segment (start 111.7 106.6) (end 112 106.6) (width 0.5) (layer "F.Cu") (net 1))
-  (segment (start 112 110.6425) (end 112 111.3) (width 0.3) (layer "F.Cu") (net 1))
   (segment (start 124.2 104.1) (end 124.235 104.135) (width 0.37) (layer "F.Cu") (net 1))
-  (segment (start 111.3355 109.9925) (end 110.7225 109.9925) (width 0.3) (layer "F.Cu") (net 1))
   (segment (start 108.485 106.91) (end 109.12 106.91) (width 0.37) (layer "F.Cu") (net 1))
   (segment (start 124.1 104) (end 124.2 104.1) (width 0.37) (layer "F.Cu") (net 1))
+  (segment (start 111.99 108.837) (end 111.99 109.3) (width 0.25) (layer "F.Cu") (net 1))
   (segment (start 124.235 105) (end 124.235 103.165) (width 0.37) (layer "F.Cu") (net 1))
   (segment (start 121.77 108.23) (end 121.29 108.23) (width 0.3) (layer "F.Cu") (net 1))
   (segment (start 112 106.6) (end 112.25 106.35) (width 0.5) (layer "F.Cu") (net 1))
+  (segment (start 112.02 110.707) (end 112.02 111.17) (width 0.25) (layer "F.Cu") (net 1))
+  (segment (start 111.3355 109.9925) (end 110.8725 109.9925) (width 0.25) (layer "F.Cu") (net 1))
   (via (at 122.7 101.7) (size 0.5) (drill 0.3) (layers "F.Cu" "B.Cu") (free) (net 1))
   (via (at 120.2 105.25) (size 0.5) (drill 0.3) (layers "F.Cu" "B.Cu") (free) (net 1))

Commit message: P2 milestone
Parts:
- moved C1 141.4 mm to (21.3, 8.54)
- moved C2 141.4 mm to (15.9, 9.35)
- moved C3 141.4 mm to (27.7, 8.71)
- moved C4 141.4 mm to (11.7, 7.08)
- moved C5 141.4 mm to (8.18, 7.08)
- moved J1 141.4 mm to (27.0, 4.00)
- moved J2 141.4 mm to (4.00, 10.0)
- moved J4 141.4 mm to (20.7, 4.00)
- moved MK1 141.4 mm to (12.8, 9.99)
- moved R1 141.4 mm to (20.8, 7.09)
- moved R2 141.4 mm to (25.1, 10.8)
- moved R3 141.4 mm to (18.1, 9.16)
- moved U2 141.4 mm to (24.5, 8.71)
- moved U3 141.4 mm to (9.94, 6.99)

Commit message: P3-Nov release
Parts:
- moved J2 10.8 mm to (0.00, 0.00)
- moved MK1 10.4 mm to (8.00, 0.77), turned to 180 degrees
- moved C4 9.05 mm to (3.99, 2.34), turned to 180 degrees
- moved C2 8.99 mm to (8.70, 4.00), turned to 0 degrees
- moved C3 8.69 mm to (19.8, 5.10)
- moved C1 8.69 mm to (13.4, 4.93)
- moved U2 8.69 mm to (16.6, 5.10)
- moved R2 8.48 mm to (17.4, 7.29)
- moved R1 7.09 mm to (15.1, 2.95), turned to 0 degrees
- moved U3 6.70 mm to (3.90, 4.10), turned to 0 degrees
- moved J4 6.17 mm to (16.0, 0.00)
- moved R3 5.86 mm to (12.9, 6.39)
- moved J1 5.66 mm to (23.0, 0.00)
- moved C5 4.36 mm to (3.99, 5.87), turned to 180 degrees
Connections:
- net /CLOCK_ renamed /CLOCK_PHY
- net /DATA_ renamed /DATA_PHY
- net /PDM_DATA_ renamed /PDM_DATA_PHY
Routing:
- net +3V3: track 24.4 -> 41.0 mm
- net GND: track 9.14 -> 5.58 mm, vias 11 -> 16
- net /DATA_PHY: track 3.46 -> 6.61 mm
- net /DATA: track 4.57 -> 1.63 mm
- net /CLOCK: track 12.4 -> 14.5 mm
- net PDM_CLOCK: track 5.11 -> 3.00 mm
- net +1V8: track 24.7 -> 26.5 mm
- removed copper zone on F.Cu, net +3V3
Other:
- board size 38 x 17.5 mm -> 39 x 12 mm

Commit message: v0.4.0
Parts:
- moved R1 0.70 mm to (15.8, 2.95)
Connections:
- J1 pad 1: GND -> unconnected-(J1-Pin_1-Pad1)
- J2 pad 1: GND -> unconnected-(J2-Pin_1-Pad1)
- MK1 pad 3: GND -> unconnected-(MK1-GND-Pad3)
Routing:
- net GND: track 5.58 -> 4.80 mm
Other:
- board text added: "v0.4.0"

Commit message: Small update for v0.4.1
Connections:
- MK1 pad 3: unconnected-(MK1-GND-Pad3) -> GND
Routing:
- net GND: track 4.80 -> 5.84 mm, vias 16 -> 18
Other:
- board text added: "${TAG}"
- board text added: "CAC_MIC"
- board text removed: "CAC_MIC 0.6mm NPTH"
- board text removed: "v0.4.0"
Changed lines of the file:
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@@
 	(generator_version "8.0")
 	(general
-		(thickness 1.6)
+		(thickness 1)
 		(legacy_teardrops no)
 	)
@@
 			(layer "dielectric 1"
 				(type "core")
-				(thickness 1.51)
+				(thickness 0.91)
 				(material "FR4")
 				(epsilon_r 4.5)
@@
 	(net 11 "/DATA")
 	(net 12 "/CLOCK_PHY")
-	(net 13 "unconnected-(MK1-GND-Pad3)")
-	(net 14 "unconnected-(J1-Pin_1-Pad1)")
-	(net 15 "unconnected-(J2-Pin_1-Pad1)")
+	(net 13 "unconnected-(J1-Pin_1-Pad1)")
+	(net 14 "unconnected-(J2-Pin_1-Pad1)")
 	(footprint "Connector_PinHeader_1.27mm:PinHeader_2x03_P1.27mm_Vertical_SMD"
 		(layer "F.Cu")
@@
 			)
 		)
+		(property ki_fp_filters "TerminalBlock*:*")
+		(sheetname "Root")
+		(sheetfile "tc2-mic-pcb.kicad_sch")
 		(attr smd)
 		(fp_arc
@@
 			(layers "*.Cu" "*.Mask")
 			(remove_unused_layers no)
-			(net 14 "unconnected-(J1-Pin_1-Pad1)")
+			(net 13 "unconnected-(J1-Pin_1-Pad1)")
 			(pinfunction "Pin_1")
 			(pintype "passive+no_connect")
@@
 			)
 		)
-		(property "Description" ""
+		(property "Description" "2-Bit Bidirectional Voltage-Level Shifter for Open-Drain and Push-Pull Application, SSOP-8"
 			(at 0 0 0)
 			(unlocked yes)
@@
 			)
 		)
+		(property ki_fp_filters "TerminalBlock*:*")
+		(sheetname "Root")
+		(sheetfile "tc2-mic-pcb.kicad_sch")
 		(attr smd)
 		(fp_arc
@@
 			(layers "*.Cu" "*.Mask")
 			(remove_unused_layers no)
-			(net 15 "unconnected-(J2-Pin_1-Pad1)")
+			(net 14 "unconnected-(J2-Pin_1-Pad1)")
 			(pinfunction "Pin_1")
 			(pintype "passive+no_connect")
@@
 		(tags "capacitor")
 		(property "Reference" "C5"
-			(at 1.3 -0.205 90)
+			(at -1.37 0.005 90)
 			(layer "F.SilkS")
 			(effects
@@
 			(size 0.3 0.3)
 			(layers "F.Cu" "F.Mask")
-			(net 13 "unconnected-(MK1-GND-Pad3)")
+			(net 1 "GND")
 			(pinfunction "GND")
-			(pintype "power_in+no_connect")
+			(pintype "power_in")
 			(zone_connect 0)
 			(options
@@
 		(layer "User.4")
 	)
-	(gr_text "v0.4.0"
+	(gr_text "${TAG}"
 		(at -4.82 5.21 180)
 		(layer "B.SilkS")
@@
 		)
 	)
-	(gr_text "CAC_MIC \n0.6mm NPTH"
+	(gr_text "CAC_MIC"
 		(at 31.5 7.33 0)
 		(layer "B.SilkS")
@@
 		)
 	)
-	(gr_text "v0.4.0"
+	(gr_text "${TAG}"
 		(at -4.92 5.22 180)
 		(layer "F.SilkS")
@@
 	)
 	(segment
+		(start 9.37 -0.01)
+		(end 8.86 -0.01)
+		(width 0.37)
+		(layer "F.Cu")
+		(net 1)
+	)
+	(segment
 		(start 14.9 4.775)
 		(end 14.025 4.775)
@@
 	)
 	(segment
+		(start 6.62 0)
+		(end 7.15 0)
+		(width 0.37)
+		(layer "F.Cu")
+		(net 1)
+	)
+	(segment
 		(start 3.82 5.555)
 		(end 3.82 4.92)
@@
 	)
 	(via
+		(at 6.62 0)
+		(size 0.46)
+		(drill 0.3)
+		(layers "F.Cu" "B.Cu")
+		(free yes)
+		(net 1)
+	)
+	(via
 		(at 14.05 -2.38)
 		(size 0.46)
@@
 		(size 0.46)
 		(drill 0.3)
+		(layers "F.Cu" "B.Cu")
+		(free yes)
+		(net 1)
+	)
+	(via
+		(at 9.37 -0.01)
+		(size 0.46)
+		(drill 0.3)
