File: tc2-mic-pcb/tc2-mic-pcb.kicad_pcb (KiCad board)
At the start: 2 copper layers, 39 x 12 mm, 19 parts, among them J401 Conn_02x03_Odd_Even, J402 Screw_Terminal_01x01, J403 Screw_Terminal_01x01, U401 AP7335-18SNG-7, U402 TXS0102DCT

Commit message: Made microphone PCB wider to make it easier for v cutting
Parts:
- moved REF** 2.70 mm to (13.0, 11.5)
Routing:
- net GND: vias 18 -> 19
Other:
- board size 39 x 12 mm -> 39 x 15 mm
Changed lines of the file:
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@@
 	(footprint "PCM_kikit:Tab"
 		(layer "F.Cu")
-		(at 13 8.8 90)
+		(at 13 11.5 90)
 		(descr "A symbol representing annotation for tab placement")
 		(property "Reference" "REF**"
@@
 	)
 	(gr_arc
-		(start 30 -4)
-		(mid 32.82842 -2.828419)
-		(end 34 0)
-		(locked yes)
+		(start -5 -1.749999)
+		(mid -3.25 0)
+		(end -5 1.749999)
 		(stroke
-			(width 0.25)
-			(type solid)
-		)
-		(layer "Edge.Cuts")
-	)
-	(gr_line
-		(start 34 7)
-		(end 34 0)
-		(locked yes)
-		(stroke
-			(width 0.25)
-			(type solid)
-		)
-		(layer "Edge.Cuts")
-	)
-	(gr_line
-		(start 30 -4)
-		(end -4 -4)
-		(locked yes)
-		(stroke
-			(width 0.25)
-			(type solid)
-		)
-		(layer "Edge.Cuts")
-	)
-	(gr_arc
-		(start -4 8)
-		(mid -4.707114 7.707115)
-		(end -5 7)
-		(locked yes)
-		(stroke
-			(width 0.25)
-			(type solid)
-		)
-		(layer "Edge.Cuts")
-	)
-	(gr_line
-		(start -5 -3)
-		(end -5 -1.75)
-		(locked yes)
-		(stroke
-			(width 0.25)
-			(type solid)
-		)
-		(layer "Edge.Cuts")
-	)
-	(gr_line
-		(start -4 8)
-		(end 33 8)
-		(locked yes)
-		(stroke
-			(width 0.25)
-			(type solid)
-		)
-		(layer "Edge.Cuts")
-	)
-	(gr_arc
-		(start -5 -3)
-		(mid -4.707095 -3.707078)
-		(end -4 -4)
-		(locked yes)
-		(stroke
-			(width 0.25)
-			(type solid)
-		)
-		(layer "Edge.Cuts")
-	)
-	(gr_circle
-		(center 30 0.00003)
-		(end 31.75 0.00003)
-		(stroke
-			(width 0.1)
+			(width 0.2)
 			(type default)
-		)
-		(fill none)
-		(layer "Edge.Cuts")
-	)
-	(gr_arc
-		(start 34 7)
-		(mid 33.707119 7.707136)
-		(end 33 8)
-		(locked yes)
-		(stroke
-			(width 0.25)
-			(type solid)
-		)
-		(layer "Edge.Cuts")
-	)
-	(gr_arc
-		(start -5 -1.75)
-		(mid -3.249997 0.00003)
-		(end -5 1.75)
-		(locked yes)
-		(stroke
-			(width 0.25)
-			(type solid)
-		)
-		(layer "Edge.Cuts")
-	)
-	(gr_line
-		(start -5 1.75)
-		(end -5 7)
-		(locked yes)
-		(stroke
-			(width 0.25)
-			(type solid)
 		)
 		(layer "Edge.Cuts")
@@
 		(center 30 0)
 		(end 31.75 0)
-		(locked yes)
 		(stroke
-			(width 0.25)
-			(type solid)
+			(width 0.2)
+			(type default)
 		)
 		(fill none)
-		(layer "User.4")
+		(layer "Edge.Cuts")
+	)
+	(gr_arc
+		(start -4.000001 11)
+		(mid -4.707107 10.707107)
+		(end -5 10.000002)
+		(stroke
+			(width 0.2)
+			(type default)
+		)
+		(layer "Edge.Cuts")
+	)
+	(gr_arc
+		(start -5 -3.000001)
+		(mid -4.707107 -3.707107)
+		(end -4.000002 -4)
+		(stroke
+			(width 0.2)
+			(type default)
+		)
+		(layer "Edge.Cuts")
+	)
+	(gr_line
+		(start -4.000002 -4)
+		(end 30 -4)
+		(stroke
+			(width 0.2)
+			(type default)
+		)
+		(layer "Edge.Cuts")
+	)
+	(gr_line
+		(start -5 -1.749999)
+		(end -5 -3.000001)
+		(stroke
+			(width 0.2)
+			(type default)
+		)
+		(layer "Edge.Cuts")
+	)
+	(gr_line
+		(start 34 0)
+		(end 34 10)
+		(stroke
+			(width 0.2)
+			(type default)
+		)
+		(layer "Edge.Cuts")
+	)
+	(gr_arc
+		(start 34 10)
+		(mid 33.707107 10.707107)
+		(end 33 11)
+		(stroke
+			(width 0.2)
+			(type default)
+		)
+		(layer "Edge.Cuts")
+	)
+	(gr_line
+		(start -5 10.000002)
+		(end -5 1.749999)
+		(stroke
+			(width 0.2)
+			(type default)
+		)
+		(layer "Edge.Cuts")
+	)
+	(gr_line
+		(start 33 11)
+		(end -4.000001 11)
+		(stroke
+			(width 0.2)
+			(type default)
+		)
+		(layer "Edge.Cuts")
+	)
+	(gr_arc
+		(start 30 -4)
+		(mid 32.828427 -2.828427)
+		(end 34 0)
+		(stroke
+			(width 0.2)
+			(type default)
+		)
+		(layer "Edge.Cuts")
+	)
+	(gr_circle
+		(center 23 0)
+		(end 25 0)
+		(stroke
+			(width 0.2)
+			(type default)
+		)
+		(fill none)
+		(layer "User.1")
+	)
+	(gr_circle
+		(center 0 0)
+		(end 2 0)
+		(stroke
+			(width 0.2)
+			(type default)
+		)
+		(fill none)
+		(layer "User.1")
 	)
 	(gr_circle
 		(center 8 0)
 		(end 9 0)
-		(locked yes)
 		(stroke
-			(width 0.25)
-			(type solid)
+			(width 0.2)
+			(type default)
 		)
 		(fill none)
-		(layer "User.4")
-	)
-	(gr_circle
-		(center 23 0)
-		(end 24 0)
-		(locked yes)
-		(stroke
-			(width 0.25)
-			(type solid)
-		)
-		(fill none)
-		(layer "User.4")
-	)
-	(gr_circle
-		(center 23 0)
-		(end 25.175 0)
-		(locked yes)
-		(stroke
-			(width 0.25)
-			(type solid)
-		)
-		(fill none)
-		(layer "User.4")
-	)
-	(gr_circle
-		(center 0 0)
-		(end 1 0)
-		(locked yes)
-		(stroke
-			(width 0.25)
-			(type solid)
-		)
-		(fill none)
-		(layer "User.4")
-	)
-	(gr_circle
-		(center 0 0)
-		(end 2.175 0)
-		(locked yes)
-		(stroke
-			(width 0.25)
-			(type solid)
-		)
-		(fill none)
-		(layer "User.4")
+		(layer "User.1")
 	)
 	(gr_text "${TAG}"
-		(at -4.82 5.21 180)
+		(at -4.5 8 180)
 		(layer "B.SilkS")
 		(effects
@@
 	)
 	(gr_text "${TAG}"
-		(at -4.92 5.22 180)
+		(at -4.5 8 180)
 		(layer "F.SilkS")
 		(effects
@@
 	)
 	(via
+		(at 14.73 7.75)
+		(size 0.46)
+		(drill 0.3)
+		(layers "F.Cu" "B.Cu")
+		(free yes)
+		(net 1)
+	)
+	(via
 		(at 11.03 3.98)
 		(size 0.46)
@@
 	)
 	(segment
+		(start 8.01 2.73)
+		(end 8.81 3.53)
+		(width 0.15)
+		(layer "F.Cu")
+		(net 9)
+	)
+	(segment
+		(start 8.81 4.75)
+		(end 11.23 7.17)
+		(width 0.15)
+		(layer "F.Cu")
+		(net 9)
+	)
+	(segment
+		(start 7.1625 1.252)
+		(end 7.675 1.252)
+		(width 0.15)
+		(layer "F.Cu")
+		(net 9)
+	)
+	(segment
+		(start 8.01 1.587)
+		(end 8.01 2.73)
+		(width 0.15)
+		(layer "F.Cu")
+		(net 9)
+	)
+	(segment
 		(start 7.675 1.252)
 		(end 8.01 1.587)
@@
 	)
 	(segment
-		(start 15.71 7.04)
+		(start 11.23 7.17)
 		(end 15.84 7.17)
 		(width 0.15)
@@
 	)
 	(segment
-		(start 8.81 4.75)
-		(end 11.1 7.04)
-		(width 0.15)
-		(layer "F.Cu")
-		(net 9)
-	)
-	(segment
 		(start 8.81 3.53)
 		(end 8.81 4.75)
-		(width 0.15)
-		(layer "F.Cu")
-		(net 9)
-	)
-	(segment
-		(start 7.1625 1.252)
-		(end 7.675 1.252)
-		(width 0.15)
-		(layer "F.Cu")
-		(net 9)
-	)
-	(segment
-		(start 8.01 2.73)
-		(end 8.81 3.53)
-		(width 0.15)
-		(layer "F.Cu")
-		(net 9)
-	)
-	(segment
-		(start 8.01 1.587)
-		(end 8.01 2.73)
-		(width 0.15)
-		(layer "F.Cu")
-		(net 9)
-	)
-	(segment
-		(start 11.1 7.04)
-		(end 15.71 7.04)
 		(width 0.15)
 		(layer "F.Cu")
@@
 		(polygon
 			(pts
-				(xy -5.39 -4.33) (xy 34.43 -4.47) (xy 34.7 8.21) (xy -5.44 8.37)
+				(xy -5.5 -4.5) (xy 34.5 -4.5) (xy 34.5 11.5) (xy -5.5 11.5)
 			)
 		)
@@
 	)
 	(group ""
-		(locked yes)
-		(members "0e031fc5-c6af-4be6-a4d9-e816d3035258" "5cd2f671-1ec1-4553-a1d9-959aa7a9d259"
-			"87a69678-834e-46f9-92bd-804d6e8f1f69" "9d8d5dc6-f516-496c-b47b-e648fb530d5d"
-			"b47bf67e-fbf7-4c9a-aa83-f0e787fe6cb7" "c194a018-560c-465a-9576-7aae5542f6f9"
-			"cf7ad916-3862-4519-88ea-aad4ea3c3dd7" "e183582c-d8d9-46b9-b809-dfbdbc6504f6"
-			"ed646fc7-10ff-45a4-8a56-cf33d846ef30" "fa3e18a6-0a3c-4499-85e0-a6deb754b51e"
+		(members "00037d3f-88fd-495d-afd5-eb4360223d0d" "0d259c6c-2f1f-4876-b4b9-dc2878d2b81a"
+			"346be6e1-5918-4a5f-b271-6f1b2c376e26" "398f83b2-f02c-495e-8c7a-71f4608eeb7b"
+			"521f814c-8eac-470c-abc2-70a33fc2163c" "6600df4a-5a95-47ba-bade-5766b72f6b1a"
+			"94d7844f-cc40-4efb-9973-e6823300247c" "9daaf7c4-7b91-4c09-8396-d6bce7eb20b3"
+			"d9b70580-e5da-497c-a605-31fdefdb70e5" "e5972eb3-e403-4ef3-901f-5d4f7bd0c5d8"
+			"f52656b2-d0bb-4fb6-8581-aeed88e92569"
 		)
 	)
 	(group ""
-		(locked yes)
-		(members "ae13e7fc-1f26-476f-9a89-7cff5d9a85e6" "e86a1c89-418d-496d-9a79-66ad8c2d8dca")
-	)
-	(group ""
-		(locked yes)
-		(members "6e51f29f-27a3-424b-84a0-2229168eb323" "984b77ee-e8fd-42ce-9eb4-136a9c9187ba"
-			"9f3cd57e-0fcd-4b01-a362-b8c76fccb253" "a3b2c582-9ecf-41ad-99e8-ecc292060498"
-			"af1b9507-3bb9-4236-8bbd-1a7a00746fdb" "c89e34c4-a9ce-4fab-869b-ddcd55808a2d"
-		)
-	)
+		(members "1cf98f13-d971-4d86-bee7-6fce7f4bec1a" "1fb59381-fa24-44d3-9aa2-e2c990368de1"
+			"f8ef4663-fd1e-45c8-ab4a-0cab190d1f3a"
+		)
+	)

Commit message: 0.8.0 WIP
Parts:
- R401, R402, R403: value 22R -> 22Ω
Changed lines of the file:
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@@
 			)
 		)
-		(property "Value" "22R"
+		(property "Value" "22Ω"
 			(at 0 1.17 0)
 			(layer "F.Fab")
@@
 			)
 		)
-		(property "Value" "22R"
+		(property "Value" "22Ω"
 			(at 0 1.17 0)
 			(layer "F.Fab")
@@
 			)
 		)
-		(property "Value" "22R"
+		(property "Value" "22Ω"
 			(at 0 1.17 0)
 			(layer "F.Fab")
