File: tc2-mic-pcb/tc2-mic-pcb.kicad_sch (KiCad schematic)
At the start: 9 parts, among them J4 Conn_02x03_Odd_Even, J7 Screw_Terminal_01x01, U14 SPH0645LM4H, U15 ME6211

Commit message: Version 2 WIP
Parts:
- removed C1: 1uF, Capacitor_SMD:C_0402_1005Metric, symbol Device:C_Small
- removed C1: 220nF, Capacitor_SMD:C_0402_1005Metric, symbol Device:C_Small
- removed R30: 22ohm, Resistor_SMD:R_0402_1005Metric, symbol Device:R
- removed U14: SPH0645LM4H, cacophony-library:MIC_SPH0645LM4H-B, symbol cacophony-library:SPH0645LM4H
- removed U15: ME6211, Package_TO_SOT_SMD:SOT-23-5, symbol cacophony-library:ME6211
- added C1: 100nF, Capacitor_SMD:C_0402_1005Metric, symbol Device:C_Small
- added C2: 100nF, Capacitor_SMD:C_1206_3216Metric, symbol Device:C_Small
- added C4, C5: 1uF, Capacitor_SMD:C_0402_1005Metric, symbol Device:C_Small
- added MK1: SPH0641LU4H-1, Sensor_Audio:Knowles_LGA-5_3.5x2.65mm, symbol Sensor_Audio:SPH0641LU4H-1
- added R1, R2, R3: 22R, Resistor_SMD:R_0402_1005Metric, symbol Device:R
- added U2: TXS0102DCT, Package_SO:SSOP-8_2.95x2.8mm_P0.65mm, symbol Logic_LevelTranslator:TXS0102DCT
- added U3: AP7335-18SNG-7, cacophony-library:U-DFN2020-6_L2.0-W2.0-P0.65-BL-EP, symbol cacophony-library:AP7335-18SNG-7
- C3: value 12pF -> 100nF; LCSC C1547 -> C1525
Connections:
- net +3V3_Lin is gone; now on net GND: C3.2
- net +5V is gone; now on net GND: J4.2 (Pin_2)
- net GND: now also J7.1 (Pin_1), J7.1 (Pin_1), C1.2, C2.2, C4.2, C5.2, MK1.2 (SEL), MK1.3 (GND), U2.2 (GND), U3.2 (GND), U3.7 (GND); no longer C3.1
- net I2S_BCLK renamed PDM_DATA
- net PDM_DATA: now also R1.2
- net I2S_DIN renamed +3V3
- net +3V3: now also C3.1, C5.1, U2.6 (OE), U2.7 (VCCB), U3.1 (EN), U3.3 (IN)
- net I2S_LRCLK renamed PDM_CLOCK
- net PDM_CLOCK: now also U2.8 (B1)
- new net +1V8: C1.1, C2.1, C4.1, MK1.5 (VDD), U2.3 (VCCA), U3.4 (OUT)
- new net CLOCK: MK1.4 (CLOCK), R2.1
- new net CLOCK_: R2.2, U2.5 (A1)
- new net DATA: R3.2, U2.4 (A2)
- new net DATA_: MK1.1 (DATA), R3.1
- new net PDM_DATA_: R1.1, U2.1 (B2)
- no-connect marks 3 -> 2
Other:
- note added: "Use Class 1 Capacitor as specified in the Mic Datasheet"
- moved on the sheet: J4, J7

Commit message: Thermal camera V2 WIP
Parts:
- MK1: footprint Sensor_Audio:Knowles_LGA-5_3.5x2.65mm -> cacophony-library:Knowles_LGA-5_3.5x2.65mm_0.6mm_NPTH
Changed lines of the file:
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@@
       (effects (font (size 1.27 1.27)) (justify right))
     )
-    (property "Footprint" "Sensor_Audio:Knowles_LGA-5_3.5x2.65mm" (at 93.98 50.8 0)
+    (property "Footprint" "cacophony-library:Knowles_LGA-5_3.5x2.65mm_0.6mm_NPTH" (at 93.98 50.8 0)
       (effects (font (size 1.27 1.27)) hide)
     )

Commit message: P3-Nov release
Connections:
- net CLOCK_ renamed CLOCK_PHY
- net DATA_ renamed DATA_PHY
- net PDM_DATA_ renamed PDM_DATA_PHY
Changed lines of the file:
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@@
     (effects (font (size 1.27 1.27)) (justify left bottom))
   )
-  (label "PDM_DATA_" (at 171.45 54.61 0) (fields_autoplaced)
+  (label "PDM_DATA_PHY" (at 171.45 54.61 0) (fields_autoplaced)
     (effects (font (size 1.27 1.27)) (justify left bottom))
   )
@@
     (effects (font (size 1.27 1.27)) (justify left bottom))
   )
-  (label "DATA_" (at 106.68 53.34 0) (fields_autoplaced)
+  (label "DATA_PHY" (at 106.68 53.34 0) (fields_autoplaced)
     (effects (font (size 1.27 1.27)) (justify left bottom))
   )
-  (label "CLOCK_" (at 139.7 49.53 0) (fields_autoplaced)
-    (effects (font (size 1.27 1.27)) (justify left bottom))
+  (label "CLOCK_PHY" (at 149.86 49.53 180) (fields_autoplaced)
+    (effects (font (size 1.27 1.27)) (justify right bottom))
   )
   (global_label "PDM_DATA" (shape input) (at 191.77 54.61 0) (fields_autoplaced)

Commit message: v0.4.0
Connections:
- net GND: no longer J7.1 (Pin_1), J7.1 (Pin_1), MK1.3 (GND)
- no-connect marks 2 -> 5

Commit message: Small update for v0.4.1
Connections:
- net GND: now also MK1.3 (GND)
- no-connect marks 5 -> 4
Other:
- moved on the sheet: C1
Changed lines of the file:
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@@
 	)
 	(junction
-		(at 149.86 31.75)
+		(at 154.94 27.94)
 		(diameter 0)
 		(color 0 0 0 0)
@@
 	)
 	(no_connect
-		(at 93.98 58.42)
-	)
-	(no_connect
 		(at 50.8 49.53)
 	)
@@
 	(wire
 		(pts
-			(xy 149.86 38.1) (xy 149.86 39.37)
+			(xy 154.94 34.29) (xy 154.94 35.56)
 		)
 		(stroke
@@
 	(wire
 		(pts
-			(xy 157.48 31.75) (xy 149.86 31.75)
+			(xy 157.48 27.94) (xy 154.94 27.94)
 		)
 		(stroke
@@
 	(wire
 		(pts
-			(xy 147.32 59.69) (xy 149.86 59.69)
-		)
-		(stroke
-			(width 0)
-			(type default)
-		)
-	)
-	(wire
-		(pts
 			(xy 160.02 64.77) (xy 160.02 66.04)
 		)
@@
 	(wire
 		(pts
-			(xy 140.97 63.5) (xy 147.32 63.5)
+			(xy 149.86 54.61) (xy 128.27 54.61)
 		)
 		(stroke
@@
 	(wire
 		(pts
-			(xy 149.86 54.61) (xy 128.27 54.61)
+			(xy 162.56 31.75) (xy 170.18 31.75)
 		)
 		(stroke
@@
 	(wire
 		(pts
-			(xy 162.56 31.75) (xy 170.18 31.75)
+			(xy 93.98 58.42) (xy 93.98 59.69)
 		)
 		(stroke
@@
 	(wire
 		(pts
-			(xy 157.48 39.37) (xy 157.48 31.75)
+			(xy 157.48 39.37) (xy 157.48 27.94)
 		)
 		(stroke
@@
 	(wire
 		(pts
-			(xy 149.86 31.75) (xy 149.86 33.02)
-		)
-		(stroke
-			(width 0)
-			(type default)
-		)
-	)
-	(wire
-		(pts
-			(xy 147.32 63.5) (xy 147.32 59.69)
+			(xy 154.94 27.94) (xy 154.94 29.21)
 		)
 		(stroke
@@
 	(wire
 		(pts
-			(xy 149.86 30.48) (xy 149.86 31.75)
+			(xy 147.32 44.45) (xy 147.32 43.18)
+		)
+		(stroke
+			(width 0)
+			(type default)
+		)
+	)
+	(wire
+		(pts
+			(xy 154.94 26.67) (xy 154.94 27.94)
 		)
 		(stroke
@@
 	(wire
 		(pts
+			(xy 149.86 44.45) (xy 147.32 44.45)
+		)
+		(stroke
+			(width 0)
+			(type default)
+		)
+	)
+	(wire
+		(pts
 			(xy 69.85 86.36) (xy 69.85 88.9)
 		)
@@
 	)
 	(symbol
+		(lib_id "power:GND")
+		(at 93.98 59.69 0)
+		(unit 1)
+		(exclude_from_sim no)
+		(in_bom yes)
+		(on_board yes)
+		(dnp no)
+		(fields_autoplaced yes)
+		(property "Reference" "#PWR06"
+			(at 93.98 66.04 0)
+			(effects
+				(font
+					(size 1.27 1.27)
+				)
+				(hide yes)
+			)
+		)
+		(property "Value" "GND"
+			(at 93.98 64.77 0)
+			(effects
+				(font
+					(size 1.27 1.27)
+				)
+				(hide yes)
+			)
+		)
+		(property "Footprint" ""
+			(at 93.98 59.69 0)
+			(effects
+				(font
+					(size 1.27 1.27)
+				)
+				(hide yes)
+			)
+		)
+		(property "Datasheet" ""
+			(at 93.98 59.69 0)
+			(effects
+				(font
+					(size 1.27 1.27)
+				)
+				(hide yes)
+			)
+		)
+		(property "Description" "Power symbol creates a global label with name \"GND\" , ground"
+			(at 93.98 59.69 0)
+			(effects
+				(font
+					(size 1.27 1.27)
+				)
+				(hide yes)
+			)
+		)
+		(pin "1"
+		)
+		(instances
+			(project "tc2-mic-pcb"
+				(path "/5f96247b-0b73-48aa-a1a8-3d96ade9d103"
+					(reference "#PWR06")
+					(unit 1)
+				)
+			)
+		)
+	)
+	(symbol
 		(lib_id "power:+3V3")
 		(at 73.66 90.17 0)
@@
 	(symbol
 		(lib_id "Device:C_Small")
-		(at 149.86 35.56 0)
+		(at 154.94 31.75 0)
 		(unit 1)
 		(exclude_from_sim no)
@@
 		(dnp no)
 		(property "Reference" "C1"
-			(at 143.51 34.29 0)
+			(at 148.59 30.48 0)
 			(effects
 				(font
@@
 		)
 		(property "Value" "100nF"
-			(at 142.24 36.83 0)
+			(at 147.32 33.02 0)
 			(effects
 				(font
@@
 		)
 		(property "Footprint" "Capacitor_SMD:C_0402_1005Metric"
-			(at 149.86 35.56 0)
+			(at 154.94 31.75 0)
 			(effects
 				(font
@@
 		)
 		(property "Datasheet" "~"
-			(at 149.86 35.56 0)
+			(at 154.94 31.75 0)
 			(effects
 				(font
@@
 		)
 		(property "Description" ""
-			(at 149.86 35.56 0)
+			(at 154.94 31.75 0)
 			(effects
 				(font
@@
 		)
 		(property "LCSC" "C1525"
-			(at 149.86 35.56 0)
+			(at 154.94 31.75 0)
 			(effects
 				(font
@@
 	(symbol
 		(lib_id "power:+1V8")
-		(at 149.86 30.48 0)
+		(at 154.94 26.67 0)
 		(unit 1)
 		(exclude_from_sim no)
@@
 		(fields_autoplaced yes)
 		(property "Reference" "#PWR05"
-			(at 149.86 34.29 0)
+			(at 154.94 30.48 0)
 			(effects
 				(font
@@
 		)
 		(property "Value" "+1V8"
-			(at 149.86 26.67 0)
+			(at 154.94 22.86 0)
 			(effects
 				(font
@@
 		)
 		(property "Footprint" ""
-			(at 149.86 30.48 0)
+			(at 154.94 26.67 0)
 			(effects
 				(font
@@
 		)
 		(property "Datasheet" ""
-			(at 149.86 30.48 0)
+			(at 154.94 26.67 0)
 			(effects
 				(font
@@
 		)
 		(property "Description" "Power symbol creates a global label with name \"+1V8\""
-			(at 149.86 30.48 0)
+			(at 154.94 26.67 0)
 			(effects
 				(font
@@
 			)
 		)
-		(property "Description" ""
+		(property "Description" "2-Bit Bidirectional Voltage-Level Shifter for Open-Drain and Push-Pull Application, SSOP-8"
 			(at 160.02 52.07 0)
 			(effects
@@
 					(size 1.27 1.27)
 				)
+				(hide yes)
 			)
 		)
@@
 	(symbol
 		(lib_id "power:+3V3")
-		(at 140.97 63.5 0)
+		(at 147.32 43.18 0)
 		(unit 1)
 		(exclude_from_sim no)
@@
 		(fields_autoplaced yes)
 		(property "Reference" "#PWR017"
-			(at 140.97 67.31 0)
+			(at 147.32 46.99 0)
 			(effects
 				(font
@@
 		)
 		(property "Value" "+3V3"
-			(at 140.97 59.69 0)
+			(at 147.32 39.37 0)
 			(effects
 				(font
@@
 		)
 		(property "Footprint" ""
-			(at 140.97 63.5 0)
+			(at 147.32 43.18 0)
 			(effects
 				(font
@@
 		)
 		(property "Datasheet" ""
-			(at 140.97 63.5 0)
+			(at 147.32 43.18 0)
 			(effects
 				(font
@@
 		)
 		(property "Description" "Power symbol creates a global label with name \"+3V3\""
-			(at 140.97 63.5 0)
+			(at 147.32 43.18 0)
 			(effects
 				(font
@@
 	(symbol
 		(lib_id "power:GND")
-		(at 149.86 39.37 0)
+		(at 154.94 35.56 0)
 		(unit 1)
 		(exclude_from_sim no)
@@
 		(fields_autoplaced yes)
 		(property "Reference" "#PWR02"
-			(at 149.86 45.72 0)
+			(at 154.94 41.91 0)
 			(effects
 				(font
@@
 		)
 		(property "Value" "GND"
-			(at 149.86 44.45 0)
+			(at 154.94 40.64 0)
 			(effects
 				(font
@@
 		)
 		(property "Footprint" ""
-			(at 149.86 39.37 0)
+			(at 154.94 35.56 0)
 			(effects
 				(font
@@
 		)
 		(property "Datasheet" ""
-			(at 149.86 39.37 0)
+			(at 154.94 35.56 0)
 			(effects
 				(font
@@
 		)
 		(property "Description" "Power symbol creates a global label with name \"GND\" , ground"
-			(at 149.86 39.37 0)
+			(at 154.94 35.56 0)
 			(effects
 				(font

Commit message: Update to use touch sensor
Parts:
- renumbered C1 to C401, C3 to C402, C2 to C403, C5 to C404, C4 to C405, J4 to J401, MK1 to MK401, R2 to R401, R3 to R402, R1 to R403, U3 to U401, U2 to U402
Changed lines of the file:
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@@
 		(dnp no)
 		(fields_autoplaced yes)
-		(property "Reference" "#PWR06"
+		(property "Reference" "#PWR0413"
 			(at 93.98 66.04 0)
 			(effects
@@
 			(project "tc2-mic-pcb"
 				(path "/5f96247b-0b73-48aa-a1a8-3d96ade9d103"
-					(reference "#PWR06")
+					(reference "#PWR0413")
 					(unit 1)
 				)
@@
 		(dnp no)
 		(fields_autoplaced yes)
-		(property "Reference" "#PWR01"
+		(property "Reference" "#PWR0415"
 			(at 73.66 93.98 0)
 			(effects
@@
 			(project "tc2-mic-pcb"
 				(path "/5f96247b-0b73-48aa-a1a8-3d96ade9d103"
-					(reference "#PWR01")
+					(reference "#PWR0415")
 					(unit 1)
 				)
@@
 		(dnp no)
 		(fields_autoplaced yes)
-		(property "Reference" "C2"
+		(property "Reference" "C403"
 			(at 78.74 45.0913 0)
 			(effects
@@
 			(project "tc2-mic-pcb"
 				(path "/5f96247b-0b73-48aa-a1a8-3d96ade9d103"
-					(reference "C2")
+					(reference "C403")
 					(unit 1)
 				)
@@
 		(on_board yes)
 		(dnp no)
-		(property "Reference" "C1"
+		(property "Reference" "C401"
 			(at 148.59 30.48 0)
 			(effects
@@
 			(project "tc2-mic-pcb"
 				(path "/5f96247b-0b73-48aa-a1a8-3d96ade9d103"
-					(reference "C1")
+					(reference "C401")
 					(unit 1)
 				)
@@
 		(dnp no)
 		(fields_autoplaced yes)
-		(property "Reference" "#FLG02"
+		(property "Reference" "#FLG0403"
 			(at 81.28 88.265 0)
 			(effects
@@
 			(project "tc2-mic-pcb"
 				(path "/5f96247b-0b73-48aa-a1a8-3d96ade9d103"
-					(reference "#FLG02")
+					(reference "#FLG0403")
 					(unit 1)
 				)
@@
 		(dnp no)
 		(fields_autoplaced yes)
-		(property "Reference" "#PWR05"
+		(property "Reference" "#PWR0401"
 			(at 154.94 30.48 0)
 			(effects
@@
 			(project "tc2-mic-pcb"
 				(path "/5f96247b-0b73-48aa-a1a8-3d96ade9d103"
-					(reference "#PWR05")
+					(reference "#PWR0401")
 					(unit 1)
 				)
@@
 		(on_board yes)
 		(dnp no)
-		(property "Reference" "J4"
+		(property "Reference" "J401"
 			(at 62.23 83.82 0)
 			(effects
@@
 			(project "tc2-mic-pcb"
 				(path "/5f96247b-0b73-48aa-a1a8-3d96ade9d103"
-					(reference "J4")
+					(reference "J401")
 					(unit 1)
 				)
@@
 		(on_board yes)
 		(dnp no)
-		(property "Reference" "R1"
+		(property "Reference" "R403"
 			(at 186.69 57.15 90)
 			(effects
@@
 			(project "tc2-mic-pcb"
 				(path "/5f96247b-0b73-48aa-a1a8-3d96ade9d103"
-					(reference "R1")
+					(reference "R403")
 					(unit 1)
 				)
@@
 		(dnp no)
 		(fields_autoplaced yes)
-		(property "Reference" "C4"
+		(property "Reference" "C405"
 			(at 58.42 47.6313 0)
 			(effects
@@
 			(project "tc2-mic-pcb"
 				(path "/5f96247b-0b73-48aa-a1a8-3d96ade9d103"
-					(reference "C4")
+					(reference "C405")
 					(unit 1)
 				)
@@
 		(on_board yes)
 		(dnp no)
-		(property "Reference" "C5"
+		(property "Reference" "C404"
 			(at 16.51 46.99 0)
 			(effects
@@
 			(project "tc2-mic-pcb"
 				(path "/5f96247b-0b73-48aa-a1a8-3d96ade9d103"
-					(reference "C5")
+					(reference "C404")
 					(unit 1)
 				)
@@
 		(on_board yes)
 		(dnp no)
-		(property "Reference" "R3"
+		(property "Reference" "R402"
 			(at 120.65 55.88 90)
 			(effects
@@
 			(project "tc2-mic-pcb"
 				(path "/5f96247b-0b73-48aa-a1a8-3d96ade9d103"
-					(reference "R3")
+					(reference "R402")
 					(unit 1)
 				)
@@
 		(on_board yes)
 		(dnp no)
-		(property "Reference" "MK1"
+		(property "Reference" "MK401"
 			(at 99.06 44.45 0)
 			(effects
@@
 			(project "tc2-mic-pcb"
 				(path "/5f96247b-0b73-48aa-a1a8-3d96ade9d103"
-					(reference "MK1")
+					(reference "MK401")
 					(unit 1)
 				)
@@
 			(project "tc2-mic-pcb"
 				(path "/5f96247b-0b73-48aa-a1a8-3d96ade9d103"
-					(reference "J1")
+					(reference "J403")
 					(unit 1)
 				)
@@
 		(dnp no)
 		(fields_autoplaced yes)
-		(property "Reference" "#PWR016"
+		(property "Reference" "#PWR0414"
 			(at 160.02 72.39 0)
 			(effects
@@
 			(project "tc2-mic-pcb"
 				(path "/5f96247b-0b73-48aa-a1a8-3d96ade9d103"
-					(reference "#PWR016")
+					(reference "#PWR0414")
 					(unit 1)
 				)
@@
 		(dnp no)
 		(fields_autoplaced yes)
-		(property "Reference" "#PWR04"
+		(property "Reference" "#PWR0404"
 			(at 170.18 45.72 0)
 			(effects
@@
 			(project "tc2-mic-pcb"
 				(path "/5f96247b-0b73-48aa-a1a8-3d96ade9d103"
-					(reference "#PWR04")
+					(reference "#PWR0404")
 					(unit 1)
 				)
@@
 		(dnp no)
 		(fields_autoplaced yes)
-		(property "Reference" "U3"
+		(property "Reference" "U401"
 			(at 39.37 38.1 0)
 			(effects
@@
 			(project "tc2-mic-pcb"
 				(path "/5f96247b-0b73-48aa-a1a8-3d96ade9d103"
-					(reference "U3")
+					(reference "U401")
 					(unit 1)
 				)
@@
 		(dnp no)
 		(fields_autoplaced yes)
-		(property "Reference" "U2"
+		(property "Reference" "U402"
 			(at 161.9759 64.77 0)
 			(effects
@@
 			(project "tc2-mic-pcb"
 				(path "/5f96247b-0b73-48aa-a1a8-3d96ade9d103"
-					(reference "U2")
+					(reference "U402")
 					(unit 1)
 				)
@@
 		(on_board yes)
 		(dnp no)
-		(property "Reference" "C3"
+		(property "Reference" "C402"
 			(at 163.83 34.29 0)
 			(effects
@@
 			(project "tc2-mic-pcb"
 				(path "/5f96247b-0b73-48aa-a1a8-3d96ade9d103"
-					(reference "C3")
+					(reference "C402")
 					(unit 1)
 				)
@@
 		(dnp no)
 		(fields_autoplaced yes)
-		(property "Reference" "#FLG03"
+		(property "Reference" "#FLG0401"
 			(at 59.69 37.465 0)
 			(effects
@@
 			(project "tc2-mic-pcb"
 				(path "/5f96247b-0b73-48aa-a1a8-3d96ade9d103"
-					(reference "#FLG03")
+					(reference "#FLG0401")
 					(unit 1)
 				)
@@
 		(dnp no)
 		(fields_autoplaced yes)
-		(property "Reference" "#FLG01"
+		(property "Reference" "#FLG0402"
 			(at 69.85 84.455 0)
 			(effects
@@
 			(project "tc2-mic-pcb"
 				(path "/5f96247b-0b73-48aa-a1a8-3d96ade9d103"
-					(reference "#FLG01")
+					(reference "#FLG0402")
 					(unit 1)
 				)
@@
 		(dnp no)
 		(fields_autoplaced yes)
-		(property "Reference" "#PWR014"
+		(property "Reference" "#PWR0411"
 			(at 22.86 59.69 0)
 			(effects
@@
 			(project "tc2-mic-pcb"
 				(path "/5f96247b-0b73-48aa-a1a8-3d96ade9d103"
-					(reference "#PWR014")
+					(reference "#PWR0411")
 					(unit 1)
 				)
@@
 		(dnp no)
 		(fields_autoplaced yes)
-		(property "Reference" "#PWR011"
+		(property "Reference" "#PWR0417"
 			(at 69.85 101.6 0)
 			(effects
@@
 			(project "tc2-mic-pcb"
 				(path "/5f96247b-0b73-48aa-a1a8-3d96ade9d103"
-					(reference "#PWR011")
+					(reference "#PWR0417")
 					(unit 1)
 				)
@@
 			(project "tc2-mic-pcb"
 				(path "/5f96247b-0b73-48aa-a1a8-3d96ade9d103"
-					(reference "#PWR03")
+					(reference "#PWR0410")
 					(unit 1)
 				)
@@
 		(dnp no)
 		(fields_autoplaced yes)
-		(property "Reference" "#PWR07"
+		(property "Reference" "#PWR0406"
 			(at 107.95 46.99 0)
 			(effects
@@
 			(project "tc2-mic-pcb"
 				(path "/5f96247b-0b73-48aa-a1a8-3d96ade9d103"
-					(reference "#PWR07")
+					(reference "#PWR0406")
 					(unit 1)
 				)
@@
 		(dnp no)
 		(fields_autoplaced yes)
-		(property "Reference" "#PWR012"
+		(property "Reference" "#PWR0408"
 			(at 55.88 46.99 0)
 			(effects
@@
 			(project "tc2-mic-pcb"
 				(path "/5f96247b-0b73-48aa-a1a8-3d96ade9d103"
-					(reference "#PWR012")
+					(reference "#PWR0408")
 					(unit 1)
 				)
@@
 		(dnp no)
 		(fields_autoplaced yes)
-		(property "Reference" "#PWR015"
+		(property "Reference" "#PWR0405"
 			(at 76.2 44.45 0)
 			(effects
@@
 			(project "tc2-mic-pcb"
 				(path "/5f96247b-0b73-48aa-a1a8-3d96ade9d103"
-					(reference "#PWR015")
+					(reference "#PWR0405")
 					(unit 1)
 				)
@@
 		(dnp no)
 		(fields_autoplaced yes)
-		(property "Reference" "#PWR08"
+		(property "Reference" "#PWR0402"
 			(at 170.18 34.29 0)
 			(effects
@@
 			(project "tc2-mic-pcb"
 				(path "/5f96247b-0b73-48aa-a1a8-3d96ade9d103"
-					(reference "#PWR08")
+					(reference "#PWR0402")
 					(unit 1)
 				)
@@
 		(dnp no)
 		(fields_autoplaced yes)
-		(property "Reference" "#PWR010"
+		(property "Reference" "#PWR0416"
 			(at 39.37 99.06 0)
 			(effects
@@
 			(project "tc2-mic-pcb"
 				(path "/5f96247b-0b73-48aa-a1a8-3d96ade9d103"
-					(reference "#PWR010")
+					(reference "#PWR0416")
 					(unit 1)
 				)
@@
 		(dnp no)
 		(fields_autoplaced yes)
-		(property "Reference" "#PWR017"
+		(property "Reference" "#PWR0409"
 			(at 147.32 46.99 0)
 			(effects
@@
 			(project "tc2-mic-pcb"
 				(path "/5f96247b-0b73-48aa-a1a8-3d96ade9d103"
-					(reference "#PWR017")
+					(reference "#PWR0409")
 					(unit 1)
 				)
@@
 			(project "tc2-mic-pcb"
 				(path "/5f96247b-0b73-48aa-a1a8-3d96ade9d103"
-					(reference "J2")
+					(reference "J402")
 					(unit 1)
 				)
@@
 		(on_board yes)
 		(dnp no)
-		(property "Reference" "R2"
+		(property "Reference" "R401"
 			(at 134.62 44.45 90)
 			(effects
@@
 			(project "tc2-mic-pcb"
 				(path "/5f96247b-0b73-48aa-a1a8-3d96ade9d103"
-					(reference "R2")
+					(reference "R401")
 					(unit 1)
 				)
@@
 		(dnp no)
 		(fields_autoplaced yes)
-		(property "Reference" "#PWR013"
+		(property "Reference" "#PWR0412"
 			(at 55.88 59.69 0)
 			(effects
@@
 			(project "tc2-mic-pcb"
 				(path "/5f96247b-0b73-48aa-a1a8-3d96ade9d103"
-					(reference "#PWR013")
+					(reference "#PWR0412")
 					(unit 1)
 				)
@@
 		(dnp no)
 		(fields_autoplaced yes)
-		(property "Reference" "#PWR02"
+		(property "Reference" "#PWR0403"
 			(at 154.94 41.91 0)
 			(effects
@@
 			(project "tc2-mic-pcb"
 				(path "/5f96247b-0b73-48aa-a1a8-3d96ade9d103"
-					(reference "#PWR02")
+					(reference "#PWR0403")
 					(unit 1)
 				)
@@
 		(dnp no)
 		(fields_autoplaced yes)
-		(property "Reference" "#PWR09"
+		(property "Reference" "#PWR0407"
 			(at 22.86 46.99 0)
 			(effects
@@
 			(project "tc2-mic-pcb"
 				(path "/5f96247b-0b73-48aa-a1a8-3d96ade9d103"
-					(reference "#PWR09")
-					(unit 1)
-				)
+					(reference "#PWR0407")
+					(unit 1)
+				)

Commit message: v0.7.2 panelise microphone boards
Parts:
- added C406: 1uF, Capacitor_SMD:C_0402_1005Metric, symbol Device:C_Small
Connections:
- net +3V3: now also C406.1
- net GND: now also C406.2
Changed lines of the file:
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@@
+	)
+	(junction
+		(at 81.28 91.44)
+		(diameter 0)
+		(color 0 0 0 0)
 	)
 	(junction
@@
 	(wire
 		(pts
+			(xy 81.28 91.44) (xy 81.28 92.71)
+		)
+		(stroke
+			(width 0)
+			(type default)
+		)
+	)
+	(wire
+		(pts
 			(xy 154.94 34.29) (xy 154.94 35.56)
 		)
@@
 		(pts
 			(xy 22.86 44.45) (xy 26.67 44.45)
+		)
+		(stroke
+			(width 0)
+			(type default)
+		)
+	)
+	(wire
+		(pts
+			(xy 81.28 97.79) (xy 81.28 99.06)
 		)
 		(stroke
@@
 	)
 	(symbol
+		(lib_id "Device:C_Small")
+		(at 81.28 95.25 0)
+		(unit 1)
+		(exclude_from_sim no)
+		(in_bom yes)
+		(on_board yes)
+		(dnp no)
+		(fields_autoplaced yes)
+		(property "Reference" "C406"
+			(at 83.82 94.6213 0)
+			(effects
+				(font
+					(size 1.27 1.27)
+				)
+				(justify left)
+			)
+		)
+		(property "Value" "1uF"
+			(at 83.82 97.1613 0)
+			(effects
+				(font
+					(size 1.27 1.27)
+				)
+				(justify left)
+			)
+		)
+		(property "Footprint" "Capacitor_SMD:C_0402_1005Metric"
+			(at 81.28 95.25 0)
+			(effects
+				(font
+					(size 1.27 1.27)
+				)
+				(hide yes)
+			)
+		)
+		(property "Datasheet" "~"
+			(at 81.28 95.25 0)
+			(effects
+				(font
+					(size 1.27 1.27)
+				)
+				(hide yes)
+			)
+		)
+		(property "Description" ""
+			(at 81.28 95.25 0)
+			(effects
+				(font
+					(size 1.27 1.27)
+				)
+				(hide yes)
+			)
+		)
+		(property "LCSC" "C52923"
+			(at 81.28 95.25 0)
+			(effects
+				(font
+					(size 1.27 1.27)
+				)
+				(hide yes)
+			)
+		)
+		(pin "1"
+		)
+		(pin "2"
+		)
+		(instances
+			(project "tc2-mic-pcb"
+				(path "/5f96247b-0b73-48aa-a1a8-3d96ade9d103"
+					(reference "C406")
+					(unit 1)
+				)
+			)
+		)
+	)
+	(symbol
 		(lib_id "power:PWR_FLAG")
 		(at 81.28 90.17 0)
@@
 					(unit 1)
 				)
+			)
+		)
+	)
+	(symbol
+		(lib_id "power:GND")
+		(at 81.28 99.06 0)
+		(unit 1)
+		(exclude_from_sim no)
+		(in_bom yes)
+		(on_board yes)
+		(dnp no)
+		(fields_autoplaced yes)
+		(property "Reference" "#PWR0418"
+			(at 81.28 105.41 0)
+			(effects
+				(font
+					(size 1.27 1.27)
+				)
+				(hide yes)
+			)
+		)
+		(property "Value" "GND"
+			(at 81.28 104.14 0)
+			(effects
+				(font
+					(size 1.27 1.27)
+				)
+			)
+		)
+		(property "Footprint" ""
+			(at 81.28 99.06 0)
+			(effects
+				(font
+					(size 1.27 1.27)
+				)
+				(hide yes)
+			)
+		)
+		(property "Datasheet" ""
+			(at 81.28 99.06 0)
+			(effects
+				(font
+					(size 1.27 1.27)
+				)
+				(hide yes)
+			)
+		)
+		(property "Description" "Power symbol creates a global label with name \"GND\" , ground"
+			(at 81.28 99.06 0)
+			(effects
+				(font
+					(size 1.27 1.27)
+				)
+				(hide yes)
+			)
+		)
+		(pin "1"
+		)
+		(instances
+			(project "tc2-mic-pcb"
+				(path "/5f96247b-0b73-48aa-a1a8-3d96ade9d103"
+					(reference "#PWR0418")
+					(unit 1)
+				)
