File: tc2-mic-pcb/tc2-mic-pcb.kicad_sch (KiCad schematic)
At the start: 15 parts, among them J401 Conn_02x03_Odd_Even, J7 Screw_Terminal_01x01, U401 AP7335-18SNG-7, U402 TXS0102DCT

Commit message: 0.8.0 WIP
Parts:
- R401, R402, R403: value 22R -> 22Ω
Changed lines of the file:
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@@
 	(label "CLOCK"
 		(at 106.68 50.8 0)
-		(fields_autoplaced yes)
 		(effects
 			(font
@@
 	(label "PDM_DATA_PHY"
 		(at 171.45 54.61 0)
-		(fields_autoplaced yes)
 		(effects
 			(font
@@
 	(label "DATA"
 		(at 135.89 54.61 0)
-		(fields_autoplaced yes)
 		(effects
 			(font
@@
 	(label "DATA_PHY"
 		(at 106.68 53.34 0)
-		(fields_autoplaced yes)
 		(effects
 			(font
@@
 	(label "CLOCK_PHY"
 		(at 149.86 49.53 180)
-		(fields_autoplaced yes)
 		(effects
 			(font
@@
 			)
 		)
-		(property "Value" "22R"
+		(property "Value" "22Ω"
 			(at 186.69 59.69 90)
 			(effects
@@
 			)
 		)
-		(property "Value" "22R"
+		(property "Value" "22Ω"
 			(at 120.65 58.42 90)
 			(effects
@@
 			)
 		)
-		(property "Value" "22R"
+		(property "Value" "22Ω"
 			(at 134.62 46.99 90)
 			(effects
