File: tc2-touch-sensor/tc2-touch-sensor.kicad_pcb (KiCad board)
At the start: 2 copper layers, 50.6 x 17.3 mm, 23 parts, among them J301 Screw_Terminal_01x01, J302 Conn_02x03_Odd_Even, J303 Screw_Terminal_01x01, Q301 AO3400A, U301 ME6216A28XG, U302 AT42QT1010-TSHR

Commit message: Small updates
Parts:
- added R307: 100k, Resistor_SMD:R_0402_1005Metric, F.Cu at (14.2, 4.43)
Connections:
- C302 pad 1: Net-(D301-K) -> ~{CAP_BUTTON}
- D301 pad 1: Net-(D301-K) -> ~{CAP_BUTTON}
- J302 pad 3: CAP_BUTTON -> ~{CAP_BUTTON}
- Q301 pad 3: Net-(D301-K) -> ~{CAP_BUTTON}
Routing:
- net ~{CAP_BUTTON}: track 0.00 -> 56.6 mm, vias 0 -> 2
- net Net-(D301-K): track 40.0 -> 0.00 mm
- net CAP_BUTTON: track 24.2 -> 12.0 mm, vias 6 -> 2

Commit message: version v0.7.1
Routing:
- net ~{CAP_BUTTON}: track 56.6 -> 53.4 mm
- net ~{LED_G}: track 6.85 -> 4.73 mm
- net ~{LED_B}: track 9.11 -> 7.77 mm
- net ~{LED_R}: track 6.95 -> 6.90 mm, vias 2 -> 0

Commit message: v0.7.3
Parts:
- added REF**: Tab, PCM_kikit:Tab, F.Cu at (17.6, 8.69)
- added REF**: Tab, PCM_kikit:Tab, F.Cu at (19.7, -9.53)
- added REF**: Tab, PCM_kikit:Tab, F.Cu at (28.0, -0.90)
- added REF**: Tab, PCM_kikit:Tab, F.Cu at (-12.1, -9.52)
- added REF**: Tab, PCM_kikit:Tab, F.Cu at (-15.2, 8.73)
Other:
- copper layers 2 -> 6

Commit message: 0.8.0 WIP
Parts:
- R301, R304, R305, R306: value 180R -> 180Ω
Changed lines of the file:
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@@
 			)
 		)
-		(property "Value" "180R"
+		(property "Value" "180Ω"
 			(at 0 1.17 90)
 			(layer "F.Fab")
@@
 			)
 		)
-		(property "Value" "180R"
+		(property "Value" "180Ω"
 			(at 0 1.17 90)
 			(layer "F.Fab")
@@
 			)
 		)
-		(property "Value" "180R"
+		(property "Value" "180Ω"
 			(at 0 1.17 90)
 			(layer "F.Fab")
@@
 			)
 		)
-		(property "Value" "180R"
+		(property "Value" "180Ω"
 			(at 0 1.17 90)
 			(layer "F.Fab")
