File: tc2-touch-sensor/tc2-touch-sensor.kicad_sch (KiCad schematic)
At the start: 23 parts, among them J301 Screw_Terminal_01x01, J302 Conn_02x03_Odd_Even, J303 Screw_Terminal_01x01, Q301 AO3400A, U301 ME6216A28XG, U302 AT42QT1010-TSHR

Commit message: Small updates
Parts:
- added R307: 100k, Resistor_SMD:R_0402_1005Metric, symbol Device:R
Connections:
- net +3V3: now also R307.2
- net CAP_BUTTON: no longer J302.3 (Pin_3)
- net ~{CAP_BUTTON}: now reaches C302.1, D301.1 (K), Q301.3 (D)
- net ~{CAP_BUTTON}: now also J302.3 (Pin_3), R307.1
Other:
- moved on the sheet: C301, C302, D301, Q301, R301

Commit message: 0.8.0 WIP
Parts:
- R301, R304, R305, R306: value 180R -> 180Ω
Changed lines of the file:
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@@
 			)
 		)
-		(property "Value" "180R"
+		(property "Value" "180Ω"
 			(at 49.53 143.51 90)
 			(effects
@@
 			)
 		)
-		(property "Value" "180R"
+		(property "Value" "180Ω"
 			(at 80.01 143.51 90)
 			(effects
@@
 			)
 		)
-		(property "Value" "180R"
+		(property "Value" "180Ω"
 			(at 80.01 156.21 90)
 			(effects
@@
 			)
 		)
-		(property "Value" "180R"
+		(property "Value" "180Ω"
 			(at 86.36 85.09 0)
 			(effects
