File: tc2-plugs-buck-boost-pcb/tc2-plugs-buck-boost-pcb.kicad_sch (KiCad schematic)
At the start: 71 parts, among them J201 JCON_M16_04Pin, J202 JCON_M16_2+4Pin, J204 Conn_02x07_Odd_Even, Q1 Q_PMOS_GSD, Q203 AO3400A, U1001 ICSRC3908SFR, U1002 ICSRC3908SFR, U1003 ICSRC3908SFR, U1004 ICSRC3908SFR, U1005 TPS63070, U201 TPS63070, U203 TPS259541DSGR, U206 ICSRC3908SFR, U210 ICSRC3908SFR, U211 ICSRC3908SFR, U212 ICSRC3908SFR

Commit message: 0.8.0 WIP
Parts:
- removed C203: 22uF, Capacitor_SMD:C_0805_2012Metric, symbol Device:C_Small
- removed C210: 8.2nF, Capacitor_SMD:C_0402_1005Metric, symbol Device:C_Small
- removed R201: 680Ω, Resistor_SMD:R_0402_1005Metric, symbol Device:R
- removed TP204: TestPoint, cacophony-library:TP_PAD, symbol Connector:TestPoint
- removed U1001, U210: ICSRC3908SFR, cacophony-library:CONN-SMD_L3.9-W0.8, symbol cacophony-library:ICSRC3908SFR
- removed U203: TPS259541DSGR, cacophony-library:WFDFN-8_L2.0-W2.0-P0.50-BL-EP, symbol cacophony-library:TPS259541DSGR
- added C211, C213: 2.2uF, Capacitor_SMD:C_0402_1005Metric, symbol Device:C_Small
- added C212: 220pF, Capacitor_SMD:C_0402_1005Metric, symbol Device:C_Small
- added D201: D_Zener, Diode_SMD:D_SOD-323, symbol Device:D_Zener
- added L201: ACM4520-901-2P-t000, cacophony-library:FILTER-SMD_4P-L4.7-W4.5-BL, symbol cacophony-library:ACM4520-901-2P-t000
- added R207, R212: 470k, Resistor_SMD:R_0402_1005Metric, symbol Device:R
- added R208: 1k, Resistor_SMD:R_0402_1005Metric, symbol Device:R
- added R210: 8.2k, Resistor_SMD:R_0402_1005Metric, symbol Device:R
- added R214: 100k, Resistor_SMD:R_0402_1005Metric, symbol Device:R
- added TP205, TP207: TestPoint, cacophony-library:TP_PAD, symbol Connector:TestPoint
- added U201: TPS259474LRPWR, cacophony-library:VQFN-10_L2.0-W2.0-P0.45-TL, symbol cacophony-library:TPS259474LRPWR
- R217: value 180R -> 180Ω
Connections:
- net GND: now also C211.2, C212.2, C213.2, D201.2 (A), L201.3, R207.2, R208.1, R210.2, U201.8 (GND); no longer J201.1
- net VCC: now also U201.6 (OUT)
- net VIN_PHY: now also L201.1
- new net: TP207.1, U201.4 (PGTH)
- new net: D201.1 (K), R207.1, R212.2, U201.1 (EN/UVLO)
- new net: C211.1, U201.10 (ITIMER)
- new net: R210.1, R214.2, U201.2 (OVLO)
- new net: TP205.1, U201.3 (PG)
- new net: C212.1, U201.7 (DVDT)
- new net: R208.2, U201.9 (ILM)
- new net GND_PHY: J201.1, L201.2
- new net VIN_PRE_FUSE: C213.1, L201.4, R212.1, R214.1, U201.5 (IN)
Other:
- moved on the sheet: C203, C38, C43, F201, Q1, Q203, R14, R38, TP6

Commit message: Updated to use field LCSC Part instead of LCSC for the JLCPCB part number
Parts:
- C1001, C1002, C203: LCSC C45783 -> (none); LCSC Part (none) -> C45783
- C1003, C204, C213: LCSC C159814 -> (none); LCSC Part (none) -> C159814
- C1004, C205: LCSC C15525 -> (none); LCSC Part (none) -> C15525
- C1005, C1006, C1007, C1008, C206, C207, C208, C209: LCSC C86295 -> (none); LCSC Part (none) -> C86295
- C1009, C210: LCSC C100072 -> (none); LCSC Part (none) -> C100072
- C228: LCSC C13832 -> (none); LCSC Part (none) -> C13832
- C38, C43: LCSC C19702 -> (none); LCSC Part (none) -> C19702
- D202: LCSC C15879 -> (none); LCSC Part (none) -> C15879
- F201: LCSC C187605 -> (none); LCSC Part (none) -> C187605
- FB1, FB1001: LCSC C76818 -> (none); LCSC Part (none) -> C76818
- L1001, L3: LCSC C5179452 -> (none); LCSC Part (none) -> C5179452
- Q1: LCSC C15127 -> (none); LCSC Part (none) -> C15127
- Q203: LCSC C20917 -> (none); LCSC Part (none) -> C20917
- R1004, R211, R213, R214, R219, R38: LCSC C25741 -> (none); LCSC Part (none) -> C25741
- R14, R208: LCSC C11702 -> (none); LCSC Part (none) -> C11702
- R202, R203: LCSC C326730 -> (none); LCSC Part (none) -> C326730
- R207, R212, R216, R221: LCSC C319591 -> (none); LCSC Part (none) -> C319591
- R217: LCSC C38941 -> (none); LCSC Part (none) -> C38941
- R218: LCSC C445618 -> (none); LCSC Part (none) -> C445618
- R222: LCSC C852538 -> (none); LCSC Part (none) -> C852538
- U1002, U1003, U1004, U206, U211, U212: LCSC C238203 -> (none)
- U1005, U201: LCSC C109322 -> (none); LCSC Part C109322 -> C109322
Changed lines of the file:
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@@
 			)
 		)
-		(property "LCSC" "C187605"
+		(property "LCSC Part" "C187605"
 			(at 384.81 104.14 90)
 			(effects
@@
 			)
 		)
-		(property "LCSC" "C45783"
+		(property "LCSC Part" "C45783"
 			(at 317.5 33.02 0)
 			(effects
@@
 			)
 		)
-		(property "LCSC" "C238203"
+		(property "LCSC Part" "C238203"
 			(at 222.25 111.76 0)
 			(effects
@@
 			)
 		)
-		(property "LCSC" "C319591"
+		(property "LCSC Part" "C319591"
 			(at 299.72 149.86 0)
 			(effects
@@
 			)
 		)
-		(property "LCSC" "C238203"
-			(at 170.18 200.66 0)
-			(effects
-				(font
-					(size 1.27 1.27)
-				)
-				(hide yes)
-			)
-		)
 		(pin "1"
 		)
@@
 			)
 		)
-		(property "LCSC" "C86295"
+		(property "LCSC Part" "C86295"
 			(at 349.25 148.59 0)
 			(effects
@@
 			)
 		)
-		(property "LCSC" "C238203"
-			(at 170.18 217.17 0)
-			(effects
-				(font
-					(size 1.27 1.27)
-				)
-				(hide yes)
-			)
-		)
 		(pin "1"
 		)
@@
 			)
 		)
-		(property "LCSC" "C13832"
+		(property "LCSC Part" "C13832"
 			(at 38.1 40.64 0)
 			(effects
@@
 			)
 		)
-		(property "LCSC" "C76818"
+		(property "LCSC Part" "C76818"
 			(at 379.73 212.09 0)
 			(effects
@@
 			)
 		)
-		(property "LCSC" "C11702"
+		(property "LCSC Part" "C11702"
 			(at 252.73 58.42 90)
 			(effects
@@
 			)
 		)
-		(property "LCSC" "C100072"
+		(property "LCSC Part" "C100072"
 			(at 255.27 172.72 0)
 			(effects
@@
 			)
 		)
-		(property "LCSC" "C109322 "
+		(property "LCSC Part" "C109322 "
 			(at 279.4 218.44 0)
 			(effects
@@
 			)
 		)
-		(property "LCSC" "C100072"
+		(property "LCSC Part" "C100072"
 			(at 262.89 240.03 0)
 			(effects
@@
 			)
 		)
-		(property "LCSC" "C86295"
+		(property "LCSC Part" "C86295"
 			(at 356.87 215.9 0)
 			(effects
@@
 			)
 		)
-		(property "LCSC" "C159814"
+		(property "LCSC Part" "C159814"
 			(at 125.73 27.94 0)
 			(effects
@@
 			)
 		)
-		(property "LCSC" "C319591"
+		(property "LCSC Part" "C319591"
 			(at 308.61 215.9 0)
 			(effects
@@
 			)
 		)
-		(property "LCSC" "C45783"
+		(property "LCSC Part" "C45783"
 			(at 327.66 33.02 0)
 			(effects
@@
 			)
 		)
-		(property "LCSC" "C45783"
+		(property "LCSC Part" "C45783"
 			(at 228.6 148.59 0)
 			(effects
@@
 			)
 		)
-		(property "LCSC" "C25741"
+		(property "LCSC Part" "C25741"
 			(at 179.07 27.94 0)
 			(effects
@@
 			)
 		)
-		(property "LCSC" "C86295"
+		(property "LCSC Part" "C86295"
 			(at 336.55 215.9 0)
 			(effects
@@
 			)
 		)
-		(property "LCSC" "C38941"
+		(property "LCSC Part" "C38941"
 			(at 48.26 35.56 0)
 			(effects
@@
 			)
 		)
-		(property "LCSC" "C25741"
+		(property "LCSC Part" "C25741"
 			(at 307.34 227.33 0)
 			(effects
@@
 			)
 		)
-		(property "LCSC" "C86295"
+		(property "LCSC Part" "C86295"
 			(at 328.93 148.59 0)
 			(effects
@@
 			)
 		)
-		(property "LCSC" "C45783"
+		(property "LCSC Part" "C45783"
 			(at 358.14 33.02 0)
 			(effects
@@
 			)
 		)
-		(property "LCSC" "C86295"
+		(property "LCSC Part" "C86295"
 			(at 360.68 148.59 0)
 			(effects
@@
 			)
 		)
-		(property "LCSC" "C15879"
+		(property "LCSC Part" "C15879"
 			(at 50.8 177.8 0)
 			(effects
@@
 			)
 		)
-		(property "LCSC" "C326730"
+		(property "LCSC Part" "C326730"
 			(at 26.67 40.64 0)
 			(effects
@@
 			)
 		)
-		(property "LCSC" "C45783"
+		(property "LCSC Part" "C45783"
 			(at 226.06 215.9 0)
 			(effects
@@
 			)
 		)
-		(property "LCSC" "C45783"
+		(property "LCSC Part" "C45783"
 			(at 218.44 148.59 0)
 			(effects
@@
 			)
 		)
-		(property "LCSC" "C86295"
+		(property "LCSC Part" "C86295"
 			(at 346.71 215.9 0)
 			(effects
@@
 			)
 		)
-		(property "LCSC" "C76818"
+		(property "LCSC Part" "C76818"
 			(at 372.11 144.78 0)
 			(effects
@@
 			)
 		)
-		(property "LCSC" "C25741"
+		(property "LCSC Part" "C25741"
 			(at 205.74 264.16 0)
 			(effects
@@
 			)
 		)
-		(property "LCSC" "C159814"
+		(property "LCSC Part" "C159814"
 			(at 242.57 148.59 0)
 			(effects
@@
 			)
 		)
-		(property "LCSC" "C159814"
+		(property "LCSC Part" "C159814"
 			(at 254 215.9 0)
 			(effects
@@
 			)
 		)
-		(property "LCSC" "C445618"
+		(property "LCSC Part" "C445618"
 			(at 308.61 219.71 0)
 			(effects
@@
 			)
 		)
-		(property "LCSC" "C319591"
+		(property "LCSC Part" "C319591"
 			(at 163.83 29.21 0)
 			(effects
@@
 			)
 		)
-		(property "LCSC" "C852538"
+		(property "LCSC Part" "C852538"
 			(at 299.72 160.02 0)
 			(effects
@@
 			)
 		)
-		(property "LCSC" "C25741"
+		(property "LCSC Part" "C25741"
 			(at 195.58 236.22 0)
 			(effects
@@
 			)
 		)
-		(property "LCSC" "C45783"
+		(property "LCSC Part" "C45783"
 			(at 368.3 33.02 0)
 			(effects
@@
 			)
 		)
-		(property "LCSC" "C109322 "
+		(property "LCSC Part" "C109322 "
 			(at 271.78 151.13 0)
 			(effects
@@
 			)
 		)
-		(property "LCSC" "C15525"
+		(property "LCSC Part" "C15525"
 			(at 323.85 215.9 0)
 			(effects
@@
 			)
 		)
-		(property "LCSC" "C20917"
+		(property "LCSC Part" "C20917"
 			(at 337.82 104.14 0)
 			(effects
@@
 			)
 		)
-		(property "LCSC" "C11702"
+		(property "LCSC Part" "C11702"
 			(at 320.04 104.14 90)
 			(effects
@@
 			)
 		)
-		(property "LCSC" "C15525"
+		(property "LCSC Part" "C15525"
 			(at 316.23 148.59 0)
 			(effects
@@
 			)
 		)
-		(property "LCSC" "C86295"
+		(property "LCSC Part" "C86295"
 			(at 339.09 148.59 0)
 			(effects
@@
 			)
 		)
-		(property "LCSC" "C238203"
+		(property "LCSC Part" "C238203"
 			(at 212.09 106.68 0)
 			(effects
@@
 			)
 		)
-		(property "LCSC" "C326730"
+		(property "LCSC Part" "C326730"
 			(at 16.51 40.64 0)
 			(effects
@@
 			)
 		)
-		(property "LCSC" "C19702"
+		(property "LCSC Part" "C19702"
 			(at 367.03 109.22 0)
 			(effects
@@
 			)
 		)
-		(property "LCSC" "C25741"
+		(property "LCSC Part" "C25741"
 			(at 351.79 92.71 0)
 			(effects
@@
 			)
 		)
-		(property "LCSC" "C25741"
+		(property "LCSC Part" "C25741"
 			(at 312.42 160.02 0)
 			(effects
@@
 			)
 		)
-		(property "LCSC" "C25741"
+		(property "LCSC Part" "C25741"
 			(at 331.47 109.22 0)
 			(effects
@@
 			)
 		)
-		(property "LCSC" "C5179452"
+		(property "LCSC Part" "C5179452"
 			(at 279.4 195.58 0)
 			(effects
@@
 			)
 		)
-		(property "LCSC" "C45783"
+		(property "LCSC Part" "C45783"
 			(at 347.98 33.02 0)
 			(effects
@@
 			)
 		)
-		(property "LCSC" "C25741"
+		(property "LCSC Part" "C25741"
 			(at 320.04 227.33 0)
 			(effects
@@
 			)
 		)
-		(property "LCSC" "C19702"
+		(property "LCSC Part" "C19702"
 			(at 373.38 86.36 0)
 			(effects
@@
 			)
 		)
-		(property "LCSC" "C45783"
+		(property "LCSC Part" "C45783"
 			(at 337.82 33.02 0)
 			(effects
@@
 			)
 		)
-		(property "LCSC" "C319591"
+		(property "LCSC Part" "C319591"
 			(at 163.83 39.37 0)
 			(effects
@@
 			)
 		)
-		(property "LCSC" "C5179452"
+		(property "LCSC Part" "C5179452"
 			(at 271.78 128.27 0)
 			(effects
@@
 			)
 		)
-		(property "LCSC" "C238203"
-			(at 179.07 209.55 0)
-			(effects
-				(font
-					(size 1.27 1.27)
-				)
-				(hide yes)
-			)
-		)
 		(pin "1"
 		)
@@
 			)
 		)
-		(property "LCSC" "C238203"
+		(property "LCSC Part" "C238203"
 			(at 236.22 106.68 0)
 			(effects
@@
 			)
 		)
-		(property "LCSC" "C15127"
+		(property "LCSC Part" "C15127"
 			(at 359.41 97.79 0)
 			(effects
@@
 			)
 		)
-		(property "LCSC" "C45783"
+		(property "LCSC Part" "C45783"
 			(at 236.22 215.9 0)
 			(effects
@@
 			)
 		)
-		(property "LCSC" "C86295"
+		(property "LCSC Part" "C86295"
 			(at 368.3 215.9 0)
 			(effects

Commit message: Tidy up
Parts:
- J204: now fitted
Changed lines of the file:
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@@
 		(in_bom yes)
 		(on_board yes)
-		(dnp yes)
+		(dnp no)
 		(fields_autoplaced yes)
 		(property "Reference" "J204"

Commit message: Update to kicad 9, fix microphone panel v cuts
Parts:
- J204: LCSC Part (none) -> C5577333; MPN (none) -> BF060-14A-B-0600-0280-0305-L-D
- renumbered C203 to C202, C203 to C204, C203 to C205, C203 to C206, C203 to C207, C43 to C208, C38 to C209, C203 to C219, C203 to C220, C204 to C221, C205 to C222, C206 to C223, C208 to C224, C209 to C225, C207 to C226, C210 to C227, FB1 to FB202, L3 to L202, Q1 to Q202, R38 to R204, R14 to R205, R38 to R206, R38 to R215, TP6 to TP201, TP6 to TP202, TP6 to TP203, U201 to U202
