File: tc2-plugs-buck-boost-pcb/tc2-plugs-buck-boost-pcb.kicad_pcb (KiCad board)
At the start: 6 copper layers, 65 x 19.5 mm, 65 parts, among them J201 JCON_M16_04Pin, J202 JCON_M16_2+4Pin, J203 Conn_02x06_Odd_Even, Q201 Q_PMOS_GSD, Q202 Q_PMOS_GSD, Q203 AO3400A, U201 TPS63070RNMR, U202 TPS63071

Commit message: Add JLPCPCB 2D barcode to PCBs
Parts:
- added U203: ~, cacophony-library:JLCPCB_QR_8mm, B.Cu at (-25.6, -8.60)
- R217: value 180R -> 180Ω

Commit message: Update layout
Parts:
- removed C201: 22uF, Capacitor_SMD:C_0805_2012Metric
- removed D201: D_Zener, cacophony-library:LL-34_L3.5-W1.5-RD
- removed Q201: Q_PMOS_GSD, Package_TO_SOT_SMD:SOT-23
- removed R201: 100k, Resistor_SMD:R_0402_1005Metric
- added C229: 10nF, Capacitor_SMD:C_0402_1005Metric, F.Cu at (-23.5, -14.5)
- added C230: 470pF, Capacitor_SMD:C_0402_1005Metric, F.Cu at (-19.4, -14.5)
- added C231: 470pF, Capacitor_SMD:C_0402_1005Metric, F.Cu at (-8.75, 0.98)
- added C232: 470pF, Capacitor_SMD:C_0402_1005Metric, F.Cu at (-10.6, 0.98)
- added D203: D_Zener, Diode_SMD:D_SOD-323, F.Cu at (-24.4, -12.4)
- added R216: 100k, Resistor_SMD:R_0402_1005Metric, F.Cu at (-24.2, -9.76)
- added R218: 68k, Resistor_SMD:R_0402_1005Metric, F.Cu at (-25.2, -9.76)
- added R219: 1k, Resistor_SMD:R_0402_1005Metric, F.Cu at (15.2, -8.07)
- added R220: 1k, Resistor_SMD:R_0402_1005Metric, F.Cu at (16.6, -6.36)
- added R221: 1k, Resistor_SMD:R_0402_1005Metric, F.Cu at (-21.7, -14.5)
- added R222: 120k, Resistor_SMD:R_0402_1005Metric, F.Cu at (-22.3, -9.89)
- added R223: 10k, Resistor_SMD:R_0402_1005Metric, F.Cu at (-23.3, -9.53)
- added TP205: TestPoint, cacophony-library:TP_PAD, F.Cu at (-21.2, -10.1)
- added TP207: TestPoint, cacophony-library:TP_PAD, F.Cu at (-19.7, -10.1)
- added U204: TPS259474LRPWR, cacophony-library:VQFN-10_L2.0-W2.0-P0.45-TL, F.Cu at (-21.9, -12.4)
- C228: value 1uF -> 2.2uF; footprint Capacitor_SMD:C_1206_3216Metric -> Capacitor_SMD:C_0402_1005Metric
- L201, L202: value INDUCTOR -> 1.5uH
- R212: value 680k -> 150k
- R214: value 130k -> 820k
- U202: value TPS63071 -> TPS63070
- moved R203 14.3 mm to (-9.65, -1.01)
- moved R202 14.2 mm to (-8.19, -1.01)
- moved C206 13.0 mm to (-28.1, -5.57), turned to 180 degrees
- moved C202 10.3 mm to (-28.1, -7.53), turned to 180 degrees
- moved R217 9.93 mm to (-10.9, -1.34), turned to 90 degrees
- moved C207 8.30 mm to (-24.7, -5.57), turned to 0 degrees
- moved C203 7.59 mm to (-28.1, -9.49), turned to 180 degrees
- moved C228 5.98 mm to (-19.8, -12.7)
- moved C205 5.92 mm to (-24.7, -7.53), turned to 0 degrees
- moved C204 4.95 mm to (-28.1, -11.4), turned to 180 degrees
- moved D202 0.79 mm to (14.4, -5.48)
- moved R212 0.67 mm to (-20.8, 2.00), turned to 0 degrees
- moved R214 0.66 mm to (-20.8, 1.06), turned to 180 degrees
Connections:
- net Net-(J201-Pad4) renamed /BATT_SENSE_PHY
- C228 pad 1: Net-(C228-Pad1) -> /VIN_PHY
- J202 pad 2: OUT_RX -> /OUT_RX_PHY
- J202 pad 3: OUT_TX -> /OUT_TX_PHY
- R202 pad 1: Net-(C228-Pad1) -> /BATT_SENSE
- R203 pad 1: Net-(C228-Pad1) -> /BATT_SENSE
- R212 pad 1: /5V_PHY -> Net-(U202-FB)
- R212 pad 2: unconnected-(R212-Pad2) -> GND
- R214 pad 1: unconnected-(R214-Pad1) -> /5V_PHY
- R214 pad 2: GND -> Net-(U202-FB)
- R217 pad 1: Net-(C228-Pad1) -> /BATT_SENSE
- U202 pad 5: /5V_PHY -> Net-(U202-FB)
Routing:
- net BATTERY_HV: track 34.4 -> 12.3 mm, vias 2 -> 0
- net BATTERY_LV: track 28.8 -> 8.61 mm, vias 2 -> 0
- net OUT_TX: track 29.1 -> 22.3 mm
- net GND: track 7.97 -> 14.0 mm, vias 76 -> 73
- net /OUT_TX_PHY: track 0.00 -> 5.82 mm
- net /VIN_PHY: track 2.99 -> 8.28 mm
- net /BATT_SENSE: track 0.00 -> 5.23 mm
- net /BATT_SENSE_PHY: track 2.74 -> 7.47 mm
- net Net-(C228-Pad1): track 4.18 -> 0.00 mm
- net Net-(D203-K): track 0.00 -> 4.12 mm
- net Net-(D201-A): track 3.60 -> 0.00 mm
- net VCC: track 6.08 -> 2.73 mm, vias 32 -> 27
- net OUT_RX: track 27.8 -> 24.6 mm
- net Net-(U204-DVDT): track 0.00 -> 2.79 mm
- net /OUT_RX_PHY: track 0.00 -> 2.63 mm
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- added copper zone on F.Cu, net /VIN_PHY

Commit message: Add git hash to PCBs
Other:
- board text added: "${HASH}"
