File: tc2-sim-usb-pcb/tc2-sim-usb-pcb.kicad_sch (KiCad schematic)
At the start: 9 parts, among them J11 Conn_01x08

Commit message: Fixed panel tabs
Parts:
- USB501: LCSC (none) -> C283546
Changed lines of the file:
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@@
+			)
+		)
+		(property "LCSC" "C283546"
+			(at 219.71 59.69 0)
+			(effects
+				(font
+					(size 1.27 1.27)
+				)
+				(hide yes)
 			)
 		)

Commit message: Upgraded to new kicad version
Parts:
- D501: renamed from D4; LCSC Part (none) -> C15879
- U503: LCSC Part (none) -> C2919617
- renumbered C37 to C501, J11 to J501
Changed lines of the file:
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@@
 (kicad_sch
-	(version 20231120)
+	(version 20250114)
 	(generator "eeschema")
-	(generator_version "8.0")
+	(generator_version "9.0")
 	(paper "A4")
 	(junction
@@
 		(dnp no)
 		(fields_autoplaced yes)
-		(property "Reference" "D4"
+		(property "Reference" "D501"
 			(at 102.87 104.775 0)
 			(effects
@@
 				)
 				(hide yes)
+			)
+		)
+		(property "LCSC Part" "C15879"
+			(at 95.25 104.14 0)
+			(effects
+				(font
+					(size 0.0254 0.0254)
+				)
 			)
 		)
@@
 		(dnp no)
 		(fields_autoplaced yes)
-		(property "Reference" "#PWR076"
+		(property "Reference" "#PWR0502"
 			(at 99.06 88.9 0)
 			(effects
@@
 		(dnp no)
 		(fields_autoplaced yes)
-		(property "Reference" "J11"
+		(property "Reference" "J501"
 			(at 238.76 130.81 0)
 			(effects
@@
 		(dnp no)
 		(fields_autoplaced yes)
-		(property "Reference" "#PWR077"
+		(property "Reference" "#PWR0504"
 			(at 95.25 120.65 0)
 			(effects
@@
 			)
 		)
+		(property "LCSC Part" "C2919617"
+			(at 120.904 81.026 0)
+			(effects
+				(font
+					(size 1.27 1.27)
+				)
+			)
+		)
 		(pin "C6"
 		)
@@
 		(dnp no)
 		(fields_autoplaced yes)
-		(property "Reference" "#PWR077"
+		(property "Reference" "#PWR0503"
 			(at 129.54 102.87 0)
 			(effects
@@
 		(on_board yes)
 		(dnp no)
-		(property "Reference" "C37"
+		(property "Reference" "C501"
 			(at 100.33 78.74 90)
 			(effects
@@
 		(dnp no)
 		(fields_autoplaced yes)
-		(property "Reference" "#PWR079"
+		(property "Reference" "#PWR0506"
 			(at 229.87 148.59 0)
 			(effects
@@
 		)
 	)
+	(embedded_fonts no)
 )

Commit message: Tidy up for making an order for v0.7.3
Parts:
- C501: LCSC C16772 -> (none); LCSC Part (none) -> C16772
- D501: LCSC C15879 -> (none)
- U503: LCSC C2919617 -> (none)
- USB501: LCSC C283546 -> (none)
Changed lines of the file:
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@@
 			)
 		)
-		(property "LCSC" "C15879"
+		(property "LCSC Part" "C15879"
 			(at 95.25 104.14 0)
 			(effects
@@
 			)
 		)
-		(property "LCSC" "C283546"
+		(property "LCSC Part" "C283546"
 			(at 219.71 59.69 0)
 			(effects
@@
 			)
 		)
-		(property "LCSC" "C2919617"
+		(property "LCSC Part" "C2919617"
 			(at 120.015 83.82 0)
 			(effects
@@
 			)
 		)
-		(property "LCSC" "C16772"
+		(property "LCSC Part" "C16772"
 			(at 102.87 81.28 0)
 			(effects
