File: tc2-sim-usb-pcb/tc2-sim-usb-pcb.kicad_pcb (KiCad board)
At the start: 6 copper layers, 22.4 x 58.2 mm, 12 parts, among them J501 Conn_01x08

Commit message: Add JLPCPCB 2D barcode to PCBs
Parts:
- added U504: ~, cacophony-library:JLCPCB_QR_8mm, B.Cu at (13.8, -10.2)
Routing:
- net USIM_RST: track 23.8 -> 22.2 mm
Changed lines of the file:
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@@
+		(embedded_fonts no)
+	)
+	(footprint "cacophony-library:JLCPCB_QR_8mm"
+		(layer "B.Cu")
+		(at 13.8 -10.2 180)
+		(property "Reference" "U504"
+			(at 0 0.5 0)
+			(unlocked yes)
+			(layer "B.SilkS")
+			(hide yes)
+			(effects
+				(font
+					(size 1 1)
+					(thickness 0.1)
+				)
+				(justify mirror)
+			)
+		)
+		(property "Value" "~"
+			(at 0 -1 0)
+			(unlocked yes)
+			(layer "B.Fab")
+			(effects
+				(font
+					(size 1 1)
+					(thickness 0.15)
+				)
+				(justify mirror)
+			)
+		)
+		(property "Datasheet" ""
+			(at 0 0 0)
+			(unlocked yes)
+			(layer "B.Fab")
+			(hide yes)
+			(effects
+				(font
+					(size 1 1)
+					(thickness 0.15)
+				)
+				(justify mirror)
+			)
+		)
+		(property "Description" ""
+			(at 0 0 0)
+			(unlocked yes)
+			(layer "B.Fab")
+			(hide yes)
+			(effects
+				(font
+					(size 1 1)
+					(thickness 0.15)
+				)
+				(justify mirror)
+			)
+		)
+		(sheetname "/")
+		(sheetfile "tc2-sim-usb-pcb.kicad_sch")
+		(attr exclude_from_pos_files exclude_from_bom)
+		(duplicate_pad_numbers_are_jumpers no)
+		(fp_rect
+			(start -4 4)
+			(end 4 -4)
+			(stroke
+				(width 0)
+				(type solid)
+			)
+			(fill yes)
+			(layer "B.SilkS")
+		)
+		(fp_text user "${REFERENCE}"
+			(at 0 -2.5 0)
+			(unlocked yes)
+			(layer "B.Fab")
+			(effects
+				(font
+					(size 1 1)
+					(thickness 0.15)
+				)
+				(justify mirror)
+			)
+		)
 		(embedded_fonts no)
 	)
@@
 	)
 	(segment
-		(start 5.395554 -1.33)
-		(end 10.405554 -6.34)
-		(width 0.25)
-		(layer "F.Cu")
-		(net "USIM_RST")
-	)
-	(segment
 		(start 4.36 -0.5)
 		(end 4.6 -0.74)
@@
 	)
 	(segment
-		(start 10.405554 -6.34)
-		(end 14.83 -6.34)
+		(start 4.6 -0.75)
+		(end 4.6 -0.74)
 		(width 0.25)
 		(layer "F.Cu")
@@
 	)
 	(segment
+		(start 9.432777 -5.367223)
+		(end 5.395554 -1.33)
+		(width 0.25)
+		(layer "F.Cu")
+		(net "USIM_RST")
+	)
+	(segment
 		(start 0 0)
 		(end 2.5 0)
@@
 	)
 	(segment
-		(start 5.18 -1.33)
-		(end 5.395554 -1.33)
-		(width 0.25)
-		(layer "F.Cu")
-		(net "USIM_RST")
-	)
-	(segment
-		(start 4.6 -0.74)
-		(end 4.6 -0.75)
+		(start 5.395554 -1.33)
+		(end 5.18 -1.33)
 		(width 0.25)
 		(layer "F.Cu")
@@
 	)
 	(segment
+		(start 5.18 -1.33)
+		(end 4.6 -0.75)
+		(width 0.25)
+		(layer "F.Cu")
+		(net "USIM_RST")
+	)
+	(segment
 		(start 15.77 -3.51)
 		(end 15.77 -2.63)
@@
 		(net "USIM_RST")
 	)
-	(segment
-		(start 4.6 -0.75)
-		(end 5.18 -1.33)
-		(width 0.25)
-		(layer "F.Cu")
-		(net "USIM_RST")
-	)
 	(via
-		(at 14.83 -6.34)
+		(at 9.432777 -5.367223)
 		(size 0.8)
 		(drill 0.4)
@@
 	)
 	(segment
-		(start 15.550004 -5.619996)
-		(end 14.83 -6.34)
+		(start 9.432777 -5.367223)
+		(end 14.372777 -5.367223)
 		(width 0.25)
 		(layer "B.Cu")
@@
 	)
 	(segment
-		(start 15.550004 -4.189996)
-		(end 15.550004 -5.619996)
+		(start 14.372777 -5.367223)
+		(end 15.550004 -4.189996)
 		(width 0.25)
 		(layer "B.Cu")

Commit message: Add git hash to PCBs
Other:
- board text added: "${HASH}"
Changed lines of the file:
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@@
+		)
+	)
+	(gr_text "${HASH}"
+		(at 5.28 14.46 90)
+		(layer "F.SilkS")
+		(effects
+			(font
+				(size 1.5 1.5)
+				(thickness 0.3)
+				(bold yes)
+			)
+			(justify left bottom)
+		)
+	)
+	(gr_text "${HASH}"
+		(at 3.52 14.25 -90)
+		(layer "B.SilkS")
+		(effects
+			(font
+				(size 1.5 1.5)
+				(thickness 0.3)
+				(bold yes)
+			)
+			(justify left bottom mirror)
 		)
 	)
